File: MK1_CPU/8bit-computer/8bit-computer.kicad_pcb (KiCad board)
At the start: 2 copper layers, 318.8 x 180.3 mm, 368 parts, among them J1 Barrel_Jack_Switch, J2 USB_B-8bit-computer-rescue, U1 74LS86, U10 74LS273, U11 74LS08, U12 74LS173, U13 74LS00, U14 74LS02, U15 74LS245, U16 74LS283, U17 74LS283, U18 74LS157, U19 74LS157, U2 74LS73, U20 74LS157, U21 74LS86, U22 74LS86, U23 74LS157, U24 74LS32, U25 74LS08, U26 74LS08, U27 74LS32, U28 74LS157, U29 74LS157, U3 LM555, U30 74LS273, U31 LM555, U32 74LS08, U33 74LS273, U35 28C64, U36 7SEGMENT_CC, U37 74LS139, U38 7SEGMENT_CC, U39 7SEGMENT_CC, U4 74LS04, U40 7SEGMENT_CC, U41 74LS00, U42 74LS161, U43 74LS138, U44 AM29F040, U45 AM29F040, U46 AM29F040, U47 74LS04, U48 74LS245, U49 74LS161, U5 74LS08, U50 74LS161, U51 74LS157, U52 CY62256, U53 74LS245, U54 74LS245, U55 74LS00, U56 74LS157, U57 74LS157, U58 74LS245, U59 74LS273, U6 LM555, U60 74LS273, U61 74LS00, U62 74LS157, U63 74LS157, U64 74LS245, U65 74LS273, U66 74LS157, U67 74LS157, U68 74LS245, U69 74LS04, U7 74LS32, U70 74LS273, U71 74LS04, U72 74LS04, U73 74LS08, U74 74LS245, U75 74LS04, U8 LM555, U9 74LS245

Commit message: version 2.0
Parts:
- removed ? (x4): MountingHole_3.2mm_M3, MountingHole:MountingHole_3.2mm_M3
- removed D101, D102, D103, D104, D108: RED, LED_THT:LED_D3.0mm
- removed R100, R101, R103, R104, R105, R106, R107, R108, R109, R110, R111, R112, R113, R114, R115, R116, R117, R118, R119, R120, R121, R122, R123, R124, R125, R126, R127, R128, R129, R130, R131, R132, R133, R134, R26, R27, R28, R29, R30, R31, R32, R35, R37, R38, R39, R40, R41, R42, R43, R44, R45, R46, R48, R50, R51, R56, R57, R58, R59, R60, R61, R62, R63, R64, R65, R66, R67, R68, R69, R70, R71, R72, R73, R74, R75, R76, R77, R78, R79, R80, R81, R82, R83, R84, R85, R86, R87, R88, R89, R90, R91, R92, R93, R94, R95, R96, R97, R98, R99: 220, Resistor_THT:R_Axial_DIN0207_L6.3mm_D2.5mm_P7.62mm_Horizontal
- removed R102, R135, R136, R137, R138, R47, R49, R54, R55: 1K, Resistor_THT:R_Axial_DIN0207_L6.3mm_D2.5mm_P7.62mm_Horizontal
- removed R52: 10k, Resistor_THT:R_Axial_DIN0207_L6.3mm_D2.5mm_P7.62mm_Horizontal
- removed R53: 100K, Resistor_THT:R_Axial_DIN0207_L6.3mm_D2.5mm_P7.62mm_Horizontal
- added C26: 0.1µF, Capacitor_THT:C_Disc_D4.3mm_W1.9mm_P5.00mm, F.Cu at (27.9, 137.2)
- added C27: 0.1µF, Capacitor_THT:C_Disc_D4.3mm_W1.9mm_P5.00mm, F.Cu at (47.0, 137.2)
- added C28: 0.1µF, Capacitor_THT:C_Disc_D4.3mm_W1.9mm_P5.00mm, F.Cu at (280.7, 123.1)
- added C29: *, Capacitor_THT:C_Disc_D4.3mm_W1.9mm_P5.00mm, F.Cu at (276.9, 123.1)
- added C30: *, Capacitor_THT:C_Disc_D4.3mm_W1.9mm_P5.00mm, F.Cu at (259.1, 118.2)
- added C31: *, Capacitor_THT:C_Disc_D4.3mm_W1.9mm_P5.00mm, F.Cu at (262.9, 123.1)
- added C32: 0.1µF, Capacitor_THT:C_Disc_D4.3mm_W1.9mm_P5.00mm, F.Cu at (222.3, 72.4)
- added C33: *, Capacitor_THT:C_Disc_D4.3mm_W1.9mm_P5.00mm, F.Cu at (204.5, 72.4)
- added C34: *, Capacitor_THT:C_Disc_D4.3mm_W1.9mm_P5.00mm, F.Cu at (90.2, 137.2)
- added C35: *, Capacitor_THT:C_Disc_D4.3mm_W1.9mm_P5.00mm, F.Cu at (93.3, 137.1)
- added C36: 0.1µF, Capacitor_THT:C_Disc_D4.3mm_W1.9mm_P5.00mm, F.Cu at (96.5, 137.2)
- added C37: 0.1µF, Capacitor_THT:C_Disc_D4.3mm_W1.9mm_P5.00mm, F.Cu at (162.6, 82.5)
- added C38: *, Capacitor_THT:C_Disc_D4.3mm_W1.9mm_P5.00mm, F.Cu at (129.5, 82.5)
- added C39: 0.1µF, Capacitor_THT:C_Disc_D4.3mm_W1.9mm_P5.00mm, F.Cu at (152.4, 183.6)
- added C40: 0.1µF, Capacitor_THT:C_Disc_D4.3mm_W1.9mm_P5.00mm, F.Cu at (147.3, 183.6)
- added C41: 0.1µF, Capacitor_THT:C_Disc_D4.3mm_W1.9mm_P5.00mm, F.Cu at (194.9, 97.8)
- added C42: *, Capacitor_THT:C_Disc_D4.3mm_W1.9mm_P5.00mm, F.Cu at (177.2, 97.8)
- added C43: 10µF, Capacitor_THT:CP_Radial_D5.0mm_P2.00mm, F.Cu at (129.5, 16.5)
- added D116: BLUE, LED_THT:LED_D3.0mm, F.Cu at (205.7, 162.6)
- added D117: BLUE, LED_THT:LED_D3.0mm, F.Cu at (161.3, 151.1)
- added D118: BLUE, LED_THT:LED_D3.0mm, F.Cu at (212.1, 162.6)
- added D119: BLUE, LED_THT:LED_D3.0mm, F.Cu at (167.6, 151.1)
- added D120: BLUE, LED_THT:LED_D3.0mm, F.Cu at (218.4, 162.6)
- added D121: BLUE, LED_THT:LED_D3.0mm, F.Cu at (174.0, 151.1)
- added D122: BLUE, LED_THT:LED_D3.0mm, F.Cu at (224.8, 162.6)
- added D123: BLUE, LED_THT:LED_D3.0mm, F.Cu at (180.3, 151.1)
- added D124: BLUE, LED_THT:LED_D3.0mm, F.Cu at (186.7, 151.1)
- added D125: BLUE, LED_THT:LED_D3.0mm, F.Cu at (193.0, 151.1)
- added D126: BLUE, LED_THT:LED_D3.0mm, F.Cu at (199.4, 151.1)
- added D127: BLUE, LED_THT:LED_D3.0mm, F.Cu at (205.7, 151.1)
- added D128: BLUE, LED_THT:LED_D3.0mm, F.Cu at (212.1, 151.1)
- added D129: BLUE, LED_THT:LED_D3.0mm, F.Cu at (218.4, 151.1)
- added D130: BLUE, LED_THT:LED_D3.0mm, F.Cu at (224.8, 151.1)
- added D131: BLUE, LED_THT:LED_D3.0mm, F.Cu at (123.2, 162.6)
- added D132: BLUE, LED_THT:LED_D3.0mm, F.Cu at (129.5, 162.6)
- added D133: BLUE, LED_THT:LED_D3.0mm, F.Cu at (135.9, 162.6)
- added D134: BLUE, LED_THT:LED_D3.0mm, F.Cu at (142.2, 162.6)
- added D135: BLUE, LED_THT:LED_D3.0mm, F.Cu at (180.3, 162.6)
- added D136: BLUE, LED_THT:LED_D3.0mm, F.Cu at (167.6, 162.6)
- added D137: BLUE, LED_THT:LED_D3.0mm, F.Cu at (174.0, 162.6)
- added D138: BLUE, LED_THT:LED_D3.0mm, F.Cu at (154.9, 162.6)
- added D139: BLUE, LED_THT:LED_D3.0mm, F.Cu at (161.3, 162.6)
- added D140: GREEN, LED_THT:LED_D3.0mm, F.Cu at (178.4, 104.1)
- added D141: GREEN, LED_THT:LED_D3.0mm, F.Cu at (184.8, 104.1)
- added D142: GREEN, LED_THT:LED_D3.0mm, F.Cu at (191.1, 104.1)
- added D143: GREEN, LED_THT:LED_D3.0mm, F.Cu at (197.5, 104.1)
- added D144: GREEN, LED_THT:LED_D3.0mm, F.Cu at (203.8, 104.1)
- added D145: GREEN, LED_THT:LED_D3.0mm, F.Cu at (210.2, 104.1)
- added D146: GREEN, LED_THT:LED_D3.0mm, F.Cu at (216.5, 104.1)
- added D147: GREEN, LED_THT:LED_D3.0mm, F.Cu at (222.9, 104.1)
- added J3: EXT-Bus, Connector_PinHeader_2.54mm:PinHeader_1x08_P2.54mm_Vertical, F.Cu at (94.0, 14.7)
- added J4: EXT-Signal, Connector_PinHeader_2.54mm:PinHeader_1x08_P2.54mm_Vertical, F.Cu at (71.1, 14.7)
- added J5: EXT-Power, Connector_PinHeader_2.54mm:PinHeader_1x02_P2.54mm_Vertical, F.Cu at (117.9, 14.7)
- added JP1: RST_EN, Jumper:SolderJumper-2_P1.3mm_Open_RoundedPad1.0x1.5mm, B.Cu at (218.4, 143.5)
- added JP2: 6-STAGES, Jumper:SolderJumper-2_P1.3mm_Bridged_RoundedPad1.0x1.5mm, B.Cu at (158.4, 181.5)
- added JP3: Arduino_VIN, Jumper:SolderJumper-2_P1.3mm_Bridged_RoundedPad1.0x1.5mm, B.Cu at (54.0, 160.0)
- added MH0: MountingHole_3.2mm_M3, MountingHole:MountingHole_3.2mm_M3, F.Cu at (306.1, 12.7)
- added MH1: MountingHole_3.2mm_M3, MountingHole:MountingHole_3.2mm_M3, F.Cu at (14.0, 12.7)
- added MH2: MountingHole_3.2mm_M3, MountingHole:MountingHole_3.2mm_M3, F.Cu at (14.0, 188.0)
- added MH3: MountingHole_3.2mm_M3, MountingHole:MountingHole_3.2mm_M3, F.Cu at (306.1, 188.0)
- added RN1: 220, Resistor_THT:R_Array_SIP9, F.Cu at (191.8, 26.7)
- added RN10: 10K, Resistor_THT:R_Array_SIP9, F.Cu at (63.5, 165.1)
- added RN11: 220, Resistor_THT:R_Array_SIP9, F.Cu at (115.6, 177.8)
- added RN12: 1K, Resistor_THT:R_Array_SIP9, F.Cu at (91.4, 177.8)
- added RN13: 1K, Resistor_THT:R_Array_SIP9, F.Cu at (226.1, 123.2)
- added RN14: 1K, Resistor_THT:R_Array_SIP9, F.Cu at (144.8, 172.7)
- added RN15: 1K, Resistor_THT:R_Array_SIP9, F.Cu at (146.1, 143.5)
- added RN16: 1K, Resistor_THT:R_Array_SIP9, F.Cu at (166.4, 135.9)
- added RN17: 1K, Resistor_THT:R_Array_SIP9, F.Cu at (171.4, 172.7)
- added RN18: 1K, Resistor_THT:R_Array_SIP9, F.Cu at (199.4, 172.7)
- added RN19: 1K, Resistor_THT:R_Array_SIP9, F.Cu at (226.1, 172.7)
- added RN2: 220, Resistor_THT:R_Array_SIP9, F.Cu at (191.8, 16.5)
- added RN20: 1K, Resistor_THT:R_Array_SIP9, F.Cu at (226.7, 97.8)
- added RN21: 1K, Resistor_THT:R_Array_SIP9, F.Cu at (135.9, 97.8)
- added RN3: 1K, Resistor_THT:R_Array_SIP9, F.Cu at (226.7, 47.0)
- added RN4: 470, Resistor_THT:R_Array_SIP9, F.Cu at (292.1, 35.8)
- added RN5: 470, Resistor_THT:R_Array_SIP9, F.Cu at (36.8, 50.0)
- added RN6: 220, Resistor_THT:R_Array_SIP9, F.Cu at (82.5, 52.1)
- added RN7: 1K, Resistor_THT:R_Array_SIP9, F.Cu at (50.2, 132.1)
- added RN8: 220, Resistor_THT:R_Array_SIP9, F.Cu at (255.3, 120.7)
- added RN9: 1K, Resistor_THT:R_Array_SIP9, F.Cu at (198.8, 72.4)
- added S0: OSHW-Logo_11.4x12mm_SilkScreen, Symbol:OSHW-Logo_11.4x12mm_SilkScreen, B.Cu at (40.6, 177.8)
- added S1: LOGO, Symbol:parrot, F.Cu at (91.9, 120.9)
- added S2: Symbol_Barrel_Polarity, Symbol:Symbol_Barrel_Polarity, F.Cu at (149.2, 18.4)
- added SW10: Reset, Button_Switch_THT:SW_PUSH_6mm_H5mm, F.Cu at (170.7, 179.1)
- added SW9: Data, Button_Switch_THT:SW_DIP_SPSTx08_Slide_9.78x22.5mm_W7.62mm_P2.54mm, F.Cu at (35.6, 102.2)
- added TP1: CLK_IN, TestPoint:TestPoint_Pad_1.0x1.0mm, B.Cu at (97.0, 111.8)
- added TP10: AND, TestPoint:TestPoint_Pad_1.0x1.0mm, B.Cu at (170.2, 167.6)
- added TP11: EI, TestPoint:TestPoint_Pad_1.0x1.0mm, B.Cu at (263.5, 71.1)
- added TP12: ~EO, TestPoint:TestPoint_Pad_1.0x1.0mm, B.Cu at (218.4, 156.2)
- added TP13: NOT, TestPoint:TestPoint_Pad_1.0x1.0mm, B.Cu at (157.5, 167.6)
- added TP14: SUB, TestPoint:TestPoint_Pad_1.0x1.0mm, B.Cu at (182.9, 167.6)
- added TP15: MI, TestPoint:TestPoint_Pad_1.0x1.0mm, B.Cu at (43.2, 50.2)
- added TP16: OI, TestPoint:TestPoint_Pad_1.0x1.0mm, B.Cu at (254.6, 161.9)
- added TP17: ~PO, TestPoint:TestPoint_Pad_1.0x1.0mm, B.Cu at (92.7, 27.3)
- added TP18: PE, TestPoint:TestPoint_Pad_1.0x1.0mm, B.Cu at (113.0, 27.9)
- added TP19: ~PI, TestPoint:TestPoint_Pad_1.0x1.0mm, B.Cu at (105.9, 25.4)
- added TP2: CLK, TestPoint:TestPoint_Pad_1.0x1.0mm, B.Cu at (81.3, 97.5)
- added TP20: ~RO, TestPoint:TestPoint_Pad_1.0x1.0mm, B.Cu at (59.7, 67.3)
- added TP21: RI, TestPoint:TestPoint_Pad_1.0x1.0mm, B.Cu at (48.3, 85.1)
- added TP22: ~SO, TestPoint:TestPoint_Pad_1.0x1.0mm, B.Cu at (237.5, 112.3)
- added TP23: SU, TestPoint:TestPoint_Pad_1.0x1.0mm, B.Cu at (302.3, 112.0)
- added TP24: SD, TestPoint:TestPoint_Pad_1.0x1.0mm, B.Cu at (293.4, 132.3)
- added TP25: SI, TestPoint:TestPoint_Pad_1.0x1.0mm, B.Cu at (298.4, 124.7)
- added TP26: ~REG-O, TestPoint:TestPoint_Pad_1.0x1.0mm, B.Cu at (207.0, 64.0)
- added TP27: REG-I, TestPoint:TestPoint_Pad_1.0x1.0mm, B.Cu at (200.0, 64.0)
- added TP28: ~IO, TestPoint:TestPoint_Pad_1.0x1.0mm, B.Cu at (81.7, 146.1)
- added TP29: II, TestPoint:TestPoint_Pad_1.0x1.0mm, B.Cu at (78.7, 134.9)
- added TP3: ~CLK, TestPoint:TestPoint_Pad_1.0x1.0mm, B.Cu at (102.9, 108.5)
- added TP30: AI, TestPoint:TestPoint_Pad_1.0x1.0mm, B.Cu at (132.8, 82.5)
- added TP31: ~AO, TestPoint:TestPoint_Pad_1.0x1.0mm, B.Cu at (165.1, 55.9)
- added TP32: RGT, TestPoint:TestPoint_Pad_1.0x1.0mm, B.Cu at (154.9, 79.2)
- added TP33: ROT, TestPoint:TestPoint_Pad_1.0x1.0mm, B.Cu at (161.3, 90.7)
- added TP34: SHF, TestPoint:TestPoint_Pad_1.0x1.0mm, B.Cu at (163.8, 167.6)
- added TP35: E0, TestPoint:TestPoint_Pad_1.0x1.0mm, B.Cu at (208.3, 167.6)
- added TP36: EXT_IN, TestPoint:TestPoint_Pad_1.0x1.0mm, B.Cu at (127.0, 44.5)
- added TP37: E1, TestPoint:TestPoint_Pad_1.0x1.0mm, B.Cu at (214.6, 167.6)
- added TP38: U0, TestPoint:TestPoint_Pad_1.0x1.0mm, B.Cu at (221.0, 167.6)
- added TP39: U1, TestPoint:TestPoint_Pad_1.0x1.0mm, B.Cu at (227.3, 167.6)
- added TP4: ~REG-O, TestPoint:TestPoint_Pad_1.0x1.0mm, B.Cu at (207.0, 38.6)
- added TP40: ~CU_EN, TestPoint:TestPoint_Pad_1.0x1.0mm, B.Cu at (229.9, 133.3)
- added TP41: ~REG-O, TestPoint:TestPoint_Pad_1.0x1.0mm, B.Cu at (207.0, 89.4)
- added TP42: REG-I, TestPoint:TestPoint_Pad_1.0x1.0mm, B.Cu at (200.0, 89.4)
- added TP5: REG-I, TestPoint:TestPoint_Pad_1.0x1.0mm, B.Cu at (200.0, 38.6)
- added TP6: ~FI, TestPoint:TestPoint_Pad_1.0x1.0mm, B.Cu at (299.7, 34.3)
- added TP7: ZF, TestPoint:TestPoint_Pad_1.0x1.0mm, B.Cu at (268.7, 77.7)
- added TP8: CF, TestPoint:TestPoint_Pad_1.0x1.0mm, B.Cu at (279.4, 71.8)
- added TP9: OR, TestPoint:TestPoint_Pad_1.0x1.0mm, B.Cu at (176.5, 167.6)
- added U34: 74HCT273, Package_DIP:DIP-20_W7.62mm, F.Cu at (256.5, 143.5)
- added U77: AM29F040, Housings_LCC:PLCC-32_THT-Socket, F.Cu at (179.1, 116.8)
- added U78: AM29F040, Housings_LCC:PLCC-32_THT-Socket, F.Cu at (133.3, 116.8)
- added U79: AM29F040, Housings_LCC:PLCC-32_THT-Socket, F.Cu at (201.9, 116.8)
- added U80: AM29F040, Housings_LCC:PLCC-32_THT-Socket, F.Cu at (156.2, 116.8)
- added U81: 74HCT138, Package_DIP:DIP-16_W7.62mm, F.Cu at (124.5, 143.5)
- added U82: 74HCT238, Package_DIP:DIP-16_W7.62mm, F.Cu at (170.2, 143.5)
- added U83: 74HCT238, Package_DIP:DIP-16_W7.62mm, F.Cu at (209.6, 135.9)
- added U84: 74HCT04, Package_DIP:DIP-14_W7.62mm, F.Cu at (170.2, 15.2)
- added U85: 74HCT245, Package_DIP:DIP-20_W7.62mm, F.Cu at (204.5, 92.7)
- added U86: 74HCT273, Package_DIP:DIP-20_W7.62mm, F.Cu at (177.2, 92.7)
- A1: value Arduino_Nano_v2.x -> Arduino Nano
- C10, C11, C17, C21, C22, C24, C9: footprint Capacitor_THT:C_Rect_L7.0mm_W6.0mm_P5.00mm -> Capacitor_THT:C_Disc_D4.3mm_W1.9mm_P5.00mm
- C12, C15, C16, C23, C25: value 0.1µF -> *; footprint Capacitor_THT:C_Rect_L7.0mm_W6.0mm_P5.00mm -> Capacitor_THT:C_Disc_D4.3mm_W1.9mm_P5.00mm
- C13, C14, C4: value 0.01µF -> 0.1µF
- C18, C19, C5, C8: value 0.1µF -> 0.01µF; footprint Capacitor_THT:C_Rect_L7.0mm_W6.0mm_P5.00mm -> Capacitor_THT:C_Disc_D4.3mm_W1.9mm_P5.00mm
- C20: value 0.01µF -> *
- C7: value 0.1µF -> 1µF; footprint Capacitor_THT:C_Rect_L7.0mm_W6.0mm_P5.00mm -> Capacitor_THT:CP_Radial_D5.0mm_P2.00mm
- D10, D105, D106, D107, D109, D110, D111, D112, D113, D114, D115, D80, D81, D82, D83: value RED -> BLUE
- D100, D76, D77, D78, D79: value RED -> YELLOW
- D11, D12, D13, D14, D15, D16, D17: value RED -> GREEN
- D19: value GREEN -> WHITE
- D20: value RED -> WHITE
- D28, D29, D30, D31, D34, D35, D36, D37: value YELLOW -> RED
- D33: value GREEN -> RED
- D38, D39, D40, D41, D42, D43, D72, D73, D74, D75: value GREEN -> YELLOW
- D44, D45, D48, D55, D56, D57, D58, D59, D60, D61, D62, D63, D98, D99: value BLUE -> YELLOW
- D46, D47, D49, D50, D51, D52, D53, D54, D64, D65, D66, D67, D9, D92, D93, D94, D95: value BLUE -> GREEN
- D84, D85, D86, D87: value YELLOW -> BLUE
- D88, D89, D90, D91: value YELLOW -> GREEN
- D96, D97: value BLUE -> WHITE
- J1: value Barrel_Jack_Switch -> USB_B-8bit-computer-rescue; footprint Connector_BarrelJack:BarrelJack_Horizontal -> Connector_USB:USB_B_OST_USB-B1HSxx_Horizontal
- J2: value USB_B-8bit-computer-rescue -> Barrel_Jack_Switch; footprint Connector_USB:USB_B_OST_USB-B1HSxx_Horizontal -> Connector_BarrelJack:BarrelJack_Horizontal
- R1, R2: value 10K -> 220
- R10, R11, R14, R15, R33, R34, R9: value 220 -> 1K
- R12, R25, R36: value 220 -> 10K
- R13: value 220 -> 470
- R16: value 220 -> 100K
- R18, R19, R21, R22: value 1K -> 10K
- R20: value 1M -> 10K
- R3, R5, R6, R7, R8: value 10K -> 1K
- R4: value 10K -> 330K
- SW1: renamed from Pulse; value SW_Push -> Multiplier; footprint Button_Switch_THT:SW_PUSH_6mm_H5mm -> Button_Switch_THT:SW_DIP_SPSTx03_Slide_9.78x9.8mm_W7.62mm_P2.54mm
- SW2: renamed from Manual; value SW_NKK_GW12LHP -> Pulse; footprint Button_Switch_THT:SW_NKK_GW12LJP -> Button_Switch_THT:SW_PUSH_6mm_H5mm
- SW3: renamed from Prog; value SW_NKK_GW12LHP -> Manual
- SW4: renamed from Address; value SW_DIP_x08 -> Prog; footprint Button_Switch_THT:SW_DIP_SPSTx08_Slide_9.78x22.5mm_W7.62mm_P2.54mm -> Button_Switch_THT:SW_DIP_SPSTx01_Slide_9.78x4.72mm_W7.62mm_P2.54mm
- SW5: renamed from Mode; value SW_NKK_GW12LHP -> Address; footprint Button_Switch_THT:SW_NKK_GW12LJP -> Button_Switch_THT:SW_DIP_SPSTx10_Slide_9.78x27.58mm_W7.62mm_P2.54mm
- SW6: renamed from Reset; value Reset -> Mode; footprint Button_Switch_THT:SW_PUSH_6mm_H5mm -> Button_Switch_THT:SW_DIP_SPSTx03_Slide_9.78x9.8mm_W7.62mm_P2.54mm
- SW7: renamed from Write; value SW_Push -> Write
- SW8: renamed from Data; value SW_DIP_x08 -> Show; footprint Button_Switch_THT:SW_DIP_SPSTx08_Slide_9.78x22.5mm_W7.62mm_P2.54mm -> Button_Switch_THT:SW_PUSH_6mm_H5mm
- U1: value 74LS86 -> 74HCT32; footprint Package_DIP:DIP-14_W7.62mm_Socket -> Package_DIP:DIP-14_W7.62mm
- U10: value 74LS273 -> 74HCT08; footprint Package_DIP:DIP-20_W7.62mm_Socket -> Package_DIP:DIP-14_W7.62mm
- U11: value 74LS08 -> 74HCT173; footprint Package_DIP:DIP-14_W7.62mm_Socket -> Package_DIP:DIP-16_W7.62mm
- U12: value 74LS173 -> 74HCT02; footprint Package_DIP:DIP-16_W7.62mm_Socket -> Package_DIP:DIP-14_W7.62mm
- U13: value 74LS00 -> 74HCT245; footprint Package_DIP:DIP-14_W7.62mm_Socket -> Package_DIP:DIP-20_W7.62mm
- U14: value 74LS02 -> 74HCT283; footprint Package_DIP:DIP-14_W7.62mm_Socket -> Package_DIP:DIP-16_W7.62mm
- U15: value 74LS245 -> 74HCT283; footprint Package_DIP:DIP-20_W7.62mm_Socket -> Package_DIP:DIP-16_W7.62mm
- U16, U17: value 74LS283 -> 74HCT157; footprint Package_DIP:DIP-16_W7.62mm_Socket -> Package_DIP:DIP-16_W7.62mm
- U18, U57, U62: value 74LS157 -> 74HCT273; footprint Package_DIP:DIP-16_W7.62mm_Socket -> Package_DIP:DIP-20_W7.62mm
- U19, U66: value 74LS157 -> 74HCT157; footprint Package_DIP:DIP-16_W7.62mm_Socket -> Package_DIP:DIP-16_W7.62mm
- U2: value 74LS73 -> 74HCT32; footprint Package_DIP:DIP-14_W7.62mm_Socket -> Package_DIP:DIP-14_W7.62mm
- U20, U23: value 74LS157 -> 74HCT86; footprint Package_DIP:DIP-16_W7.62mm_Socket -> Package_DIP:DIP-14_W7.62mm
- U21: value 74LS86 -> 74HCT86; footprint Package_DIP:DIP-14_W7.62mm_Socket -> Package_DIP:DIP-14_W7.62mm
- U22: value 74LS86 -> 74HCT157; footprint Package_DIP:DIP-14_W7.62mm_Socket -> Package_DIP:DIP-16_W7.62mm
- U24, U27: value 74LS32 -> 74HCT32; footprint Package_DIP:DIP-14_W7.62mm_Socket -> Package_DIP:DIP-14_W7.62mm
- U25, U26, U32, U5: value 74LS08 -> 74HCT08; footprint Package_DIP:DIP-14_W7.62mm_Socket -> Package_DIP:DIP-14_W7.62mm
- U28: value 74LS157 -> 74HCT32; footprint Package_DIP:DIP-16_W7.62mm_Socket -> Package_DIP:DIP-14_W7.62mm
- U29, U51: footprint Package_DIP:DIP-16_W7.62mm_Socket -> Package_DIP:DIP-16_W7.62mm
- U3, U6: value LM555 -> NE555; footprint Package_DIP:DIP-8_W7.62mm_Socket -> Package_DIP:DIP-8_W7.62mm
- U30: value 74LS273 -> 74LS157; footprint Package_DIP:DIP-20_W7.62mm_Socket -> Package_DIP:DIP-16_W7.62mm
- U31: value LM555 -> 74HCT273; footprint Package_DIP:DIP-8_W7.62mm_Socket -> Package_DIP:DIP-20_W7.62mm
- U33: value 74LS273 -> NE555; footprint Package_DIP:DIP-20_W7.62mm_Socket -> Package_DIP:DIP-8_W7.62mm
- U35: value 28C64 -> 74HCT107; footprint Package_DIP:DIP-28_W15.24mm_Socket -> Package_DIP:DIP-14_W7.62mm
- U36: value 7SEGMENT_CC -> 28C64; footprint Display_7Segment:7SegmentLED_LTS6760_LTS6780 -> Package_DIP:DIP-28_W15.24mm_Socket
- U37: value 74LS139 -> 7SEGMENT_CC; footprint Package_DIP:DIP-16_W7.62mm_Socket -> Display_7Segment:7SegmentLED_LTS6760_LTS6780
- U38: value 7SEGMENT_CC -> 74HCT139; footprint Display_7Segment:7SegmentLED_LTS6760_LTS6780 -> Package_DIP:DIP-16_W7.62mm
- U4: value 74LS04 -> 74HCT04; footprint Package_DIP:DIP-14_W7.62mm_Socket -> Package_DIP:DIP-14_W7.62mm
- U41: value 74LS00 -> 7SEGMENT_CC; footprint Package_DIP:DIP-14_W7.62mm_Socket -> Display_7Segment:7SegmentLED_LTS6760_LTS6780
- U42, U49: value 74LS161 -> 74HCT245; footprint Package_DIP:DIP-16_W7.62mm_Socket -> Package_DIP:DIP-20_W7.62mm
- U43: value 74LS138 -> 74HCT161; footprint Package_DIP:DIP-16_W7.62mm_Socket -> Package_DIP:DIP-16_W7.62mm
- U44: value AM29F040 -> 74HCT161; footprint Housings_LCC:PLCC-32_THT-Socket -> Package_DIP:DIP-16_W7.62mm
- U45: value AM29F040 -> 74HCT157; footprint Housings_LCC:PLCC-32_THT-Socket -> Package_DIP:DIP-16_W7.62mm
- U46: value AM29F040 -> 74HCT00; footprint Housings_LCC:PLCC-32_THT-Socket -> Package_DIP:DIP-14_W7.62mm
- U47: value 74LS04 -> CY62256; footprint Package_DIP:DIP-14_W7.62mm_Socket -> Package_DIP:DIP-28_W15.24mm_Socket
- U48: value 74LS245 -> 74HCT245; footprint Package_DIP:DIP-20_W7.62mm_Socket -> Package_DIP:DIP-20_W7.62mm
- U50: value 74LS161 -> 74LS157; footprint Package_DIP:DIP-16_W7.62mm_Socket -> Package_DIP:DIP-16_W7.62mm
- U52: value CY62256 -> 74HCT245; footprint Package_DIP:DIP-28_W15.24mm_Socket -> Package_DIP:DIP-20_W7.62mm
- U53, U54: value 74LS245 -> 74HCT193; footprint Package_DIP:DIP-20_W7.62mm_Socket -> Package_DIP:DIP-16_W7.62mm
- U55: value 74LS00 -> 74HCT00; footprint Package_DIP:DIP-14_W7.62mm_Socket -> Package_DIP:DIP-14_W7.62mm
- U56, U67: value 74LS157 -> 74HCT245; footprint Package_DIP:DIP-16_W7.62mm_Socket -> Package_DIP:DIP-20_W7.62mm
- U58, U64, U74: value 74LS245 -> 74HCT08; footprint Package_DIP:DIP-20_W7.62mm_Socket -> Package_DIP:DIP-14_W7.62mm
- U59, U60: value 74LS273 -> 74HCT245; footprint Package_DIP:DIP-20_W7.62mm_Socket -> Package_DIP:DIP-20_W7.62mm
- U61: value 74LS00 -> 74HCT273; footprint Package_DIP:DIP-14_W7.62mm_Socket -> Package_DIP:DIP-20_W7.62mm
- U63: value 74LS157 -> 74HCT04; footprint Package_DIP:DIP-16_W7.62mm_Socket -> Package_DIP:DIP-14_W7.62mm
- U65, U70: value 74LS273 -> 74HCT157; footprint Package_DIP:DIP-20_W7.62mm_Socket -> Package_DIP:DIP-16_W7.62mm
- U68, U9: value 74LS245 -> 74HCT273; footprint Package_DIP:DIP-20_W7.62mm_Socket -> Package_DIP:DIP-20_W7.62mm
- U69: value 74LS04 -> 74HCT157; footprint Package_DIP:DIP-14_W7.62mm_Socket -> Package_DIP:DIP-16_W7.62mm
- U7: value 74LS32 -> NE555; footprint Package_DIP:DIP-14_W7.62mm_Socket -> Package_DIP:DIP-8_W7.62mm
- U71: value 74LS04 -> 74HCT02; footprint Package_DIP:DIP-14_W7.62mm_Socket -> Package_DIP:DIP-14_W7.62mm
- U72: value 74LS04 -> 74HCT245; footprint Package_DIP:DIP-14_W7.62mm_Socket -> Package_DIP:DIP-20_W7.62mm
- U73: value 74LS08 -> 74HCT107; footprint Package_DIP:DIP-14_W7.62mm_Socket -> Package_DIP:DIP-14_W7.62mm
- U75: value 74LS04 -> 74HCT161; footprint Package_DIP:DIP-14_W7.62mm_Socket -> Package_DIP:DIP-16_W7.62mm
- U8: value LM555 -> 74HCT245; footprint Package_DIP:DIP-8_W7.62mm_Socket -> Package_DIP:DIP-20_W7.62mm
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- renumbered Speed to RV1
Connections:
- A1 pad 13: Net-(A1-Pad13) -> /PC Interface/MI
- A1 pad 14: Net-(A1-Pad14) -> /PC Interface/HL
- A1 pad 15: Net-(A1-Pad15) -> /PC Interface/RI
- A1 pad 19: (no net) -> /Clock/CLK_IN
- A1 pad 20: (no net) -> /PC Interface/CLR
- A1 pad 21: (no net) -> /PC Interface/CU_DIS
- A1 pad 30: VCC -> Net-(A1-Pad30)
- C12 pad 1: VCC -> Net-(C12-Pad1)
- C13 pad 1: Net-(C13-Pad1) -> VCC
- C14 pad 1: Net-(C14-Pad1) -> VCC
- C15 pad 1: VCC -> Net-(C15-Pad1)
- C16 pad 1: VCC -> Net-(C16-Pad1)
- C18 pad 1: VCC -> Net-(C18-Pad1)
- C19 pad 1: VCC -> Net-(C19-Pad1)
- C20 pad 1: /A register/CLK -> Net-(C20-Pad1)
- C20 pad 2: Net-(C20-Pad2) -> GND
- C23 pad 1: VCC -> /Control logic/~PI
- C25 pad 1: VCC -> Net-(C25-Pad1)
- C3 pad 2: GND -> Net-(C3-Pad2)
- C4 pad 1: Net-(C4-Pad1) -> Net-(C3-Pad1)
- C4 pad 2: GND -> Net-(C4-Pad2)
- C5 pad 1: Net-(C5-Pad1) -> Net-(C3-Pad1)
- C5 pad 2: GND -> Net-(C5-Pad2)
- C7 pad 1: VCC -> Net-(C7-Pad1)
- C8 pad 1: VCC -> Net-(C8-Pad1)
- D1 pad 2: /A register/BUS_7 -> /BUS_0
- D10 pad 2: /ALU/B_7 -> /CLK
- D100 pad 2: /A register/A_7 -> Net-(D100-Pad2)
- D105 pad 2: /A register/A_2 -> /Clock/HLT
- D106 pad 2: /A register/A_1 -> /A register/ROT
- D107 pad 2: /A register/A_0 -> /Control logic/MI
- D109 pad 2: Net-(D109-Pad2) -> /Control logic/RI
- D11 pad 2: /ALU/B_6 -> /B register/OUT_7
- D110 pad 2: Net-(D110-Pad2) -> /Control logic/SU
- D112 pad 2: Net-(D112-Pad2) -> /Control logic/SD
- D113 pad 2: Net-(D113-Pad2) -> /Control logic/II
- D114 pad 2: Net-(D114-Pad2) -> /Control logic/OI
- D12 pad 2: /ALU/B_5 -> /B register/OUT_6
- D13 pad 2: /ALU/B_4 -> /B register/OUT_5
- D14 pad 2: /ALU/B_3 -> /B register/OUT_4
- D15 pad 2: /ALU/B_2 -> /B register/OUT_3
- D16 pad 2: /ALU/B_1 -> /B register/OUT_2
- D17 pad 2: /ALU/B_0 -> /B register/OUT_1
- D18 pad 2: /ALU/CF -> /B register/OUT_0
- D19 pad 2: /ALU/ZF -> /ALU/CF
- D2 pad 2: /A register/BUS_6 -> /BUS_1
- D20 pad 2: Net-(D20-Pad2) -> /ALU/ZF
- D28 pad 2: /MAR/A7 -> Net-(D28-Pad2)
- D29 pad 2: /MAR/A6 -> /MAR/A7
- D3 pad 2: /A register/BUS_5 -> /BUS_2
- D30 pad 2: /MAR/A5 -> /MAR/A6
- D31 pad 2: /MAR/A4 -> /MAR/A5
- D32 pad 1: /MAR/PROG -> Net-(D32-Pad1)
- D32 pad 2: Net-(D32-Pad2) -> /MAR/A4
- D33 pad 1: Net-(D33-Pad1) -> /MAR/~PROG
- D4 pad 2: /A register/BUS_4 -> /BUS_3
- D44 pad 2: /Clock/HLT -> Net-(D44-Pad2)
- D45 pad 2: /Control logic/MI -> Net-(D45-Pad2)
- D46 pad 2: /Control logic/RI -> Net-(D46-Pad2)
- D48 pad 2: Net-(D48-Pad2) -> /RAM/STK
- D49 pad 2: /Control logic/II -> Net-(D49-Pad2)
- D5 pad 2: /A register/BUS_3 -> /BUS_4
- D50 pad 2: /A register/AI -> Net-(D50-Pad2)
- D53 pad 2: /ALU/SU -> Net-(D53-Pad2)
- D54 pad 2: /B register/BI -> Net-(D54-Pad2)
- D55 pad 2: /Control logic/OI -> /Instruction register/HL
- D56 pad 2: /Control logic/CE -> Net-(D56-Pad2)
- D6 pad 2: /A register/BUS_2 -> /BUS_5
- D60 pad 2: /ALU/OR -> Net-(D60-Pad2)
- D61 pad 2: /ALU/AND -> Net-(D61-Pad2)
- D62 pad 2: /A register/SFT -> Net-(D62-Pad2)
- D63 pad 2: /A register/ROT -> Net-(D63-Pad2)
- D64 pad 2: /A register/RGT -> /C register/OUT_7
- D65 pad 2: /Control logic/STK -> /C register/OUT_6
- D66 pad 2: /Control logic/SI -> /C register/OUT_5
- D67 pad 2: /Control logic/SO -> /C register/OUT_4
- D68 pad 2: Net-(D68-Pad2) -> /C register/OUT_3
- D69 pad 2: Net-(D69-Pad2) -> /C register/OUT_2
- D7 pad 2: /A register/BUS_1 -> /BUS_6
- D70 pad 2: Net-(D70-Pad2) -> /C register/OUT_1
- D71 pad 2: Net-(D71-Pad2) -> /C register/OUT_0
- D8 pad 2: /A register/BUS_0 -> /BUS_7
- D80 pad 2: Net-(D80-Pad2) -> /IR_7
- D81 pad 2: Net-(D81-Pad2) -> /IR_6
- D82 pad 2: Net-(D82-Pad2) -> /IR_5
- D83 pad 2: Net-(D83-Pad2) -> /IR_4
- D84 pad 2: Net-(D84-Pad2) -> /IR_3
- D85 pad 2: Net-(D85-Pad2) -> /IR_2
- D86 pad 2: Net-(D86-Pad2) -> /IR_1
- D87 pad 2: Net-(D87-Pad2) -> /IR_0
- D88 pad 2: Net-(D88-Pad2) -> /A_7
- D89 pad 2: Net-(D89-Pad2) -> /A_6
- D9 pad 2: /A register/CLK -> Net-(D9-Pad2)
- D90 pad 2: Net-(D90-Pad2) -> /A_5
- D91 pad 2: Net-(D91-Pad2) -> /A_4
- D92 pad 2: /Control logic/IR_7 -> /A_3
- D93 pad 2: /Control logic/IR_6 -> /A_2
- D94 pad 2: /Control logic/IR_5 -> /A_1
- D95 pad 2: /Control logic/IR_4 -> /A_0
- D96 pad 2: /Control logic/IR_3 -> /Control logic/IRQ0
- D97 pad 2: /Control logic/IR_2 -> /Control logic/IRQ1
- D98 pad 2: /Control logic/IR_1 -> Net-(D98-Pad2)
- D99 pad 2: /Control logic/IR_0 -> Net-(D99-Pad2)
- J1 pad 2: GND -> (no net)
- J2 pad 2: (no net) -> GND
- R1 pad 1: /A register/BUS_7 -> VCC
- R1 pad 2: GND -> Net-(R1-Pad2)
- R10 pad 1: Net-(D2-Pad1) -> GND
- R10 pad 2: GND -> Net-(D19-Pad1)
- R11 pad 1: Net-(D3-Pad1) -> GND
- R11 pad 2: GND -> Net-(D20-Pad1)
- R12 pad 1: Net-(D4-Pad1) -> VCC
- R12 pad 2: GND -> /MAR/~PROG
- R13 pad 1: Net-(D5-Pad1) -> VCC
- R13 pad 2: GND -> Net-(D33-Pad2)
- R14 pad 1: Net-(D6-Pad1) -> VCC
- R14 pad 2: GND -> Net-(R14-Pad2)
- R15 pad 1: Net-(D7-Pad1) -> VCC
- R15 pad 2: GND -> Net-(R15-Pad2)
- R16 pad 1: Net-(D8-Pad1) -> Net-(R16-Pad1)
- R16 pad 2: GND -> Net-(C18-Pad1)
- R17 pad 2: Net-(R17-Pad2) -> Net-(R16-Pad1)
- R18 pad 2: Net-(R17-Pad2) -> GND
- R19 pad 1: VCC -> Net-(R19-Pad1)
- R19 pad 2: Net-(R19-Pad2) -> GND
- R2 pad 1: /A register/BUS_6 -> Net-(R2-Pad1)
- R2 pad 2: GND -> Net-(R1-Pad2)
- R20 pad 1: VCC -> Net-(R20-Pad1)
- R20 pad 2: Net-(C5-Pad1) -> GND
- R21 pad 1: VCC -> Net-(R21-Pad1)
- R21 pad 2: Net-(R21-Pad2) -> VCC
- R22 pad 1: VCC -> Net-(R22-Pad1)
- R22 pad 2: Net-(R22-Pad2) -> VCC
- R23 pad 1: Net-(D9-Pad1) -> Net-(D48-Pad1)
- R24 pad 1: Net-(D10-Pad1) -> Net-(D55-Pad1)
- R25 pad 1: Net-(D11-Pad1) -> VCC
- R25 pad 2: GND -> Net-(JP2-Pad1)
- R3 pad 1: /A register/BUS_5 -> VCC
- R3 pad 2: GND -> Net-(R3-Pad2)
- R33 pad 2: Net-(D19-Pad1) -> Net-(D96-Pad1)
- R34 pad 1: Net-(D20-Pad1) -> GND
- R34 pad 2: GND -> Net-(D97-Pad1)
- R36 pad 1: Net-(D22-Pad1) -> /PC Interface/CLR
- R4 pad 1: /A register/BUS_4 -> VCC
- R4 pad 2: GND -> Net-(C7-Pad1)
- R5 pad 1: /A register/BUS_3 -> Net-(D9-Pad2)
- R5 pad 2: GND -> VCC
- R6 pad 1: /A register/BUS_2 -> VCC
- R6 pad 2: GND -> Net-(D9-Pad1)
- R7 pad 1: /A register/BUS_1 -> /Clock/CLK_IN
- R8 pad 1: /A register/BUS_0 -> VCC
- R8 pad 2: GND -> Net-(R8-Pad2)
- R9 pad 1: Net-(D1-Pad1) -> Net-(D10-Pad1)
- RV1 pad 2: Net-(R18-Pad1) -> Net-(R2-Pad1)
- SW1 pad 2: Net-(R19-Pad2) -> GND
- SW2 pad 1: (no net) -> GND
- SW2 pad 2: (no net) -> Net-(R3-Pad2)
- SW3 pad 4: /MAR/PROG -> Net-(D9-Pad1)
- SW3 pad 6: Net-(D33-Pad1) -> Net-(R8-Pad2)
- SW4 pad 1: Net-(SW4-Pad1) -> GND
- SW4 pad 2: Net-(SW4-Pad2) -> /MAR/~PROG
- SW5 pad 1: (no net) -> GND
- SW5 pad 2: (no net) -> Net-(SW5-Pad2)
- SW5 pad 3: (no net) -> Net-(SW5-Pad3)
- SW5 pad 4: VCC -> Net-(SW5-Pad4)
- SW5 pad 6: Net-(R52-Pad1) -> Net-(SW5-Pad6)
- SW6 pad 1: Net-(R55-Pad1) -> VCC
- SW7 pad 2: Net-(SW7-Pad2) -> Net-(R21-Pad1)
- SW8 pad 1: Net-(SW8-Pad1) -> GND
- SW8 pad 2: Net-(SW8-Pad2) -> Net-(R22-Pad1)
- U1 pad 1: /PC Interface/MI -> /Control logic/MI
- U1 pad 10: /Control logic/HL -> /MAR/HL
- U1 pad 11: Net-(U1-Pad11) -> /RAM/RI
- U1 pad 12: /ALU/B_7 -> /Control logic/RI
- U1 pad 13: /ALU/SU -> /PC Interface/RI
- U1 pad 2: /Control logic/MI -> /PC Interface/MI
- U1 pad 4: /PC Interface/RI -> /MAR/STK
- U1 pad 5: /Control logic/RI -> /Control logic/STK
- U1 pad 6: /RAM/RI -> /RAM/STK
- U1 pad 9: /PC Interface/HL -> Net-(U1-Pad9)
- U10 pad 1: /A register/~CLR -> Net-(U10-Pad1)
- U10 pad 10: GND -> Net-(U10-Pad10)
- U10 pad 11: Net-(U10-Pad11) -> Net-(C15-Pad1)
- U10 pad 12: /ALU/B_4 -> /ALU/EI
- U10 pad 13: /A register/BUS_4 -> /CLK
- U10 pad 14: /A register/BUS_5 -> VCC
- U10 pad 2: /ALU/B_0 -> Net-(U10-Pad2)
- U10 pad 3: /A register/BUS_0 -> Net-(U10-Pad3)
- U10 pad 4: /A register/BUS_1 -> Net-(U10-Pad4)
- U10 pad 5: /ALU/B_1 -> Net-(U10-Pad5)
- U10 pad 6: /ALU/B_2 -> Net-(U10-Pad1)
- U10 pad 7: /A register/BUS_2 -> GND
- U10 pad 8: /A register/BUS_3 -> Net-(U10-Pad2)
- U10 pad 9: /ALU/B_3 -> Net-(U10-Pad9)
- U11 pad 1: Net-(U11-Pad1) -> GND
- U11 pad 10: Net-(U11-Pad10) -> /ALU/~FI
- U11 pad 11: Net-(U11-Pad11) -> (no net)
- U11 pad 12: /ALU/B_3 -> (no net)
- U11 pad 13: /A register/A_3 -> Net-(U10-Pad3)
- U11 pad 14: VCC -> Net-(U11-Pad14)
- U11 pad 2: Net-(U11-Pad2) -> GND
- U11 pad 3: Net-(U11-Pad3) -> /ALU/CF
- U11 pad 4: Net-(U11-Pad4) -> /ALU/ZF
- U11 pad 5: Net-(U11-Pad5) -> (no net)
- U11 pad 6: Net-(U11-Pad1) -> (no net)
- U11 pad 7: GND -> /CLK
- U11 pad 8: Net-(U11-Pad2) -> GND
- U11 pad 9: Net-(U11-Pad9) -> /ALU/~FI
- U12 pad 1: GND -> Net-(U10-Pad4)
- U12 pad 10: /ALU/~FI -> Net-(U10-Pad9)
- U12 pad 11: (no net) -> Net-(D27-Pad2)
- U12 pad 12: (no net) -> Net-(D28-Pad2)
- U12 pad 13: Net-(U11-Pad3) -> Net-(U10-Pad10)
- U12 pad 14: Net-(U12-Pad14) -> VCC
- U12 pad 2: GND -> Net-(D21-Pad2)
- U12 pad 3: /ALU/CF -> Net-(D22-Pad2)
- U12 pad 4: /ALU/ZF -> Net-(U10-Pad5)
- U12 pad 5: (no net) -> Net-(D23-Pad2)
- U12 pad 6: (no net) -> Net-(D24-Pad2)
- U12 pad 7: /A register/CLK -> GND
- U12 pad 8: GND -> Net-(D25-Pad2)
- U12 pad 9: /ALU/~FI -> Net-(D26-Pad2)
- U13 pad 1: Net-(U13-Pad1) -> VCC
- U13 pad 10: /ALU/OR -> GND
- U13 pad 11: Net-(U13-Pad11) -> /BUS_0
- U13 pad 12: Net-(U13-Pad12) -> /BUS_1
- U13 pad 13: Net-(U13-Pad12) -> /BUS_2
- U13 pad 14: VCC -> /BUS_3
- U13 pad 2: Net-(U13-Pad2) -> Net-(D21-Pad2)
- U13 pad 3: Net-(U13-Pad3) -> Net-(D22-Pad2)
- U13 pad 4: /ALU/AND -> Net-(D23-Pad2)
- U13 pad 5: /ALU/AND -> Net-(D24-Pad2)
- U13 pad 6: Net-(U13-Pad1) -> Net-(D25-Pad2)
- U13 pad 7: GND -> Net-(D26-Pad2)
- U13 pad 8: Net-(U13-Pad2) -> Net-(D27-Pad2)
- U13 pad 9: /ALU/OR -> Net-(D28-Pad2)
- U14 pad 1: Net-(U11-Pad4) -> Net-(U14-Pad1)
- U14 pad 10: Net-(U11-Pad9) -> Net-(U14-Pad10)
- U14 pad 11: Net-(D26-Pad2) -> Net-(U14-Pad11)
- U14 pad 12: Net-(D27-Pad2) -> /A_7
- U14 pad 13: Net-(U11-Pad10) -> Net-(U14-Pad13)
- U14 pad 14: VCC -> /A_6
- U14 pad 2: Net-(D20-Pad2) -> Net-(U14-Pad2)
- U14 pad 3: Net-(D21-Pad2) -> /A_5
- U14 pad 4: Net-(U11-Pad5) -> Net-(U14-Pad4)
- U14 pad 5: Net-(D22-Pad2) -> /A_4
- U14 pad 6: Net-(D23-Pad2) -> Net-(U14-Pad6)
- U14 pad 7: GND -> Net-(U14-Pad7)
- U14 pad 8: Net-(D24-Pad2) -> GND
- U14 pad 9: Net-(D25-Pad2) -> Net-(U11-Pad14)
- U15 pad 1: VCC -> Net-(U15-Pad1)
- U15 pad 10: GND -> Net-(U15-Pad10)
- U15 pad 11: /A register/BUS_0 -> Net-(U15-Pad11)
- U15 pad 12: /A register/BUS_1 -> /A_3
- U15 pad 13: /A register/BUS_2 -> Net-(U15-Pad13)
- U15 pad 14: /A register/BUS_3 -> /A_2
- U15 pad 15: /A register/BUS_4 -> Net-(U15-Pad15)
- U15 pad 16: /A register/BUS_5 -> VCC
- U15 pad 2: Net-(D20-Pad2) -> Net-(U15-Pad2)
- U15 pad 3: Net-(D21-Pad2) -> /A_1
- U15 pad 4: Net-(D22-Pad2) -> Net-(U15-Pad4)
- U15 pad 5: Net-(D23-Pad2) -> /A_0
- U15 pad 6: Net-(D24-Pad2) -> Net-(U15-Pad6)
- U15 pad 7: Net-(D25-Pad2) -> Net-(U15-Pad7)
- U15 pad 8: Net-(D26-Pad2) -> GND
- U15 pad 9: Net-(D27-Pad2) -> Net-(U14-Pad7)
- U16 pad 11: Net-(U1-Pad11) -> Net-(U14-Pad4)
- U16 pad 12: /A register/A_7 -> Net-(D23-Pad2)
- U16 pad 14: /A register/A_6 -> Net-(U14-Pad1)
- U16 pad 15: Net-(U16-Pad15) -> GND
- U16 pad 2: Net-(U16-Pad2) -> Net-(U14-Pad10)
- U16 pad 3: /A register/A_5 -> Net-(U16-Pad3)
- U16 pad 4: Net-(U16-Pad4) -> Net-(D21-Pad2)
- U16 pad 5: /A register/A_4 -> Net-(U14-Pad13)
- U16 pad 7: Net-(U16-Pad7) -> Net-(D22-Pad2)
- U16 pad 9: Net-(U12-Pad14) -> Net-(D24-Pad2)
- U17 pad 1: Net-(U17-Pad1) -> Net-(U16-Pad1)
- U17 pad 11: Net-(U17-Pad11) -> Net-(U15-Pad4)
- U17 pad 12: /A register/A_3 -> Net-(D27-Pad2)
- U17 pad 14: /A register/A_2 -> Net-(U15-Pad1)
- U17 pad 15: Net-(U17-Pad15) -> GND
- U17 pad 2: Net-(U17-Pad2) -> Net-(U15-Pad10)
- U17 pad 3: /A register/A_1 -> Net-(U17-Pad3)
- U17 pad 4: Net-(U17-Pad4) -> Net-(D25-Pad2)
- U17 pad 5: /A register/A_0 -> Net-(U15-Pad13)
- U17 pad 7: /ALU/SU -> Net-(D26-Pad2)
- U17 pad 9: Net-(U16-Pad7) -> Net-(D28-Pad2)
- U18 pad 1: Net-(U13-Pad3) -> /~CLR
- U18 pad 10: Net-(U18-Pad10) -> GND
- U18 pad 11: Net-(U16-Pad4) -> Net-(C15-Pad1)
- U18 pad 12: Net-(D22-Pad2) -> Net-(U18-Pad12)
- U18 pad 13: Net-(U18-Pad13) -> /BUS_4
- U18 pad 14: Net-(U16-Pad1) -> /BUS_5
- U18 pad 15: GND -> Net-(U18-Pad15)
- U18 pad 16: VCC -> Net-(U18-Pad16)
- U18 pad 2: Net-(U16-Pad10) -> Net-(U18-Pad2)
- U18 pad 3: Net-(U18-Pad3) -> /BUS_0
- U18 pad 4: Net-(D20-Pad2) -> /BUS_1
- U18 pad 5: Net-(U16-Pad13) -> Net-(U18-Pad5)
- U18 pad 7: Net-(D21-Pad2) -> /BUS_2
- U18 pad 8: GND -> /BUS_3
- U18 pad 9: Net-(D23-Pad2) -> Net-(U18-Pad9)
- U19 pad 1: Net-(U13-Pad3) -> /ALU/OR
- U19 pad 11: Net-(U17-Pad4) -> Net-(U19-Pad11)
- U19 pad 12: Net-(D26-Pad2) -> Net-(U16-Pad13)
- U19 pad 14: Net-(U17-Pad1) -> Net-(U19-Pad14)
- U19 pad 2: Net-(U17-Pad10) -> Net-(U19-Pad2)
- U19 pad 4: Net-(D24-Pad2) -> Net-(U16-Pad3)
- U19 pad 5: Net-(U17-Pad13) -> Net-(U19-Pad5)
- U19 pad 7: Net-(D25-Pad2) -> Net-(U16-Pad6)
- U19 pad 9: Net-(D27-Pad2) -> Net-(U16-Pad10)
- U2 pad 1: Net-(U2-Pad1) -> /Control logic/HL
- U2 pad 10: VCC -> /Clock/CLK_IN
- U2 pad 11: VCC -> Net-(U16-Pad1)
- U2 pad 12: (no net) -> /ALU/AND
- U2 pad 13: Net-(U2-Pad13) -> /ALU/OR
- U2 pad 2: VCC -> /PC Interface/HL
- U2 pad 3: VCC -> Net-(U1-Pad9)
- U2 pad 4: VCC -> Net-(U2-Pad4)
- U2 pad 6: VCC -> Net-(U2-Pad6)
- U2 pad 7: VCC -> GND
- U2 pad 8: Net-(U2-Pad1) -> /CLK
- U2 pad 9: (no net) -> Net-(U2-Pad9)
- U20 pad 1: /ALU/OR -> Net-(U18-Pad19)
- U20 pad 11: Net-(U20-Pad11) -> Net-(U14-Pad6)
- U20 pad 12: Net-(U18-Pad13) -> Net-(U18-Pad12)
- U20 pad 13: Net-(U20-Pad13) -> Net-(U20-Pad10)
- U20 pad 14: Net-(U20-Pad14) -> VCC
- U20 pad 2: Net-(U20-Pad2) -> Net-(U20-Pad10)
- U20 pad 3: Net-(U20-Pad3) -> Net-(U14-Pad11)
- U20 pad 4: Net-(U18-Pad3) -> Net-(U18-Pad16)
- U20 pad 5: Net-(U20-Pad5) -> Net-(U20-Pad10)
- U20 pad 6: Net-(U20-Pad6) -> Net-(U14-Pad15)
- U20 pad 7: Net-(U18-Pad6) -> GND
- U20 pad 8: GND -> Net-(U14-Pad2)
- U20 pad 9: Net-(U18-Pad10) -> Net-(U18-Pad15)
- U21 pad 1: /ALU/B_6 -> Net-(U18-Pad9)
- U21 pad 10: /ALU/SU -> Net-(U20-Pad10)
- U21 pad 11: Net-(U17-Pad11) -> Net-(U15-Pad6)
- U21 pad 12: /ALU/B_3 -> Net-(U18-Pad2)
- U21 pad 13: /ALU/SU -> Net-(U20-Pad10)
- U21 pad 2: /ALU/SU -> Net-(U20-Pad10)
- U21 pad 3: Net-(U16-Pad15) -> Net-(U15-Pad11)
- U21 pad 4: /ALU/B_5 -> Net-(U18-Pad6)
- U21 pad 5: /ALU/SU -> Net-(U20-Pad10)
- U21 pad 6: Net-(U16-Pad2) -> Net-(U15-Pad15)
- U21 pad 8: Net-(U16-Pad6) -> Net-(U15-Pad2)
- U21 pad 9: /ALU/B_4 -> Net-(U18-Pad5)
- U22 pad 1: /ALU/B_2 -> /ALU/OR
- U22 pad 10: /ALU/SU -> Net-(U22-Pad10)
- U22 pad 11: (no net) -> Net-(U22-Pad11)
- U22 pad 12: (no net) -> Net-(U17-Pad13)
- U22 pad 13: (no net) -> Net-(U22-Pad13)
- U22 pad 14: VCC -> Net-(U22-Pad14)
- U22 pad 2: /ALU/SU -> Net-(U22-Pad2)
- U22 pad 3: Net-(U17-Pad15) -> Net-(U22-Pad3)
- U22 pad 4: /ALU/B_1 -> Net-(U17-Pad3)
- U22 pad 5: /ALU/SU -> Net-(U22-Pad5)
- U22 pad 6: Net-(U17-Pad2) -> Net-(U22-Pad6)
- U22 pad 7: GND -> Net-(U17-Pad6)
- U22 pad 8: Net-(U17-Pad6) -> GND
- U22 pad 9: /ALU/B_0 -> Net-(U17-Pad10)
- U23 pad 1: /ALU/OR -> /ALU/NOT
- U23 pad 10: Net-(U23-Pad10) -> (no net)
- U23 pad 11: Net-(U23-Pad11) -> (no net)
- U23 pad 12: Net-(U19-Pad13) -> (no net)
- U23 pad 13: Net-(U23-Pad13) -> (no net)
- U23 pad 14: Net-(U23-Pad14) -> VCC
- U23 pad 2: Net-(U11-Pad11) -> Net-(U20-Pad10)
- U23 pad 3: Net-(U23-Pad3) -> Net-(U15-Pad7)
- U23 pad 4: Net-(U19-Pad3) -> Net-(U23-Pad4)
- U23 pad 5: Net-(U23-Pad5) -> Net-(JP1-Pad1)
- U23 pad 7: Net-(U19-Pad6) -> GND
- U23 pad 8: GND -> (no net)
- U23 pad 9: Net-(U19-Pad10) -> (no net)
- U24 pad 1: /A register/A_3 -> /A_2
- U24 pad 10: /ALU/B_6 -> Net-(U18-Pad2)
- U24 pad 11: Net-(U20-Pad13) -> Net-(U22-Pad3)
- U24 pad 12: /A register/A_5 -> /A_3
- U24 pad 13: /ALU/B_5 -> Net-(U18-Pad9)
- U24 pad 2: /ALU/B_3 -> Net-(U18-Pad6)
- U24 pad 3: Net-(U23-Pad3) -> Net-(U22-Pad6)
- U24 pad 4: /A register/A_7 -> /A_1
- U24 pad 5: /ALU/B_7 -> Net-(U18-Pad5)
- U24 pad 6: Net-(U20-Pad3) -> Net-(U22-Pad13)
- U24 pad 8: Net-(U20-Pad6) -> Net-(U22-Pad10)
- U24 pad 9: /A register/A_6 -> /A_0
- U25 pad 1: /ALU/B_2 -> Net-(U18-Pad9)
- U25 pad 10: /A register/A_0 -> /A_1
- U25 pad 11: Net-(U20-Pad2) -> Net-(U22-Pad11)
- U25 pad 12: /ALU/B_7 -> Net-(U18-Pad2)
- U25 pad 13: /A register/A_7 -> /A_0
- U25 pad 2: /A register/A_2 -> /A_3
- U25 pad 3: Net-(U23-Pad5) -> Net-(U22-Pad2)
- U25 pad 4: /ALU/B_1 -> Net-(U18-Pad6)
- U25 pad 5: /A register/A_1 -> /A_2
- U25 pad 6: Net-(U23-Pad14) -> Net-(U22-Pad5)
- U25 pad 8: Net-(U23-Pad11) -> Net-(U22-Pad14)
- U25 pad 9: /ALU/B_0 -> Net-(U18-Pad5)
- U26 pad 1: /ALU/B_6 -> Net-(U18-Pad19)
- U26 pad 10: /A register/A_4 -> /A_5
- U26 pad 11: Net-(U26-Pad11) -> Net-(U19-Pad11)
- U26 pad 12: /A register/CLK -> Net-(U18-Pad12)
- U26 pad 13: /MAR/MI -> /A_4
- U26 pad 2: /A register/A_6 -> /A_7
- U26 pad 3: Net-(U20-Pad5) -> Net-(U19-Pad2)
- U26 pad 4: /ALU/B_5 -> Net-(U18-Pad16)
- U26 pad 5: /A register/A_5 -> /A_6
- U26 pad 6: Net-(U20-Pad14) -> Net-(U19-Pad5)
- U26 pad 8: Net-(U20-Pad11) -> Net-(U19-Pad14)
- U26 pad 9: /ALU/B_4 -> Net-(U18-Pad15)
- U27 pad 1: /A register/A_4 -> /ALU/SUB
- U27 pad 10: (no net) -> Net-(U18-Pad16)
- U27 pad 11: (no net) -> Net-(U19-Pad13)
- U27 pad 12: (no net) -> /A_5
- U27 pad 13: (no net) -> Net-(U18-Pad15)
- U27 pad 2: /ALU/B_4 -> /ALU/NOT
- U27 pad 4: (no net) -> /A_7
- U27 pad 5: (no net) -> Net-(U18-Pad19)
- U27 pad 6: (no net) -> Net-(U19-Pad3)
- U27 pad 8: (no net) -> Net-(U19-Pad6)
- U27 pad 9: (no net) -> /A_6
- U28 pad 1: /MAR/PROG -> /A_4
- U28 pad 10: Net-(U28-Pad10) -> (no net)
- U28 pad 11: Net-(SW4-Pad1) -> (no net)
- U28 pad 12: /MAR/A1 -> (no net)
- U28 pad 13: Net-(U28-Pad13) -> (no net)
- U28 pad 14: Net-(SW4-Pad2) -> VCC
- U28 pad 2: Net-(SW4-Pad13) -> Net-(U18-Pad12)
- U28 pad 3: Net-(U28-Pad3) -> Net-(U19-Pad10)
- U28 pad 4: /MAR/A3 -> /A register/SFT
- U28 pad 5: Net-(SW4-Pad14) -> /A register/ROT
- U28 pad 7: /MAR/A2 -> GND
- U28 pad 8: GND -> (no net)
- U28 pad 9: /MAR/A0 -> (no net)
- U29 pad 1: /MAR/PROG -> /MAR/~PROG
- U29 pad 11: Net-(SW4-Pad5) -> Net-(SW5-Pad2)
- U29 pad 12: /MAR/A5 -> /MAR/A1
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Routing:
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Other:
- board size 318.8 x 180.3 mm -> 297.2 x 180.3 mm
- board text added: "*"
- board text added: "+"
- board text added: "-"
- board text added: "0"
- board text added: "1"
- board text added: "2"
- board text added: "3"
- board text added: "4"
- board text added: "5"
- board text added: "6"
- board text added: "7"
- board text added: "AUX 5V DC"
- board text added: "BO"
- board text added: "C"
- board text added: "CI"
- board text added: "CLK"
- board text added: "CLR"
- board text added: "Control Words"
- board text added: "D"
- board text added: "DI"
- board text added: "DO"
- board text added: "Designed by"
- board text added: "EI"
- board text added: "EN0"
- board text added: "EN1"
- board text added: "EXT Interface"
- board text added: "HL"
- board text added: "IRQ0"
- board text added: "IRQ1"
- board text added: "NOT"
- board text added: "PE"
- board text added: "PI"
- board text added: "PO"
- board text added: "Programming Interface"
- board text added: "SD"
- board text added: "SHF"
- board text added: "SIG0"
- board text added: "SIG1"
- board text added: "STK"
- board text added: "SUB"
- board text added: "Step counter"
- board text added: "U0"
- board text added: "U1"
- board text added: "v2.0b"
- board text added: "| 7 - 0 |"
- board text removed: "CE"
- board text removed: "Control words"
- board text removed: "FI"
- board text removed: "J"
- board text removed: "PC Interface"
- board text removed: "RGT"
- board text removed: "SFT"
- board text removed: "SP"
- board text removed: "Step Counter"
- board text removed: "v0.1a"

Commit message: resistor label update
Parts:
- RN1: value 220 -> 1K
- RN10: value 10K -> 1K
- RN2: value 220 -> 470
