File: MK1_CPU/8bit-computer/8bit-computer.kicad_pcb (KiCad board)
At the start: 2 copper layers, 297.2 x 180.3 mm, 388 parts, among them J1 USB_B-8bit-computer-rescue, J2 Barrel_Jack_Switch, J3 EXT-Bus, J4 EXT-Signal, J5 EXT-Power, SW1 Multiplier, SW10 Reset, SW2 Pulse, SW3 Manual, SW4 Prog, SW5 Address, SW6 Mode, SW7 Write, SW8 Show, SW9 Data, U1 74HCT32, U10 74HCT08, U11 74HCT173, U12 74HCT02, U13 74HCT245, U14 74HCT283, U15 74HCT283, U16 74HCT157, U17 74HCT157, U18 74HCT273, U19 74HCT157, U2 74HCT32, U20 74HCT86, U21 74HCT86, U22 74HCT157, U23 74HCT86, U24 74HCT32, U25 74HCT08, U26 74HCT08, U27 74HCT32, U28 74HCT32, U29 74LS157, U3 NE555, U30 74LS157, U31 74HCT273, U32 74HCT08, U33 NE555, U34 74HCT273, U35 74HCT107, U36 28C64, U37 7SEGMENT_CC, U38 74HCT139, U39 7SEGMENT_CC, U4 74HCT04, U40 7SEGMENT_CC, U41 7SEGMENT_CC, U42 74HCT245, U43 74HCT161, U44 74HCT161, U45 74HCT157, U46 74HCT00, U47 CY62256, U48 74HCT245, U49 74HCT245, U5 74HCT08, U50 74LS157, U51 74LS157, U52 74HCT245, U53 74HCT193, U54 74HCT193, U55 74HCT00, U56 74HCT245, U57 74HCT273, U58 74HCT08, U59 74HCT245, U6 NE555, U60 74HCT245, U61 74HCT273, U62 74HCT273, U63 74HCT04, U64 74HCT08, U65 74HCT157, U66 74HCT157, U67 74HCT245, U68 74HCT273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

Commit message: revision 2.0d
Parts:
- removed the C34 at (90.2, 137.2)
- removed the C35 at (93.3, 137.1)
- removed the D72 at (72.4, 182.9)
- removed the D73 at (78.7, 182.9)
- removed the D74 at (85.1, 182.9)
- removed the D75 at (91.4, 182.9)
- removed the D76 at (97.8, 182.9)
- removed the D77 at (104.1, 182.9)
- removed the D78 at (110.5, 182.9)
- removed the D79 at (116.8, 182.9)
- removed the J4 at (71.1, 14.7)
- removed J5: EXT-Power, Connector_PinHeader_2.54mm:PinHeader_1x02_P2.54mm_Vertical
- removed the JP1 at (218.4, 143.5)
- removed JP2: 6-STAGES, Jumper:SolderJumper-2_P1.3mm_Bridged_RoundedPad1.0x1.5mm
- removed the R25 at (158.4, 185.2)
- removed the RN11 at (115.6, 177.8)
- removed S0: OSHW-Logo_11.4x12mm_SilkScreen, Symbol:OSHW-Logo_11.4x12mm_SilkScreen
- removed S1: LOGO, Symbol:parrot
- removed S2: Symbol_Barrel_Polarity, Symbol:Symbol_Barrel_Polarity
- removed the TP28 at (81.7, 146.1)
- removed the U27 at (303.5, 53.3)
- removed the U62 at (90.2, 143.5)
- removed the U63 at (139.7, 177.8)
- removed the U74 at (184.2, 185.4)
- removed U84: 74HCT04, Package_DIP:DIP-14_W7.62mm
- added C27: 0.01µf, Capacitor_THT:C_Disc_D4.3mm_W1.9mm_P5.00mm, F.Cu at (71.1, 102.2)
- added C39: 0.01µF, Capacitor_THT:C_Disc_D4.3mm_W1.9mm_P5.00mm, F.Cu at (141.6, 178.5)
- added C44: 0.01µf, Capacitor_THT:C_Disc_D4.3mm_W1.9mm_P5.00mm, F.Cu at (71.1, 106.7)
- added G0: LOGO, Symbol:parrot, F.Cu at (92.7, 147.3)
- added G1: Symbol_Barrel_Polarity, Symbol:Symbol_Barrel_Polarity, F.Cu at (170.8, 18.4)
- added G2: KiCad-Logo2_8mm_SilkScreen, Symbol:KiCad-Logo2_8mm_SilkScreen, B.Cu at (29.2, 177.8)
- added G3: OSHW-Logo_11.4x12mm_SilkScreen, Symbol:OSHW-Logo_11.4x12mm_SilkScreen, B.Cu at (54.6, 179.1)
- added R27: 1K, Resistor_THT:R_Axial_DIN0207_L6.3mm_D2.5mm_P7.62mm_Horizontal, F.Cu at (121.9, 15.2)
- added R28: 1K, Resistor_THT:R_Axial_DIN0207_L6.3mm_D2.5mm_P7.62mm_Horizontal, F.Cu at (128.3, 15.2)
- added R30: 10K, Resistor_THT:R_Axial_DIN0207_L6.3mm_D2.5mm_P7.62mm_Horizontal, F.Cu at (177.8, 185.4)
- added R31: 10K, Resistor_THT:R_Axial_DIN0207_L6.3mm_D2.5mm_P7.62mm_Horizontal, F.Cu at (171.4, 185.4)
- added R32: 10K, Resistor_THT:R_Axial_DIN0207_L6.3mm_D2.5mm_P7.62mm_Horizontal, F.Cu at (124.5, 177.8)
- added U12: 74HCT32, Package_DIP:DIP-14_W7.62mm, F.Cu at (295.9, 59.7)
- C17: renamed from C16; value * -> 0.01
- C24: renamed from C23; value * -> 0.01µf
- J4: renamed from J3; value EXT-Bus -> EXT-CONN; footprint Connector_PinHeader_2.54mm:PinHeader_1x08_P2.54mm_Vertical -> Connector_PinHeader_2.54mm:PinHeader_2x09_P2.54mm_Vertical
- JP1: renamed from JP3; value Arduino_VIN -> POWER
- RN1: value 1K -> 10K
- U60: value 74HCT245 -> 74HCT04; footprint Package_DIP:DIP-20_W7.62mm -> Package_DIP:DIP-14_W7.62mm
- moved MH0 292.1 mm to (14.0, 12.7)
- moved MH2 292.1 mm to (306.1, 188.0)
- moved MH1 175.3 mm to (14.0, 188.0)
- moved MH3 175.3 mm to (306.1, 12.7)
- moved U55 96.1 mm to (184.2, 185.4)
- moved TP6 74.0 mm to (252.7, 91.4)
- moved U28 72.0 mm to (295.9, 39.4), turned to 0 degrees
- moved D102 63.5 mm to (218.4, 151.1)
- moved U70 59.8 mm to (71.1, 40.6), turned to 90 degrees
- moved U27 57.1 mm to (250.2, 94.0), turned to 270 degrees
- moved TP35 56.4 mm to (71.1, 36.8)
- moved U69 55.0 mm to (115.6, 33.0)
- moved U71 49.8 mm to (115.6, 15.2), turned to 270 degrees
- moved C5 45.2 mm to (116.8, 102.2), turned to 180 degrees
- moved TP2 38.4 mm to (81.3, 135.9)
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- renumbered C43 to C1, C9 to C10, C10 to C11, C11 to C12, C12 to C13, C13 to C14, C14 to C15, C15 to C16, C17 to C18, C18 to C19, C1 to C2, C19 to C20, C20 to C21, C21 to C22, C22 to C23, C24 to C25, C25 to C26, C26 to C28, C27 to C29, C2 to C3, C28 to C30, C29 to C31, C31 to C32, C30 to C33, C32 to C34, C33 to C35, C3 to C4, C39 to C40, C40 to C41, C41 to C42, C42 to C43, C4 to C5, C5 to C6, C6 to C7, C7 to C8, C8 to C9, D113 to D100, D114 to D101, D115 to D102, D116 to D103, D117 to D104, D118 to D105, D119 to D106, D120 to D107, D121 to D108, D122 to D109, D123 to D110, D124 to D111, D125 to D112, D126 to D113, D127 to D114, D128 to D115, D129 to D116, D130 to D117, D131 to D118, D132 to D119, D133 to D120, D134 to D121, D135 to D122, D136 to D123, D137 to D124, D138 to D125, D139 to D126, D140 to D127, D141 to D128, D142 to D129, D143 to D130, D144 to D131, D145 to D132, D146 to D133, D147 to D134, D80 to D72, D81 to D73, D82 to D74, D83 to D75, D84 to D76, D85 to D77, D86 to D78, D87 to D79, D88 to D80, D89 to D81, D90 to D82, D91 to D83, D92 to D84, D93 to D85, D94 to D86, D95 to D87, D96 to D88, D97 to D89, D98 to D90, D99 to D91, D100 to D92, D105 to D93, D106 to D94, D107 to D95, D109 to D96, D110 to D97, D111 to D98, D112 to D99, R33 to R25, R34 to R26, R36 to R29, RN12 to RN11, RN21 to RN12, TP29 to TP28, TP30 to TP29, TP31 to TP30, TP32 to TP31, TP33 to TP32, TP34 to TP33, TP35 to TP34, TP36 to TP35, TP37 to TP36, TP38 to TP37, TP39 to TP38, TP40 to TP39, TP41 to TP40, TP42 to TP41, U12 to U13, U13 to U14, U14 to U15, U15 to U16, U16 to U17, U17 to U18, U18 to U19, U19 to U20, U20 to U21, U21 to U22, U22 to U23, U23 to U24, U24 to U25, U25 to U26, U26 to U27, U32 to U29, U29 to U30, U30 to U31, U31 to U32, U65 to U62, U66 to U63, U67 to U65, U68 to U66, U69 to U67, U70 to U68, U71 to U69, U72 to U70, U73 to U71, U75 to U72, U77 to U73, U78 to U74, U79 to U75, U80 to U76, U81 to U77, U82 to U78, U83 to U79, U85 to U80, U86 to U81
Connections:
- C17 pad 1: Net-(C16-Pad1) (its old number) -> Net-(C17-Pad1)
- C21 pad 1: Net-(C20-Pad1) (its old number) -> Net-(C21-Pad1)
- C31 pad 1: Net-(C29-Pad1) -> Net-(C31-Pad1)
- C32 pad 1: Net-(C31-Pad1) -> Net-(C32-Pad1)
- C33 pad 1: Net-(C30-Pad1) -> Net-(C33-Pad1)
- C43 pad 1: Net-(C42-Pad1) -> Net-(C43-Pad1)
- D102 pad 2: Net-(D115-Pad2) -> Net-(D102-Pad2)
- D119 pad 2: Net-(D132-Pad2) -> Net-(D119-Pad2)
- D55 pad 2: /Instruction register/HL -> /RAM/HL
- D93 pad 2: /Clock/HLT -> /Control logic/HLT
- D98 pad 2: Net-(D111-Pad2) -> Net-(D98-Pad2)
- J4 pad 1: Net-(J3-Pad1) -> Net-(J4-Pad1)
- J4 pad 2: Net-(J3-Pad2) -> Net-(J4-Pad2)
- J4 pad 3: Net-(J3-Pad3) -> Net-(J4-Pad3)
- J4 pad 4: Net-(J3-Pad4) -> Net-(J4-Pad4)
- J4 pad 5: Net-(J3-Pad5) -> /Control logic/E0
- J4 pad 6: Net-(J3-Pad6) -> Net-(J4-Pad6)
- J4 pad 7: Net-(J3-Pad7) -> /Control logic/E1
- J4 pad 8: Net-(J3-Pad8) -> Net-(J4-Pad8)
- R13 pad 1: VCC -> Net-(D33-Pad2)
- R13 pad 2: Net-(D33-Pad2) -> VCC
- RN13 pad 9: Net-(JP1-Pad1) -> Net-(C39-Pad1)
- RN15 pad 5: /Clock/HLT -> /Control logic/HLT
- RN16 pad 5: Net-(D115-Pad2) -> (no net)
- RN16 pad 6: Net-(D111-Pad2) -> Net-(D98-Pad2)
- SW5 pad 1: GND -> Net-(SW5-Pad1)
- SW5 pad 12: GND -> Net-(R14-Pad2)
- SW5 pad 20: Net-(R14-Pad2) -> GND
- SW5 pad 9: Net-(SW5-Pad9) -> GND
- TP15 pad 1: Net-(C16-Pad1) (its old number) -> Net-(C17-Pad1)
- TP16 pad 1: Net-(C20-Pad1) (its old number) -> Net-(C21-Pad1)
- TP23 pad 1: Net-(C31-Pad1) -> Net-(C32-Pad1)
- TP24 pad 1: Net-(C29-Pad1) -> Net-(C31-Pad1)
- TP25 pad 1: Net-(C30-Pad1) -> Net-(C33-Pad1)
- TP28 pad 1: Net-(TP29-Pad1) -> Net-(TP28-Pad1)
- TP41 pad 1: Net-(C42-Pad1) -> Net-(C43-Pad1)
- U1 pad 11: /RAM/RI -> /Clock/HLT
- U1 pad 12: /Control logic/RI -> /Control logic/HLT
- U1 pad 13: /PC Interface/RI -> /PC Interface/CU_DIS
- U1 pad 8: /Instruction register/HL -> /RAM/HL
- U17 pad 1: Net-(U16-Pad1) (its old number) -> Net-(U12-Pad3)
- U18 pad 1: Net-(U16-Pad1) (its old number) -> Net-(U12-Pad3)
- U19 pad 12: Net-(U18-Pad12) -> Net-(U19-Pad12)
- U19 pad 15: Net-(U18-Pad15) -> Net-(U19-Pad15)
- U19 pad 16: Net-(U18-Pad16) -> Net-(U19-Pad16)
- U19 pad 19: Net-(U18-Pad19) -> Net-(U19-Pad19)
- U19 pad 2: Net-(U18-Pad2) -> Net-(U12-Pad13)
- U19 pad 5: Net-(U18-Pad5) -> Net-(U12-Pad10)
- U19 pad 6: Net-(U18-Pad6) (its old number) -> Net-(U12-Pad5)
- U19 pad 9: Net-(U18-Pad9) -> Net-(U19-Pad9)
- U2 pad 1: /Control logic/HL -> /Control logic/RI
- U2 pad 10: /Clock/CLK_IN -> Net-(U2-Pad10)
- U2 pad 11: Net-(U16-Pad1) (its old number) -> /CLK
- U2 pad 12: /ALU/AND -> Net-(U2-Pad12)
- U2 pad 13: /ALU/OR -> /Clock/CLK_IN
- U2 pad 2: /PC Interface/HL -> /PC Interface/RI
- U2 pad 3: Net-(U1-Pad9) -> /RAM/RI
- U2 pad 4: Net-(U2-Pad4) -> /Control logic/HL
- U2 pad 5: Net-(U2-Pad5) -> /PC Interface/HL
- U2 pad 6: Net-(U2-Pad6) -> Net-(U1-Pad9)
- U2 pad 8: /CLK -> Net-(U2-Pad8)
- U20 pad 10: Net-(U19-Pad10) -> Net-(U20-Pad10)
- U20 pad 13: Net-(U19-Pad13) -> Net-(U20-Pad13)
- U20 pad 3: Net-(U19-Pad3) -> Net-(U20-Pad3)
- U20 pad 6: Net-(U19-Pad6) -> Net-(U20-Pad6)
- U21 pad 1: Net-(U18-Pad19) -> Net-(U19-Pad19)
- U21 pad 10: Net-(U20-Pad10) -> Net-(U21-Pad10)
- U21 pad 12: Net-(U18-Pad12) -> Net-(U19-Pad12)
- U21 pad 13: Net-(U20-Pad10) -> Net-(U21-Pad10)
- U21 pad 2: Net-(U20-Pad10) -> Net-(U21-Pad10)
- U21 pad 4: Net-(U18-Pad16) -> Net-(U19-Pad16)
- U21 pad 5: Net-(U20-Pad10) -> Net-(U21-Pad10)
- U21 pad 9: Net-(U18-Pad15) -> Net-(U19-Pad15)
- U22 pad 1: Net-(U18-Pad9) -> Net-(U19-Pad9)
- U22 pad 10: Net-(U20-Pad10) -> Net-(U21-Pad10)
- U22 pad 12: Net-(U18-Pad2) -> Net-(U12-Pad13)
- U22 pad 13: Net-(U20-Pad10) -> Net-(U21-Pad10)
- U22 pad 2: Net-(U20-Pad10) -> Net-(U21-Pad10)
- U22 pad 4: Net-(U18-Pad6) (its old number) -> Net-(U12-Pad5)
- U22 pad 5: Net-(U20-Pad10) -> Net-(U21-Pad10)
- U22 pad 9: Net-(U18-Pad5) -> Net-(U12-Pad10)
- U23 pad 10: Net-(U22-Pad10) -> Net-(U12-Pad11)
- U23 pad 13: Net-(U22-Pad13) -> Net-(U12-Pad8)
- U23 pad 3: Net-(U22-Pad3) -> Net-(U23-Pad3)
- U23 pad 6: Net-(U22-Pad6) -> Net-(U12-Pad6)
- U24 pad 2: Net-(U20-Pad10) -> Net-(U21-Pad10)
- U24 pad 4: Net-(U23-Pad4) -> Net-(C39-Pad1)
- U24 pad 5: Net-(JP1-Pad1) -> /~CLR
- U25 pad 1: /A_2 -> /A_3
- U25 pad 10: Net-(U18-Pad2) -> Net-(U19-Pad19)
- U25 pad 11: Net-(U22-Pad3) -> Net-(U20-Pad6)
- U25 pad 12: /A_3 -> /A_6
- U25 pad 13: Net-(U18-Pad9) -> Net-(U19-Pad16)
- U25 pad 2: Net-(U18-Pad6) (its old number) -> Net-(U19-Pad9)
- U25 pad 3: Net-(U22-Pad6) -> Net-(U23-Pad3)
- U25 pad 4: /A_1 -> /ALU/SUB
- U25 pad 5: Net-(U18-Pad5) -> /ALU/NOT
- U25 pad 6: Net-(U22-Pad13) -> Net-(U21-Pad10)
- U25 pad 8: Net-(U22-Pad10) -> Net-(U20-Pad3)
- U25 pad 9: /A_0 -> /A_7
- U26 pad 1: Net-(U18-Pad9) -> Net-(U19-Pad9)
- U26 pad 12: Net-(U18-Pad2) -> Net-(U12-Pad13)
- U26 pad 4: Net-(U18-Pad6) (its old number) -> Net-(U12-Pad5)
- U26 pad 9: Net-(U18-Pad5) -> Net-(U12-Pad10)
- U27 pad 1: Net-(U18-Pad19) -> Net-(U19-Pad19)
- U27 pad 12: Net-(U18-Pad12) -> Net-(U19-Pad12)
- U27 pad 4: Net-(U18-Pad16) -> Net-(U19-Pad16)
- U27 pad 9: Net-(U18-Pad15) -> Net-(U19-Pad15)
- U28 pad 1: /A_4 -> /A_5
- U28 pad 10: (no net) -> /A register/ROT
- U28 pad 2: Net-(U18-Pad12) -> Net-(U19-Pad15)
- U28 pad 3: Net-(U19-Pad10) -> Net-(U20-Pad13)
- U28 pad 4: /A register/SFT -> /A_4
- U28 pad 5: /A register/ROT -> Net-(U19-Pad12)
- U28 pad 6: Net-(U28-Pad6) -> Net-(U20-Pad10)
- U28 pad 8: (no net) -> Net-(U28-Pad8)
- U28 pad 9: (no net) -> /A register/SFT
- U29 pad 1: /CLK -> Net-(R15-Pad2)
- U29 pad 10: /CLK -> /MAR/MI
- U29 pad 11: Net-(C29-Pad1) -> Net-(C21-Pad1)
- U29 pad 12: /Control logic/SD -> /Control logic/OI
- U29 pad 2: /MAR/MI -> Net-(U29-Pad2)
- U29 pad 3: Net-(C16-Pad1) (its old number) -> /MAR/STK
- U29 pad 4: /Control logic/OI -> Net-(R14-Pad2)
- U29 pad 5: /CLK -> Net-(U29-Pad2)
- U29 pad 6: Net-(C20-Pad1) (its old number) -> /MAR/HL
- U29 pad 8: Net-(C31-Pad1) -> Net-(C17-Pad1)
- U29 pad 9: /Control logic/SU -> /CLK
- U31 pad 2: Net-(SW5-Pad9) -> Net-(SW5-Pad1)
- U32 pad 11: Net-(C16-Pad1) (its old number) -> Net-(C17-Pad1)
- U34 pad 11: Net-(C20-Pad1) (its old number) -> Net-(C21-Pad1)
- U4 pad 10: Net-(TP21-Pad1) -> Net-(U4-Pad10)
- U4 pad 11: Net-(U4-Pad11) -> /MAR/~PROG
- U4 pad 12: Net-(U4-Pad12) -> Net-(TP21-Pad1)
- U4 pad 13: Net-(A1-Pad16) -> Net-(U4-Pad13)
- U4 pad 8: Net-(U4-Pad8) -> Net-(U29-Pad2)
- U46 pad 10: Net-(U4-Pad8) -> Net-(U4-Pad10)
- U46 pad 11: Net-(U4-Pad11) -> Net-(U4-Pad13)
- U47 pad 1: /MAR/A4 -> /MAR/A5
- U47 pad 2: /MAR/A5 -> /MAR/A6
- U47 pad 21: /Instruction register/HL -> /MAR/A0
- U47 pad 22: Net-(U4-Pad11) -> Net-(U4-Pad13)
- U47 pad 23: /MAR/A0 -> /MAR/A1
- U47 pad 24: /MAR/A1 -> /MAR/A2
- U47 pad 25: /MAR/A2 -> /MAR/A3
- U47 pad 26: /MAR/A3 -> /MAR/A4
- U47 pad 3: /MAR/A6 -> /MAR/A7
- U47 pad 4: /MAR/A7 -> /RAM/HL
- U5 pad 3: Net-(U2-Pad4) -> Net-(U2-Pad9)
- U5 pad 6: Net-(U2-Pad5) -> Net-(U2-Pad10)
- U5 pad 8: Net-(U2-Pad9) -> Net-(U2-Pad12)
- U5 pad 9: Net-(U2-Pad6) -> Net-(U2-Pad8)
- U53 pad 11: Net-(C30-Pad1) -> Net-(C33-Pad1)
- U54 pad 11: Net-(C30-Pad1) -> Net-(C33-Pad1)
- U54 pad 4: Net-(C29-Pad1) -> Net-(C31-Pad1)
- U54 pad 5: Net-(C31-Pad1) -> Net-(C32-Pad1)
- U55 pad 1: /Control logic/SI -> /Control logic/SU
- U55 pad 10: (no net) -> /CLK
- U55 pad 3: Net-(C30-Pad1) -> Net-(C32-Pad1)
- U55 pad 4: (no net) -> /Control logic/SD
- U55 pad 5: (no net) -> /CLK
- U55 pad 6: (no net) -> Net-(C31-Pad1)
- U55 pad 8: (no net) -> Net-(C33-Pad1)
- U55 pad 9: (no net) -> /Control logic/SI
- U58 pad 10: Net-(U58-Pad10) -> /A register/ROT
- U58 pad 11: Net-(TP29-Pad1) -> Net-(U58-Pad11)
- U58 pad 12: /~CLK -> /A register/ROT
- U58 pad 13: /Control logic/II -> /A_0
- U58 pad 4: Net-(TP29-Pad1) -> /~CLK
- U58 pad 5: /Instruction register/HL -> /Control logic/II
- U58 pad 6: Net-(C34-Pad1) -> Net-(TP28-Pad1)
- U58 pad 8: Net-(C35-Pad1) (its old number) -> Net-(U58-Pad8)
- U58 pad 9: Net-(TP29-Pad1) -> /A_7
- U59 pad 19: Net-(U4-Pad12) -> Net-(U59-Pad19)
- U60 pad 1: VCC -> Net-(A1-Pad16)
- U60 pad 10: GND -> /Control logic/~RO
- U60 pad 11: /BUS_0 -> Net-(D98-Pad2)
- U60 pad 12: /BUS_1 -> /Control logic/~PI
- U60 pad 13: /BUS_2 -> Net-(D119-Pad2)
- U60 pad 14: /BUS_3 -> VCC
- U60 pad 2: Net-(D72-Pad2) -> Net-(U59-Pad19)
- U60 pad 3: Net-(D73-Pad2) -> /PC Interface/CLR
- U60 pad 4: Net-(D74-Pad2) -> /~CLR
- U60 pad 5: Net-(D75-Pad2) -> /~CLR
- U60 pad 6: Net-(D76-Pad2) -> /CLR
- U60 pad 7: Net-(D77-Pad2) -> GND
- U60 pad 8: Net-(D78-Pad2) -> /ALU/~FI
- U60 pad 9: Net-(D79-Pad2) -> Net-(D102-Pad2)
- U61 pad 11: Net-(C35-Pad1) (its old number) -> Net-(TP28-Pad1)
- U62 pad 2: Net-(U64-Pad3) -> Net-(U58-Pad8)
- U63 pad 10: Net-(U64-Pad6) -> Net-(U58-Pad11)
- U64 pad 1: /A_7 -> /CLK
- U64 pad 10: /A register/AI -> /Control logic/E0
- U64 pad 11: Net-(U64-Pad11) -> Net-(C43-Pad1)
- U64 pad 12: /Control logic/EXT_I -> /CLK
- U64 pad 13: /Control logic/E1 -> /Control logic/DI
- U64 pad 2: /A register/ROT -> /A register/AI
- U64 pad 3: Net-(U64-Pad3) -> Net-(C38-Pad1)
- U64 pad 4: /A register/ROT -> /Control logic/EXT_I
- U64 pad 5: /A_0 -> /Control logic/E1
- U64 pad 8: Net-(C38-Pad1) -> Net-(U64-Pad8)
- U64 pad 9: /CLK -> /Control logic/EXT_I
- U67 pad 1: Net-(U28-Pad6) -> Net-(U28-Pad8)
- U68 pad 1: Net-(U28-Pad6) -> Net-(U28-Pad8)
- U69 pad 5: Net-(U64-Pad11) -> Net-(U64-Pad6)
- U69 pad 9: Net-(U71-Pad9) -> Net-(U64-Pad8)
- U70 pad 2: Net-(J3-Pad1) -> Net-(J4-Pad2)
- U70 pad 3: Net-(J3-Pad2) -> Net-(J4-Pad4)
- U70 pad 4: Net-(J3-Pad3) -> Net-(J4-Pad6)
- U70 pad 5: Net-(J3-Pad4) -> Net-(J4-Pad8)
- U70 pad 6: Net-(J3-Pad5) -> Net-(J4-Pad10)
- U70 pad 7: Net-(J3-Pad6) -> Net-(J4-Pad12)
- U70 pad 8: Net-(J3-Pad7) -> Net-(J4-Pad14)
- U70 pad 9: Net-(J3-Pad8) -> Net-(J4-Pad16)
- U71 pad 8: Net-(J4-Pad2) -> Net-(J4-Pad3)
- U73 pad 21: /Clock/HLT -> /Control logic/HLT
- U74 pad 13: Net-(D115-Pad2) -> (no net)
- U74 pad 14: Net-(D111-Pad2) -> Net-(D98-Pad2)
- U75 pad 18: Net-(U79-Pad18) -> Net-(D102-Pad2)
- U76 pad 13: Net-(JP1-Pad2) -> Net-(C39-Pad1)
- U76 pad 18: (no net) -> /A register/RGT
- U78 pad 7: Net-(D132-Pad2) -> Net-(D119-Pad2)
- U79 pad 9: /A register/RGT -> (no net)
- U81 pad 11: Net-(C42-Pad1) -> Net-(C43-Pad1)
Routing:
- net GND: track 2673.7 -> 0.00 mm, vias 4 -> 0
- net VCC: track 2201.0 -> 0.00 mm, vias 4 -> 0
- net /BUS_6: track 895.8 -> 0.00 mm, vias 13 -> 0
- net /BUS_7: track 873.0 -> 0.00 mm, vias 9 -> 0
- net /BUS_1: track 866.2 -> 0.00 mm, vias 14 -> 0
- net /BUS_5: track 853.6 -> 0.00 mm, vias 11 -> 0
- net /CLK: track 824.9 -> 0.00 mm, vias 8 -> 0
- net /BUS_3: track 816.3 -> 0.00 mm, vias 9 -> 0
- net /BUS_0: track 812.1 -> 0.00 mm, vias 13 -> 0
- net /BUS_2: track 798.4 -> 0.00 mm, vias 17 -> 0
- net /BUS_4: track 785.5 -> 0.00 mm, vias 16 -> 0
- net /CLR: track 640.9 -> 0.00 mm, vias 1 -> 0
- net /~CLR: track 623.7 -> 0.00 mm, vias 5 -> 0
- net /Control logic/U0: track 506.6 -> 0.00 mm, vias 4 -> 0
- net /Control logic/~PO: track 433.3 -> 0.00 mm, vias 4 -> 0
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- removed copper zone on B.Cu, net GND
- removed copper zone on F.Cu, net GND
Other:
- board text added: "DAT"
- board text added: "EXT CONN"
- board text added: "FI"
- board text added: "Instruction Register"
- board text added: "v2.0d"
- board text removed: "HL"
- board text removed: "IO"
- board text removed: "Instruction"
- board text removed: "Register"
- board text removed: "v2.0b"

Commit message: PCB tracks revision
Parts:
- added C45: 0.01µF, Capacitor_THT:C_Disc_D4.3mm_W1.9mm_P5.00mm, F.Cu at (74.9, 28.6)
- JP1: value POWER -> Arduino_VIN
Connections:
- A1 pad 1: (no net) -> Net-(A1-Pad1)
- A1 pad 17: (no net) -> Net-(A1-Pad17)
- A1 pad 18: (no net) -> Net-(A1-Pad18)
- A1 pad 2: (no net) -> Net-(A1-Pad2)
- A1 pad 22: (no net) -> Net-(A1-Pad22)
- A1 pad 23: (no net) -> Net-(A1-Pad23)
- A1 pad 24: (no net) -> Net-(A1-Pad24)
- A1 pad 25: (no net) -> Net-(A1-Pad25)
- A1 pad 26: (no net) -> Net-(A1-Pad26)
- A1 pad 27: (no net) -> Net-(A1-Pad27)
- A1 pad 28: (no net) -> Net-(A1-Pad28)
- A1 pad 3: (no net) -> Net-(A1-Pad3)
- J1 pad 2: (no net) -> Net-(J1-Pad2)
- J1 pad 3: (no net) -> Net-(J1-Pad3)
- J2 pad 3: (no net) -> Net-(J2-Pad3)
- RN10 pad 2: (no net) -> Net-(RN10-Pad2)
- RN16 pad 5: (no net) -> Net-(RN16-Pad5)
- RN17 pad 2: (no net) -> Net-(RN17-Pad2)
- RV1 pad 3: (no net) -> Net-(RV1-Pad3)
- SW3 pad 1: (no net) -> Net-(SW3-Pad1)
- SW3 pad 2: (no net) -> Net-(SW3-Pad2)
- SW3 pad 3: (no net) -> Net-(SW3-Pad3)
- U11 pad 11: (no net) -> Net-(U11-Pad11)
- U11 pad 12: (no net) -> Net-(U11-Pad12)
- U11 pad 5: (no net) -> Net-(U11-Pad5)
- U11 pad 6: (no net) -> Net-(U11-Pad6)
- U33 pad 4: (no net) -> Net-(U33-Pad4)
- U35 pad 3: (no net) -> Net-(U35-Pad3)
- U35 pad 5: (no net) -> Net-(U35-Pad5)
- U44 pad 15: (no net) -> Net-(U44-Pad15)
- U45 pad 10: (no net) -> Net-(U45-Pad10)
- U45 pad 11: (no net) -> Net-(U45-Pad11)
- U45 pad 2: (no net) -> Net-(U45-Pad2)
- U45 pad 3: (no net) -> Net-(U45-Pad3)
- U45 pad 4: (no net) -> Net-(U45-Pad4)
- U45 pad 5: (no net) -> Net-(U45-Pad5)
- U45 pad 6: (no net) -> Net-(U45-Pad6)
- U45 pad 7: (no net) -> Net-(U45-Pad7)
- U45 pad 9: (no net) -> Net-(U45-Pad9)
- U53 pad 12: (no net) -> Net-(U53-Pad12)
- U53 pad 13: (no net) -> Net-(U53-Pad13)
- U7 pad 7: (no net) -> Net-(U7-Pad7)
- U71 pad 2: (no net) -> Net-(U71-Pad2)
- U71 pad 6: (no net) -> Net-(U71-Pad6)
- U72 pad 11: (no net) -> Net-(U72-Pad11)
- U72 pad 15: (no net) -> Net-(U72-Pad15)
- U72 pad 3: (no net) -> Net-(U72-Pad3)
- U72 pad 4: (no net) -> Net-(U72-Pad4)
- U72 pad 5: (no net) -> Net-(U72-Pad5)
- U72 pad 6: (no net) -> Net-(U72-Pad6)
- U74 pad 13: (no net) -> Net-(U74-Pad13)
- U76 pad 14: (no net) -> Net-(U76-Pad14)
- U76 pad 15: (no net) -> Net-(U76-Pad15)
- U76 pad 17: (no net) -> Net-(U76-Pad17)
- U77 pad 15: (no net) -> Net-(U77-Pad15)
- U78 pad 15: (no net) -> Net-(U78-Pad15)
- U79 pad 15: (no net) -> Net-(U79-Pad15)
- U79 pad 9: (no net) -> Net-(U79-Pad9)
Routing:
- net GND: track 0.00 -> 2672.4 mm, vias 0 -> 6
- net VCC: track 0.00 -> 2180.8 mm, vias 0 -> 3
- net /BUS_7: track 0.00 -> 884.5 mm, vias 0 -> 6
- net /BUS_6: track 0.00 -> 856.7 mm, vias 0 -> 6
- net /BUS_2: track 0.00 -> 839.8 mm, vias 0 -> 9
- net /CLK: track 0.00 -> 838.9 mm, vias 0 -> 6
- net /BUS_3: track 0.00 -> 835.2 mm, vias 0 -> 11
- net /BUS_5: track 0.00 -> 819.4 mm, vias 0 -> 7
- net /BUS_1: track 0.00 -> 771.8 mm, vias 0 -> 8
- net /BUS_0: track 0.00 -> 769.8 mm, vias 0 -> 8
- net /BUS_4: track 0.00 -> 756.7 mm, vias 0 -> 7
- net /~CLR: track 0.00 -> 591.3 mm, vias 0 -> 7
- net /CLR: track 0.00 -> 566.6 mm, vias 0 -> 4
- net /Control logic/U0: track 0.00 -> 495.5 mm, vias 0 -> 6
- net /A_0: track 0.00 -> 481.4 mm, vias 0 -> 5
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- added copper zone on B.Cu, net GND
- added copper zone on F.Cu, net GND
