File: MK1_CPU/8bit-computer/PC-interface.sch (KiCad schematic (older format))
At the start: 8 parts, among them U72 74LS04, U74 74LS245, U75 74LS04

Commit message: version 2.0
Parts:
- removed R135, R136, R137, R138: 1K, Resistor_THT:R_Axial_DIN0207_L6.3mm_D2.5mm_P7.62mm_Horizontal, symbol Device:R
- removed U72: 74LS04, Package_DIP:DIP-14_W7.62mm_Socket, symbol 8bit-computer-rescue:74LS04
- removed unit 3 of U75
- removed unit 4 of U75
- removed unit 5 of U75
- removed unit 1 of U75
- added JP3: Arduino_VIN, Jumper:SolderJumper-2_P1.3mm_Bridged_RoundedPad1.0x1.5mm, symbol Jumper:SolderJumper_2_Bridged
- added RN10: 1K, Resistor_THT:R_Array_SIP9, symbol Device:R_Network08
- A1: value Arduino_Nano_v2.x -> Arduino Nano
- U4: renamed from U75; value 74LS04 -> 74HCT04; footprint Package_DIP:DIP-14_W7.62mm_Socket -> Package_DIP:DIP-14_W7.62mm; symbol 8bit-computer-rescue:74LS04 -> 8bit-computer-rescue:74HCT04
- U59: renamed from U74; value 74LS245 -> 74HCT245; footprint Package_DIP:DIP-20_W7.62mm_Socket -> Package_DIP:DIP-20_W7.62mm; symbol 8bit-computer-rescue:74LS245 -> 8bit-computer-rescue:74HCT245
Connections:
- net labels added: CLK_OUT, CLR, CU_DIS
- wire segments 60 -> 71
- no-connect marks 15 -> 13

Commit message: revision 2.0d
Parts:
- renumbered JP3 to JP1, U4 to U60
Connections:
- net at A1.16 (D13), RN10.6 (R5): now also U60.1; no longer U60.13
- net at U59.19 (CE): now also U60.2; no longer U60.12
Changed lines of the file:
@@
 $EndComp
 $Comp
-L 8bit-computer-rescue:74HCT04 U4
-U 6 1 68295FCC
+L 8bit-computer-rescue:74HCT04 U60
+U 1 1 68295FCC
 P 4550 4250
-F 0 "U4" H 4550 4565 50  0000 C CNN
+F 0 "U60" H 4550 4565 50  0000 C CNN
 F 1 "74HCT04" H 4550 4474 50  0000 C CNN
 F 2 "Package_DIP:DIP-14_W7.62mm" H 4550 4250 50  0001 C CNN
 F 3 "" H 4550 4250 50  0001 C CNN
-	6    4550 4250
+	1    4550 4250
 	-1   0    0    -1
 $EndComp
@@
 NoConn ~ 6350 6700
 $Comp
-L Jumper:SolderJumper_2_Bridged JP3
+L Jumper:SolderJumper_2_Bridged JP1
 U 1 1 5EF7019F
 P 5950 2500
-F 0 "JP3" V 5996 2412 50  0000 R CNN
+F 0 "JP1" V 5996 2412 50  0000 R CNN
 F 1 "Arduino_VIN" V 5905 2412 50  0000 R CNN
 F 2 "Jumper:SolderJumper-2_P1.3mm_Bridged_RoundedPad1.0x1.5mm" H 5950 2500 50  0001 C CNN
