File: MK1_CPU/8bit-computer/a-register.sch (KiCad schematic (older format))
At the start: 24 parts, among them U32 74LS08, U62 74LS157, U63 74LS157, U64 74LS245, U65 74LS273, U66 74LS157, U67 74LS157

Commit message: version 2.0
Parts:
- removed R119, R120, R121, R122, R123, R124, R125, R126: 220, Resistor_THT:R_Axial_DIN0207_L6.3mm_D2.5mm_P7.62mm_Horizontal, symbol Device:R
- added C38: *, Capacitor_THT:C_Disc_D4.3mm_W1.9mm_P5.00mm, symbol Device:C
- added RN21: 1K, Resistor_THT:R_Array_SIP9, symbol Device:R_Network08
- added TP30: AI, TestPoint:TestPoint_Pad_1.0x1.0mm, symbol Connector:TestPoint
- added TP31: ~AO, TestPoint:TestPoint_Pad_1.0x1.0mm, symbol Connector:TestPoint
- added TP32: RGT, TestPoint:TestPoint_Pad_1.0x1.0mm, symbol Connector:TestPoint
- added TP33: ROT, TestPoint:TestPoint_Pad_1.0x1.0mm, symbol Connector:TestPoint
- added TP34: SHF, TestPoint:TestPoint_Pad_1.0x1.0mm, symbol Connector:TestPoint
- added U28: 74HCT32, Package_DIP:DIP-14_W7.62mm, symbol 8bit-computer-rescue:74HCT32
- C37: renamed from C24; footprint Capacitor_THT:C_Rect_L7.0mm_W6.0mm_P5.00mm -> Capacitor_THT:C_Disc_D4.3mm_W1.9mm_P5.00mm
- D88: renamed from D100; value RED -> GREEN
- D89: renamed from D101; value RED -> GREEN
- D90: renamed from D102; value RED -> GREEN
- D91: renamed from D103; value RED -> GREEN
- D92: renamed from D104; value RED -> GREEN
- D93: renamed from D105; value RED -> GREEN
- D94: renamed from D106; value RED -> GREEN
- D95: renamed from D107; value RED -> GREEN
- U64: renamed from U32; value 74LS08 -> 74HCT08; footprint Package_DIP:DIP-14_W7.62mm_Socket -> Package_DIP:DIP-14_W7.62mm; symbol 8bit-computer-rescue:74LS08 -> 8bit-computer-rescue:74HCT08
- U65: renamed from U62; value 74LS157 -> 74HCT157; footprint Package_DIP:DIP-16_W7.62mm_Socket -> Package_DIP:DIP-16_W7.62mm; symbol 8bit-computer-rescue:74LS157 -> 8bit-computer-rescue:74HCT157
- U66: renamed from U63; value 74LS157 -> 74HCT157; footprint Package_DIP:DIP-16_W7.62mm_Socket -> Package_DIP:DIP-16_W7.62mm; symbol 8bit-computer-rescue:74LS157 -> 8bit-computer-rescue:74HCT157
- U67: renamed from U64; value 74LS245 -> 74HCT245; footprint Package_DIP:DIP-20_W7.62mm_Socket -> Package_DIP:DIP-20_W7.62mm; symbol 8bit-computer-rescue:74LS245 -> 8bit-computer-rescue:74HCT245
- U68: renamed from U65; value 74LS273 -> 74HCT273; footprint Package_DIP:DIP-20_W7.62mm_Socket -> Package_DIP:DIP-20_W7.62mm; symbol 8bit-computer-rescue:74LS273 -> 8bit-computer-rescue:74HCT273
- U69: renamed from U66; value 74LS157 -> 74HCT157; footprint Package_DIP:DIP-16_W7.62mm_Socket -> Package_DIP:DIP-16_W7.62mm; symbol 8bit-computer-rescue:74LS157 -> 8bit-computer-rescue:74HCT157
- U70: renamed from U67; value 74LS157 -> 74HCT157; footprint Package_DIP:DIP-16_W7.62mm_Socket -> Package_DIP:DIP-16_W7.62mm; symbol 8bit-computer-rescue:74LS157 -> 8bit-computer-rescue:74HCT157
Connections:
- net labels added: OUT_0, OUT_1, OUT_2, OUT_3, OUT_4, OUT_5, OUT_6, OUT_7
- net labels removed: A_0, A_1, A_2, A_3, A_4, A_5, A_6, A_7
- wire segments 303 -> 315

Commit message: revision 2.0d
Parts:
- renumbered D88 to D80, D89 to D81, D90 to D82, D91 to D83, D92 to D84, D93 to D85, D94 to D86, D95 to D87, RN21 to RN12, TP30 to TP29, TP31 to TP30, TP32 to TP31, TP33 to TP32, TP34 to TP33, U64 to U58, U65 to U62, U66 to U63, U67 to U65, U68 to U66, U69 to U67, U70 to U68
Connections:
- net AI: now also U64.2; no longer U64.10
- net CLK: now also U64.1; no longer U64.9
- net OUT_0: now also U58.13; no longer U58.5
- net OUT_7: now also U58.9; no longer U58.1
- net ROT: now also U28.10, U58.10, U58.12; no longer U28.5, U58.2, U58.4
- net SFT: now also U28.9; no longer U28.4
- net at U67.1 (S), U68.1 (S): now also U28.8; no longer U28.6
- net at U63.10 (I1d): now also U58.11; no longer U58.6
- net at U62.2 (I0a): now also U58.8; no longer U58.3
- net at C38.1, TP29.1, U66.11 (Cp): now also U64.3; no longer U64.8
Changed lines of the file:
@@
 $EndDescr
 $Comp
-L 8bit-computer-rescue:74HCT245 U67
+L 8bit-computer-rescue:74HCT245 U65
 U 1 1 5B61AC1A
 P 3600 2700
-F 0 "U67" H 3700 3275 50  0000 L BNN
+F 0 "U65" H 3700 3275 50  0000 L BNN
 F 1 "74HCT245" H 3650 2125 50  0000 L TNN
 F 2 "Package_DIP:DIP-20_W7.62mm" H 3600 2700 50  0001 C CNN
@@
 BUS_7
 $Comp
-L power:GND #PWR089
+L power:GND #PWR085
 U 1 1 5B61AC3D
 P 3550 6100
-F 0 "#PWR089" H 3550 5850 50  0001 C CNN
+F 0 "#PWR085" H 3550 5850 50  0001 C CNN
 F 1 "GND" H 3550 5950 50  0000 C CNN
 F 2 "" H 3550 6100 50  0001 C CNN
@@
 CLK
 $Comp
-L power:VCC #PWR090
+L power:VCC #PWR086
 U 1 1 5B537572
 P 4300 3050
-F 0 "#PWR090" H 4300 2900 50  0001 C CNN
+F 0 "#PWR086" H 4300 2900 50  0001 C CNN
 F 1 "VCC" H 4300 3200 50  0000 C CNN
 F 2 "" H 4300 3050 50  0001 C CNN
@@
 $EndComp
 $Comp
-L power:GND #PWR087
+L power:GND #PWR083
 U 1 1 5B632BEC
 P 700 6400
-F 0 "#PWR087" H 700 6150 50  0001 C CNN
+F 0 "#PWR083" H 700 6150 50  0001 C CNN
 F 1 "GND" H 700 6250 50  0000 C CNN
 F 2 "" H 700 6400 50  0001 C CNN
@@
 $EndComp
 $Comp
-L power:VCC #PWR086
+L power:VCC #PWR082
 U 1 1 5B632C28
 P 700 5900
-F 0 "#PWR086" H 700 5750 50  0001 C CNN
+F 0 "#PWR082" H 700 5750 50  0001 C CNN
 F 1 "VCC" H 700 6050 50  0000 C CNN
 F 2 "" H 700 5900 50  0001 C CNN
@@
 	3900 4100 5900 4100
 $Comp
-L 8bit-computer-rescue:74HCT157 U70
+L 8bit-computer-rescue:74HCT157 U68
 U 1 1 5F3AF4BF
 P 9300 4100
-F 0 "U70" H 9300 4875 50  0000 C CNN
+F 0 "U68" H 9300 4875 50  0000 C CNN
 F 1 "74HCT157" H 9300 4784 50  0000 C CNN
 F 2 "Package_DIP:DIP-16_W7.62mm" H 9300 4100 50  0001 C CNN
@@
 $EndComp
 $Comp
-L 8bit-computer-rescue:74HCT157 U69
+L 8bit-computer-rescue:74HCT157 U67
 U 1 1 5F3AA992
 P 9300 2550
-F 0 "U69" H 9300 3325 50  0000 C CNN
+F 0 "U67" H 9300 3325 50  0000 C CNN
 F 1 "74HCT157" H 9300 3234 50  0000 C CNN
 F 2 "Package_DIP:DIP-16_W7.62mm" H 9300 2550 50  0001 C CNN
@@
 Connection ~ 8400 4550
 $Comp
-L 8bit-computer-rescue:74HCT157 U65
+L 8bit-computer-rescue:74HCT157 U62
 U 1 1 5F3BAE9F
 P 1850 2600
-F 0 "U65" H 1850 3375 50  0000 C CNN
+F 0 "U62" H 1850 3375 50  0000 C CNN
 F 1 "74HCT157" H 1850 3284 50  0000 C CNN
 F 2 "Package_DIP:DIP-16_W7.62mm" H 1850 2600 50  0001 C CNN
@@
 $EndComp
 $Comp
-L 8bit-computer-rescue:74HCT157 U66
+L 8bit-computer-rescue:74HCT157 U63
 U 1 1 5F3BAE95
 P 1850 4150
-F 0 "U66" H 1850 4925 50  0000 C CNN
+F 0 "U63" H 1850 4925 50  0000 C CNN
 F 1 "74HCT157" H 1850 4834 50  0000 C CNN
 F 2 "Package_DIP:DIP-16_W7.62mm" H 1850 4150 50  0001 C CNN
@@
 	1000 4600 1100 4600
 $Comp
-L power:GND #PWR088
+L power:GND #PWR084
 U 1 1 5F5DF5DD
 P 950 5350
-F 0 "#PWR088" H 950 5100 50  0001 C CNN
+F 0 "#PWR084" H 950 5100 50  0001 C CNN
 F 1 "GND" H 955 5177 50  0000 C CNN
 F 2 "" H 950 5350 50  0001 C CNN
@@
 	8450 4700 8600 4700
 $Comp
-L power:GND #PWR092
+L power:GND #PWR088
 U 1 1 5F5DEB5E
 P 8600 4750
-F 0 "#PWR092" H 8600 4500 50  0001 C CNN
+F 0 "#PWR088" H 8600 4500 50  0001 C CNN
 F 1 "GND" H 8605 4577 50  0000 C CNN
 F 2 "" H 8600 4750 50  0001 C CNN
@@
 	2950 6350 7850 6350
 $Comp
-L 8bit-computer-rescue:74HCT08 U64
-U 2 1 6471A2E8
+L 8bit-computer-rescue:74HCT08 U58
+U 4 1 6471A2E8
 P 1750 7550
-F 0 "U64" H 1750 7916 50  0000 C CNN
+F 0 "U58" H 1750 7916 50  0000 C CNN
 F 1 "74HCT08" H 1750 7825 50  0000 C CNN
 F 2 "Package_DIP:DIP-14_W7.62mm" H 1750 7550 50  0001 C CNN
 F 3 "" H 1750 7550 50  0001 C CNN
-	2    1750 7550
+	4    1750 7550
 	-1   0    0    -1
 $EndComp
 $Comp
-L 8bit-computer-rescue:74HCT08 U64
-U 1 1 6471ACD7
+L 8bit-computer-rescue:74HCT08 U58
+U 3 1 6471ACD7
 P 1750 6750
-F 0 "U64" H 1750 7116 50  0000 C CNN
+F 0 "U58" H 1750 7116 50  0000 C CNN
 F 1 "74HCT08" H 1750 7025 50  0000 C CNN
 F 2 "Package_DIP:DIP-14_W7.62mm" H 1750 6750 50  0001 C CNN
 F 3 "" H 1750 6750 50  0001 C CNN
-	1    1750 6750
+	3    1750 6750
 	-1   0    0    -1
 $EndComp
@@
 	2500 5250 550  5250
 $Comp
-L Device:LED_ALT D95
+L Device:LED_ALT D87
 U 1 1 5B535463
 P 6000 5500
-F 0 "D95" H 6000 5600 50  0000 C CNN
+F 0 "D87" H 6000 5600 50  0000 C CNN
 F 1 "GREEN" H 6000 5400 50  0000 C CNN
 F 2 "LED_THT:LED_D3.0mm" H 6000 5500 50  0001 C CNN
@@
 $EndComp
 $Comp
-L 8bit-computer-rescue:74HCT273 U68
+L 8bit-computer-rescue:74HCT273 U66
 U 1 1 5FBE8D0A
 P 5800 2700
-F 0 "U68" V 5754 3287 50  0000 L CNN
+F 0 "U66" V 5754 3287 50  0000 L CNN
 F 1 "74HCT273" V 5845 3287 50  0000 L CNN
 F 2 "Package_DIP:DIP-20_W7.62mm" H 5800 2700 50  0001 C CNN
@@
 $Comp
 L 8bit-computer-rescue:74HCT08 U64
-U 3 1 5FD2C5C4
+U 1 1 5FD2C5C4
 P 2200 1700
 F 0 "U64" H 2200 2066 50  0000 C CNN
@@
 F 2 "Package_DIP:DIP-14_W7.62mm" H 2200 1700 50  0001 C CNN
 F 3 "" H 2200 1700 50  0001 C CNN
-	3    2200 1700
+	1    2200 1700
 	1    0    0    -1
 $EndComp
@@
 $Comp
 L 8bit-computer-rescue:74HCT32 U28
-U 2 1 5E994DE4
+U 3 1 5E994DE4
 P 9300 5450
 F 0 "U28" H 9300 5816 50  0000 C CNN
@@
 F 2 "Package_DIP:DIP-14_W7.62mm" H 9300 5450 50  0001 C CNN
 F 3 "" H 9300 5450 50  0001 C CNN
-	2    9300 5450
+	3    9300 5450
 	-1   0    0    -1
 $EndComp
@@
 $EndComp
 $Comp
-L power:GND #PWR091
+L power:GND #PWR087
 U 1 1 61844BA6
 P 4850 2250
-F 0 "#PWR091" H 4850 2000 50  0001 C CNN
+F 0 "#PWR087" H 4850 2000 50  0001 C CNN
 F 1 "GND" H 4850 2100 50  0000 C CNN
 F 2 "" H 4850 2250 50  0001 C CNN
@@
 P 4450 1650
 AR Path="/5B533ECB/774D1F1A" Ref="TP?"  Part="1"
-AR Path="/5B53468B/774D1F1A" Ref="TP30"  Part="1"
-F 0 "TP30" H 4508 1768 50  0000 L CNN
+AR Path="/5B53468B/774D1F1A" Ref="TP29"  Part="1"
+F 0 "TP29" H 4508 1768 50  0000 L CNN
 F 1 "AI" H 4508 1677 50  0000 L CNN
 F 2 "TestPoint:TestPoint_Pad_1.0x1.0mm" H 4650 1650 50  0001 C CNN
@@
 P 4550 3650
 AR Path="/5B533ECB/77525277" Ref="TP?"  Part="1"
-AR Path="/5B53468B/77525277" Ref="TP31"  Part="1"
-F 0 "TP31" H 4608 3774 50  0000 L CNN
+AR Path="/5B53468B/77525277" Ref="TP30"  Part="1"
+F 0 "TP30" H 4608 3774 50  0000 L CNN
 F 1 "~AO" H 4608 3676 50  0000 L CNN
 F 2 "TestPoint:TestPoint_Pad_1.0x1.0mm" H 4750 3650 50  0001 C CNN
@@
 P 9300 6250
 AR Path="/5B533ECB/7755D3B6" Ref="TP?"  Part="1"
-AR Path="/5B53468B/7755D3B6" Ref="TP32"  Part="1"
-F 0 "TP32" H 9358 6368 50  0000 L CNN
+AR Path="/5B53468B/7755D3B6" Ref="TP31"  Part="1"
+F 0 "TP31" H 9358 6368 50  0000 L CNN
 F 1 "RGT" H 9358 6277 50  0000 L CNN
 F 2 "TestPoint:TestPoint_Pad_1.0x1.0mm" H 9500 6250 50  0001 C CNN
@@
 P 10000 5300
 AR Path="/5B533ECB/775967F6" Ref="TP?"  Part="1"
-AR Path="/5B53468B/775967F6" Ref="TP34"  Part="1"
-F 0 "TP34" H 10058 5418 50  0000 L CNN
+AR Path="/5B53468B/775967F6" Ref="TP33"  Part="1"
+F 0 "TP33" H 10058 5418 50  0000 L CNN
 F 1 "SHF" H 10058 5327 50  0000 L CNN
 F 2 "TestPoint:TestPoint_Pad_1.0x1.0mm" H 10200 5300 50  0001 C CNN
@@
 P 9300 6700
 AR Path="/5B533ECB/775CFBD2" Ref="TP?"  Part="1"
-AR Path="/5B53468B/775CFBD2" Ref="TP33"  Part="1"
-F 0 "TP33" H 9358 6818 50  0000 L CNN
+AR Path="/5B53468B/775CFBD2" Ref="TP32"  Part="1"
+F 0 "TP32" H 9358 6818 50  0000 L CNN
 F 1 "ROT" H 9358 6727 50  0000 L CNN
 F 2 "TestPoint:TestPoint_Pad_1.0x1.0mm" H 9500 6700 50  0001 C CNN
@@
 	9300 6750 3400 6750
 $Comp
-L Device:R_Network08 RN21
+L Device:R_Network08 RN12
 U 1 1 7876B230
 P 4300 6050
-F 0 "RN21" H 3820 6004 50  0000 R CNN
+F 0 "RN12" H 3820 6004 50  0000 R CNN
 F 1 "1K" H 3820 6095 50  0000 R CNN
 F 2 "Resistor_THT:R_Array_SIP9" V 4775 6050 50  0001 C CNN
@@
 	5700 5200 5700 5350
 $Comp
-L Device:LED_ALT D94
+L Device:LED_ALT D86
 U 1 1 5B535434
 P 5700 5500
-F 0 "D94" H 5700 5600 50  0000 C CNN
+F 0 "D86" H 5700 5600 50  0000 C CNN
 F 1 "GREEN" H 5700 5400 50  0000 C CNN
 F 2 "LED_THT:LED_D3.0mm" H 5700 5500 50  0001 C CNN
@@
 	3900 5650 3900 5850
 $Comp
-L Device:LED_ALT D93
+L Device:LED_ALT D85
 U 1 1 5B61AC27
 P 5400 5500
-F 0 "D93" H 5400 5600 50  0000 C CNN
+F 0 "D85" H 5400 5600 50  0000 C CNN
 F 1 "GREEN" H 5400 5400 50  0000 C CNN
 F 2 "LED_THT:LED_D3.0mm" H 5400 5500 50  0001 C CNN
@@
 $EndComp
 $Comp
-L Device:LED_ALT D92
+L Device:LED_ALT D84
 U 1 1 5B61AC25
 P 5100 5500
-F 0 "D92" H 5100 5600 50  0000 C CNN
+F 0 "D84" H 5100 5600 50  0000 C CNN
 F 1 "GREEN" H 5100 5400 50  0000 C CNN
 F 2 "LED_THT:LED_D3.0mm" H 5100 5500 50  0001 C CNN
@@
 $EndComp
 $Comp
-L Device:LED_ALT D91
+L Device:LED_ALT D83
 U 1 1 5B61AC22
 P 4800 5500
-F 0 "D91" H 4800 5600 50  0000 C CNN
+F 0 "D83" H 4800 5600 50  0000 C CNN
 F 1 "GREEN" H 4800 5400 50  0000 C CNN
 F 2 "LED_THT:LED_D3.0mm" H 4800 5500 50  0001 C CNN
@@
 $EndComp
 $Comp
-L Device:LED_ALT D90
+L Device:LED_ALT D82
 U 1 1 5B53538E
 P 4500 5500
-F 0 "D90" H 4500 5600 50  0000 C CNN
+F 0 "D82" H 4500 5600 50  0000 C CNN
 F 1 "GREEN" H 4500 5400 50  0000 C CNN
 F 2 "LED_THT:LED_D3.0mm" H 4500 5500 50  0001 C CNN
@@
 $EndComp
 $Comp
-L Device:LED_ALT D89
+L Device:LED_ALT D81
 U 1 1 5B61AC1F
 P 4200 5500
-F 0 "D89" H 4200 5600 50  0000 C CNN
+F 0 "D81" H 4200 5600 50  0000 C CNN
 F 1 "GREEN" H 4200 5400 50  0000 C CNN
 F 2 "LED_THT:LED_D3.0mm" H 4200 5500 50  0001 C CNN
@@
 $EndComp
 $Comp
-L Device:LED_ALT D88
+L Device:LED_ALT D80
 U 1 1 5B61AC1D
 P 3900 5500
-F 0 "D88" H 3900 5600 50  0000 C CNN
+F 0 "D80" H 3900 5600 50  0000 C CNN
 F 1 "GREEN" H 3900 5400 50  0000 C CNN
 F 2 "LED_THT:LED_D3.0mm" H 3900 5500 50  0001 C CNN
