File: MK1_CPU/8bit-computer/alu.sch (KiCad schematic (older format))
At the start: 41 parts, among them U1 74LS86, U11 74LS08, U12 74LS173, U13 74LS00, U14 74LS02, U15 74LS245, U16 74LS283, U17 74LS283, U18 74LS157, U19 74LS157, U20 74LS157, U21 74LS86, U22 74LS86, U23 74LS157, U24 74LS32, U25 74LS08, U26 74LS08, U27 74LS32, U7 74LS32

Commit message: version 2.0
Parts:
- removed R34, R35, R36, R37, R38, R39, R40, R41: 220, Resistor_THT:R_Axial_DIN0207_L6.3mm_D2.5mm_P7.62mm_Horizontal, symbol Device:R
- removed U13: 74LS00, Package_DIP:DIP-14_W7.62mm_Socket, symbol 8bit-computer-rescue:74LS00
- added C15: *, Capacitor_THT:C_Disc_D4.3mm_W1.9mm_P5.00mm, symbol Device:C
- added RN4: 470, Resistor_THT:R_Array_SIP9, symbol Device:R_Network08
- added TP10: AND, TestPoint:TestPoint_Pad_1.0x1.0mm, symbol Connector:TestPoint
- added TP11: EI, TestPoint:TestPoint_Pad_1.0x1.0mm, symbol Connector:TestPoint
- added TP12: ~EO, TestPoint:TestPoint_Pad_1.0x1.0mm, symbol Connector:TestPoint
- added TP13: NOT, TestPoint:TestPoint_Pad_1.0x1.0mm, symbol Connector:TestPoint
- added TP14: SUB, TestPoint:TestPoint_Pad_1.0x1.0mm, symbol Connector:TestPoint
- added TP6: ~FI, TestPoint:TestPoint_Pad_1.0x1.0mm, symbol Connector:TestPoint
- added TP7: ZF, TestPoint:TestPoint_Pad_1.0x1.0mm, symbol Connector:TestPoint
- added TP8: CF, TestPoint:TestPoint_Pad_1.0x1.0mm, symbol Connector:TestPoint
- added TP9: OR, TestPoint:TestPoint_Pad_1.0x1.0mm, symbol Connector:TestPoint
- added unit 4 of U10
- added U18: 74HCT273, Package_DIP:DIP-20_W7.62mm, symbol 8bit-computer-rescue:74HCT273
- added U2: 74HCT32, Package_DIP:DIP-14_W7.62mm, symbol 8bit-computer-rescue:74HCT32
- added U23: 74HCT86, Package_DIP:DIP-14_W7.62mm, symbol 8bit-computer-rescue:74HCT86
- added unit 1 of U27
- C13: renamed from C10; footprint Capacitor_THT:C_Rect_L7.0mm_W6.0mm_P5.00mm -> Capacitor_THT:C_Disc_D4.3mm_W1.9mm_P5.00mm
- C14: renamed from C11; footprint Capacitor_THT:C_Rect_L7.0mm_W6.0mm_P5.00mm -> Capacitor_THT:C_Disc_D4.3mm_W1.9mm_P5.00mm
- D19: renamed from D18; value GREEN -> WHITE
- D20: renamed from D19; value GREEN -> WHITE
- R10: renamed from R32; value 220 -> 1K
- R11: renamed from R33; value 220 -> 1K
- U10, U25: renamed from U11; value 74LS08 -> 74HCT08; footprint Package_DIP:DIP-14_W7.62mm_Socket -> Package_DIP:DIP-14_W7.62mm; symbol 8bit-computer-rescue:74LS08 -> 8bit-computer-rescue:74HCT08
- U11: renamed from U12; value 74LS173 -> 74HCT173; footprint Package_DIP:DIP-16_W7.62mm_Socket -> Package_DIP:DIP-16_W7.62mm; symbol 8bit-computer-rescue:74LS173 -> 8bit-computer-rescue:74HCT173
- U12: renamed from U14; value 74LS02 -> 74HCT02; footprint Package_DIP:DIP-14_W7.62mm_Socket -> Package_DIP:DIP-14_W7.62mm; symbol 8bit-computer-rescue:74LS02 -> 8bit-computer-rescue:74HCT02
- U13: renamed from U15; value 74LS245 -> 74HCT245; footprint Package_DIP:DIP-20_W7.62mm_Socket -> Package_DIP:DIP-20_W7.62mm; symbol 8bit-computer-rescue:74LS245 -> 8bit-computer-rescue:74HCT245
- U14: renamed from U16; value 74LS283 -> 74HCT283; footprint Package_DIP:DIP-16_W7.62mm_Socket -> Package_DIP:DIP-16_W7.62mm; symbol 8bit-computer-rescue:74LS283 -> 8bit-computer-rescue:74HCT283
- U15: renamed from U17; value 74LS283 -> 74HCT283; footprint Package_DIP:DIP-16_W7.62mm_Socket -> Package_DIP:DIP-16_W7.62mm; symbol 8bit-computer-rescue:74LS283 -> 8bit-computer-rescue:74HCT283
- U16: renamed from U18; value 74LS157 -> 74HCT157; footprint Package_DIP:DIP-16_W7.62mm_Socket -> Package_DIP:DIP-16_W7.62mm; symbol 8bit-computer-rescue:74LS157 -> 8bit-computer-rescue:74HCT157
- U17: renamed from U19; value 74LS157 -> 74HCT157; footprint Package_DIP:DIP-16_W7.62mm_Socket -> Package_DIP:DIP-16_W7.62mm; symbol 8bit-computer-rescue:74LS157 -> 8bit-computer-rescue:74HCT157
- U19: renamed from U20; value 74LS157 -> 74HCT157; footprint Package_DIP:DIP-16_W7.62mm_Socket -> Package_DIP:DIP-16_W7.62mm; symbol 8bit-computer-rescue:74LS157 -> 8bit-computer-rescue:74HCT157
- U20: renamed from U21; value 74LS86 -> 74HCT86; footprint Package_DIP:DIP-14_W7.62mm_Socket -> Package_DIP:DIP-14_W7.62mm; symbol 8bit-computer-rescue:74LS86 -> 8bit-computer-rescue:74HCT86
- U20: renamed from U1; value 74LS86 -> 74HCT86; footprint Package_DIP:DIP-14_W7.62mm_Socket -> Package_DIP:DIP-14_W7.62mm; symbol 8bit-computer-rescue:74LS86 -> 8bit-computer-rescue:74HCT86
- U21: renamed from U22; value 74LS86 -> 74HCT86; footprint Package_DIP:DIP-14_W7.62mm_Socket -> Package_DIP:DIP-14_W7.62mm; symbol 8bit-computer-rescue:74LS86 -> 8bit-computer-rescue:74HCT86
- U21: value 74LS86 -> 74HCT86; footprint Package_DIP:DIP-14_W7.62mm_Socket -> Package_DIP:DIP-14_W7.62mm; symbol 8bit-computer-rescue:74LS86 -> 8bit-computer-rescue:74HCT86
- U22: renamed from U23; value 74LS157 -> 74HCT157; footprint Package_DIP:DIP-16_W7.62mm_Socket -> Package_DIP:DIP-16_W7.62mm; symbol 8bit-computer-rescue:74LS157 -> 8bit-computer-rescue:74HCT157
- U24: value 74LS32 -> 74HCT32; footprint Package_DIP:DIP-14_W7.62mm_Socket -> Package_DIP:DIP-14_W7.62mm; symbol 8bit-computer-rescue:74LS32 -> 8bit-computer-rescue:74HCT32
- U24: renamed from U7; value 74LS32 -> 74HCT32; footprint Package_DIP:DIP-14_W7.62mm_Socket -> Package_DIP:DIP-14_W7.62mm; symbol 8bit-computer-rescue:74LS32 -> 8bit-computer-rescue:74HCT32
- U25, U26: value 74LS08 -> 74HCT08; footprint Package_DIP:DIP-14_W7.62mm_Socket -> Package_DIP:DIP-14_W7.62mm; symbol 8bit-computer-rescue:74LS08 -> 8bit-computer-rescue:74HCT08
- U26: renamed from U25; value 74LS08 -> 74HCT08; footprint Package_DIP:DIP-14_W7.62mm_Socket -> Package_DIP:DIP-14_W7.62mm; symbol 8bit-computer-rescue:74LS08 -> 8bit-computer-rescue:74HCT08
- U27: renamed from U24; value 74LS32 -> 74HCT32; footprint Package_DIP:DIP-14_W7.62mm_Socket -> Package_DIP:DIP-14_W7.62mm; symbol 8bit-computer-rescue:74LS32 -> 8bit-computer-rescue:74HCT32
- U28: renamed from U27; value 74LS32 -> 74HCT32; footprint Package_DIP:DIP-14_W7.62mm_Socket -> Package_DIP:DIP-14_W7.62mm; symbol 8bit-computer-rescue:74LS32 -> 8bit-computer-rescue:74HCT32
- renumbered D20 to D21, D21 to D22, D22 to D23, D23 to D24, D24 to D25, D25 to D26, D26 to D27, D27 to D28
Connections:
- net labels added: EI, NOT, SUB, ~CLR
- net labels removed: B_0, B_1, B_2, B_3, B_4, B_5, B_6, B_7, SU
- wire segments 509 -> 581

Commit message: revision 2.0d
Parts:
- renumbered C13 to C14, C14 to C15, C15 to C16, U24 to U12, U2 to U12, U12 to U13, U13 to U14, U14 to U15, U15 to U16, U16 to U17, U17 to U18, U18 to U19, U19 to U20, U20 to U21, U21 to U22, U22 to U23, U23 to U24, U24 to U25, U27 to U25, U25 to U26, U26 to U27, U27 to U28
Connections:
- net AND: now also U12.1; no longer U12.12
- net A_0: now also U12.12; no longer U12.9
- net A_1: now also U12.9; no longer U12.4
- net A_2: now also U12.4; no longer U12.1
- net A_3: now also U25.1; no longer U25.12
- net A_4: now also U28.4; no longer U28.1
- net A_5: now also U28.1; no longer U28.12
- net A_6: now also U25.12; no longer U25.9
- net A_7: now also U25.9; no longer U25.4
- net NOT: now also U25.5; no longer U25.2
- net OR: now also U12.2; no longer U12.13
- net SUB: now also U25.4; no longer U25.1
- net at U21.10 (IN2), U21.13 (IN2), U21.2 (IN2)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: now also U25.6; no longer U25.3
- net at U19.5 (Q1), U22.9 (IN1), U26.9: now also U12.10; no longer U12.5
- net at U19.2 (Q0), U22.12 (IN1), U26.12: now also U12.13; no longer U12.10
- net at U19.9 (Q3), U22.1 (IN1), U26.1: now also U25.2; no longer U25.13
- net at U19.6 (Q2), U22.4 (IN1), U26.4: now also U12.5; no longer U12.2
- net at U19.15 (Q5), U21.9 (IN1), U27.9: now also U28.2; no longer U28.13
- net at U19.12 (Q4), U21.12 (IN1), U27.12: now also U28.5; no longer U28.2
- net at U19.19 (Q7), U21.1 (IN1), U27.1: now also U25.10; no longer U25.5
- net at U19.16 (Q6), U21.4 (IN1), U27.4: now also U25.13; no longer U25.10
- net at U23.3 (I1a): now also U25.3; no longer U25.11
- net at U23.6 (I1b): now also U12.6; no longer U12.3
- net at U23.13 (I1c): now also U12.8; no longer U12.6
- net at U23.10 (I1d): now also U12.11; no longer U12.8
- net at U20.3 (I1a): now also U25.8; no longer U25.6
- net at U20.6 (I1b): now also U25.11; no longer U25.8
- net at U20.13 (I1c): now also U28.3; no longer U28.11
- net at U20.10 (I1d): now also U28.6; no longer U28.3
- net at U17.1 (S), U18.1 (S): now also U12.3; no longer U12.11
