File: MK1_CPU/8bit-computer/b-register.sch (KiCad schematic (older format))
At the start: 20 parts, among them U10 74LS273, U5 74LS08, U9 74LS245

Commit message: version 2.0
Parts:
- removed R24, R25, R26, R27, R28, R29, R30, R31: 220, Resistor_THT:R_Axial_DIN0207_L6.3mm_D2.5mm_P7.62mm_Horizontal, symbol Device:R
- added C12: *, Capacitor_THT:C_Disc_D4.3mm_W1.9mm_P5.00mm, symbol Device:C
- added RN3: 1K, Resistor_THT:R_Array_SIP9, symbol Device:R_Network08
- added TP4: ~REG-O, TestPoint:TestPoint_Pad_1.0x1.0mm, symbol Connector:TestPoint
- added TP5: REG-I, TestPoint:TestPoint_Pad_1.0x1.0mm, symbol Connector:TestPoint
- C11: renamed from C9; footprint Capacitor_THT:C_Rect_L7.0mm_W6.0mm_P5.00mm -> Capacitor_THT:C_Disc_D4.3mm_W1.9mm_P5.00mm
- D11: renamed from D10; value RED -> GREEN
- D12: renamed from D11; value RED -> GREEN
- D13: renamed from D12; value RED -> GREEN
- D14: renamed from D13; value RED -> GREEN
- D15: renamed from D14; value RED -> GREEN
- D16: renamed from D15; value RED -> GREEN
- D17: renamed from D16; value RED -> GREEN
- D18: renamed from D17; value RED -> GREEN
- U5: value 74LS08 -> 74HCT08; footprint Package_DIP:DIP-14_W7.62mm_Socket -> Package_DIP:DIP-14_W7.62mm; symbol 8bit-computer-rescue:74LS08 -> 8bit-computer-rescue:74HCT08
- U8: renamed from U9; value 74LS245 -> 74HCT245; footprint Package_DIP:DIP-20_W7.62mm_Socket -> Package_DIP:DIP-20_W7.62mm; symbol 8bit-computer-rescue:74LS245 -> 8bit-computer-rescue:74HCT245
- U9: renamed from U10; value 74LS273 -> 74HCT273; footprint Package_DIP:DIP-20_W7.62mm_Socket -> Package_DIP:DIP-20_W7.62mm; symbol 8bit-computer-rescue:74LS273 -> 8bit-computer-rescue:74HCT273
Connections:
- net labels added: OUT_0, OUT_1, OUT_2, OUT_3, OUT_4, OUT_5, OUT_6, OUT_7, REG-I, ~REG-O
- net labels removed: BI, B_0, B_1, B_2, B_3, B_4, B_5, B_6, B_7, ~BO
- wire segments 126 -> 130
Other:
- moved on the sheet: C41

Commit message: revision 2.0d
Parts:
- renumbered C11 to C12, C12 to C13
Connections:
- net CLK: now also U5.12; no longer U5.9
- net REG-I: now also U5.13; no longer U5.10
- net at C13.1, TP5.1, U9.11 (Cp): now also U5.11; no longer U5.8
Changed lines of the file:
@@
 $Descr USLetter 11000 8500
 encoding utf-8
-Sheet 10 16
+Sheet 16 16
 Title ""
 Date ""
@@
 AR Path="/5F79BBF0/5B5346E8" Ref="U?"  Part="1"
 AR Path="/5F7B99D0/5B5346E8" Ref="U56"  Part="1"
-AR Path="/5F7BF5BB/5B5346E8" Ref="U85"  Part="1"
-F 0 "U85" H 3700 3175 50  0000 L BNN
+AR Path="/5F7BF5BB/5B5346E8" Ref="U80"  Part="1"
+F 0 "U80" H 3700 3175 50  0000 L BNN
 F 1 "74HCT245" H 3650 2025 50  0000 L TNN
 F 2 "Package_DIP:DIP-20_W7.62mm" H 3600 2600 50  0001 C CNN
@@
 AR Path="/5F79BBF0/5B61AC1C" Ref="D?"  Part="1"
 AR Path="/5F7B99D0/5B61AC1C" Ref="D64"  Part="1"
-AR Path="/5F7BF5BB/5B61AC1C" Ref="D140"  Part="1"
-F 0 "D140" H 3900 5600 50  0000 C CNN
+AR Path="/5F7BF5BB/5B61AC1C" Ref="D127"  Part="1"
+F 0 "D127" H 3900 5600 50  0000 C CNN
 F 1 "GREEN" H 3900 5400 50  0000 C CNN
 F 2 "LED_THT:LED_D3.0mm" H 3900 5500 50  0001 C CNN
@@
 AR Path="/5F79BBF0/5B53536E" Ref="D?"  Part="1"
 AR Path="/5F7B99D0/5B53536E" Ref="D65"  Part="1"
-AR Path="/5F7BF5BB/5B53536E" Ref="D141"  Part="1"
-F 0 "D141" H 4200 5600 50  0000 C CNN
+AR Path="/5F7BF5BB/5B53536E" Ref="D128"  Part="1"
+F 0 "D128" H 4200 5600 50  0000 C CNN
 F 1 "GREEN" H 4200 5400 50  0000 C CNN
 F 2 "LED_THT:LED_D3.0mm" H 4200 5500 50  0001 C CNN
@@
 AR Path="/5F79BBF0/5B61AC20" Ref="D?"  Part="1"
 AR Path="/5F7B99D0/5B61AC20" Ref="D66"  Part="1"
-AR Path="/5F7BF5BB/5B61AC20" Ref="D142"  Part="1"
-F 0 "D142" H 4500 5600 50  0000 C CNN
+AR Path="/5F7BF5BB/5B61AC20" Ref="D129"  Part="1"
+F 0 "D129" H 4500 5600 50  0000 C CNN
 F 1 "GREEN" H 4500 5400 50  0000 C CNN
 F 2 "LED_THT:LED_D3.0mm" H 4500 5500 50  0001 C CNN
@@
 AR Path="/5F79BBF0/5B61AC23" Ref="D?"  Part="1"
 AR Path="/5F7B99D0/5B61AC23" Ref="D67"  Part="1"
-AR Path="/5F7BF5BB/5B61AC23" Ref="D143"  Part="1"
-F 0 "D143" H 4800 5600 50  0000 C CNN
+AR Path="/5F7BF5BB/5B61AC23" Ref="D130"  Part="1"
+F 0 "D130" H 4800 5600 50  0000 C CNN
 F 1 "GREEN" H 4800 5400 50  0000 C CNN
 F 2 "LED_THT:LED_D3.0mm" H 4800 5500 50  0001 C CNN
@@
 AR Path="/5F79BBF0/5B61AC24" Ref="D?"  Part="1"
 AR Path="/5F7B99D0/5B61AC24" Ref="D68"  Part="1"
-AR Path="/5F7BF5BB/5B61AC24" Ref="D144"  Part="1"
-F 0 "D144" H 5100 5600 50  0000 C CNN
+AR Path="/5F7BF5BB/5B61AC24" Ref="D131"  Part="1"
+F 0 "D131" H 5100 5600 50  0000 C CNN
 F 1 "GREEN" H 5100 5400 50  0000 C CNN
 F 2 "LED_THT:LED_D3.0mm" H 5100 5500 50  0001 C CNN
@@
 AR Path="/5F79BBF0/5B61AC26" Ref="D?"  Part="1"
 AR Path="/5F7B99D0/5B61AC26" Ref="D69"  Part="1"
-AR Path="/5F7BF5BB/5B61AC26" Ref="D145"  Part="1"
-F 0 "D145" H 5400 5600 50  0000 C CNN
+AR Path="/5F7BF5BB/5B61AC26" Ref="D132"  Part="1"
+F 0 "D132" H 5400 5600 50  0000 C CNN
 F 1 "GREEN" H 5400 5400 50  0000 C CNN
 F 2 "LED_THT:LED_D3.0mm" H 5400 5500 50  0001 C CNN
@@
 AR Path="/5F79BBF0/5B61AC28" Ref="D?"  Part="1"
 AR Path="/5F7B99D0/5B61AC28" Ref="D70"  Part="1"
-AR Path="/5F7BF5BB/5B61AC28" Ref="D146"  Part="1"
-F 0 "D146" H 5700 5600 50  0000 C CNN
+AR Path="/5F7BF5BB/5B61AC28" Ref="D133"  Part="1"
+F 0 "D133" H 5700 5600 50  0000 C CNN
 F 1 "GREEN" H 5700 5400 50  0000 C CNN
 F 2 "LED_THT:LED_D3.0mm" H 5700 5500 50  0001 C CNN
@@
 AR Path="/5F79BBF0/5B61AC2A" Ref="D?"  Part="1"
 AR Path="/5F7B99D0/5B61AC2A" Ref="D71"  Part="1"
-AR Path="/5F7BF5BB/5B61AC2A" Ref="D147"  Part="1"
-F 0 "D147" H 6000 5600 50  0000 C CNN
+AR Path="/5F7BF5BB/5B61AC2A" Ref="D134"  Part="1"
+F 0 "D134" H 6000 5600 50  0000 C CNN
 F 1 "GREEN" H 6000 5400 50  0000 C CNN
 F 2 "LED_THT:LED_D3.0mm" H 6000 5500 50  0001 C CNN
@@
 AR Path="/5F79BBF0/5B536319" Ref="#PWR?"  Part="1"
 AR Path="/5F7B99D0/5B536319" Ref="#PWR074"  Part="1"
-AR Path="/5F7BF5BB/5B536319" Ref="#PWR0121"  Part="1"
-F 0 "#PWR0121" H 5300 6200 50  0001 C CNN
+AR Path="/5F7BF5BB/5B536319" Ref="#PWR0114"  Part="1"
+F 0 "#PWR0114" H 5300 6200 50  0001 C CNN
 F 1 "GND" H 5300 6300 50  0000 C CNN
 F 2 "" H 5300 6450 50  0001 C CNN
@@
 AR Path="/5F79BBF0/5B61AC3F" Ref="#PWR?"  Part="1"
 AR Path="/5F7B99D0/5B61AC3F" Ref="#PWR073"  Part="1"
-AR Path="/5F7BF5BB/5B61AC3F" Ref="#PWR0120"  Part="1"
-F 0 "#PWR0120" H 4300 2800 50  0001 C CNN
+AR Path="/5F7BF5BB/5B61AC3F" Ref="#PWR0113"  Part="1"
+F 0 "#PWR0113" H 4300 2800 50  0001 C CNN
 F 1 "VCC" H 4300 3100 50  0000 C CNN
 F 2 "" H 4300 2950 50  0001 C CNN
@@
 ~CLR
 $Comp
-L Device:C C11
+L Device:C C12
 U 1 1 5B6331E0
 P 1650 2000
-AR Path="/5B53AFFA/5B6331E0" Ref="C11"  Part="1"
+AR Path="/5B53AFFA/5B6331E0" Ref="C12"  Part="1"
 AR Path="/6432FCD8/5B6331E0" Ref="C?"  Part="1"
 AR Path="/5F79BBF0/5B6331E0" Ref="C?"  Part="1"
-AR Path="/5F7B99D0/5B6331E0" Ref="C32"  Part="1"
-AR Path="/5F7BF5BB/5B6331E0" Ref="C41"  Part="1"
-F 0 "C41" H 1675 2100 50  0000 L CNN
+AR Path="/5F7B99D0/5B6331E0" Ref="C34"  Part="1"
+AR Path="/5F7BF5BB/5B6331E0" Ref="C42"  Part="1"
+F 0 "C42" H 1675 2100 50  0000 L CNN
 F 1 "0.1µF" H 1675 1900 50  0000 L CNN
 F 2 "Capacitor_THT:C_Disc_D4.3mm_W1.9mm_P5.00mm" H 1688 1850 50  0001 C CNN
@@
 AR Path="/5F79BBF0/5B633224" Ref="#PWR?"  Part="1"
 AR Path="/5F7B99D0/5B633224" Ref="#PWR071"  Part="1"
-AR Path="/5F7BF5BB/5B633224" Ref="#PWR0118"  Part="1"
-F 0 "#PWR0118" H 1650 1600 50  0001 C CNN
+AR Path="/5F7BF5BB/5B633224" Ref="#PWR0111"  Part="1"
+F 0 "#PWR0111" H 1650 1600 50  0001 C CNN
 F 1 "VCC" H 1650 1900 50  0000 C CNN
 F 2 "" H 1650 1750 50  0001 C CNN
@@
 AR Path="/5F79BBF0/5B633260" Ref="#PWR?"  Part="1"
 AR Path="/5F7B99D0/5B633260" Ref="#PWR072"  Part="1"
-AR Path="/5F7BF5BB/5B633260" Ref="#PWR0119"  Part="1"
-F 0 "#PWR0119" H 1650 2000 50  0001 C CNN
+AR Path="/5F7BF5BB/5B633260" Ref="#PWR0112"  Part="1"
+F 0 "#PWR0112" H 1650 2000 50  0001 C CNN
 F 1 "GND" H 1650 2100 50  0000 C CNN
 F 2 "" H 1650 2250 50  0001 C CNN
@@
 AR Path="/5F79BBF0/5EA366FE" Ref="U?"  Part="1"
 AR Path="/5F7B99D0/5EA366FE" Ref="U57"  Part="1"
-AR Path="/5F7BF5BB/5EA366FE" Ref="U86"  Part="1"
-F 0 "U86" V 6254 3187 50  0000 L CNN
+AR Path="/5F7BF5BB/5EA366FE" Ref="U81"  Part="1"
+F 0 "U81" V 6254 3187 50  0000 L CNN
 F 1 "74HCT273" V 6345 3187 50  0000 L CNN
 F 2 "Package_DIP:DIP-20_W7.62mm" H 6300 2600 50  0001 C CNN
@@
 $Comp
 L 8bit-computer-rescue:74HCT08 U5
-U 3 1 5EA392A6
+U 4 1 5EA392A6
 P 8750 1800
 AR Path="/5B53AFFA/5EA392A6" Ref="U5"  Part="4"
 AR Path="/5F79BBF0/5EA392A6" Ref="U?"  Part="4"
 AR Path="/5F7B99D0/5EA392A6" Ref="U58"  Part="1"
-AR Path="/5F7BF5BB/5EA392A6" Ref="U74"  Part="3"
-F 0 "U74" H 8750 1414 50  0000 C CNN
+AR Path="/5F7BF5BB/5EA392A6" Ref="U64"  Part="4"
+F 0 "U64" H 8750 1414 50  0000 C CNN
 F 1 "74HCT08" H 8750 1505 50  0000 C CNN
 F 2 "Package_DIP:DIP-14_W7.62mm" H 8750 1800 50  0001 C CNN
 F 3 "" H 8750 1800 50  0001 C CNN
-	3    8750 1800
+	4    8750 1800
 	-1   0    0    1
 $EndComp
@@
 	3900 5250 3900 5350
 $Comp
-L Device:C C12
+L Device:C C13
 U 1 1 6187CB8A
 P 7700 2050
-AR Path="/5B53AFFA/6187CB8A" Ref="C12"  Part="1"
+AR Path="/5B53AFFA/6187CB8A" Ref="C13"  Part="1"
 AR Path="/6432FCD8/6187CB8A" Ref="C?"  Part="1"
 AR Path="/5F79BBF0/6187CB8A" Ref="C?"  Part="1"
-AR Path="/5F7B99D0/6187CB8A" Ref="C33"  Part="1"
-AR Path="/5F7BF5BB/6187CB8A" Ref="C42"  Part="1"
-F 0 "C42" H 7725 2150 50  0000 L CNN
+AR Path="/5F7B99D0/6187CB8A" Ref="C35"  Part="1"
+AR Path="/5F7BF5BB/6187CB8A" Ref="C43"  Part="1"
+F 0 "C43" H 7725 2150 50  0000 L CNN
 F 1 "*" H 7725 1950 50  0000 L CNN
 F 2 "Capacitor_THT:C_Disc_D4.3mm_W1.9mm_P5.00mm" H 7738 1900 50  0001 C CNN
@@
 AR Path="/5F79BBF0/6187CB90" Ref="#PWR?"  Part="1"
 AR Path="/5F7B99D0/6187CB90" Ref="#PWR075"  Part="1"
-AR Path="/5F7BF5BB/6187CB90" Ref="#PWR0122"  Part="1"
-F 0 "#PWR0122" H 7700 2050 50  0001 C CNN
+AR Path="/5F7BF5BB/6187CB90" Ref="#PWR0115"  Part="1"
+F 0 "#PWR0115" H 7700 2050 50  0001 C CNN
 F 1 "GND" H 7700 2150 50  0000 C CNN
 F 2 "" H 7700 2300 50  0001 C CNN
@@
 AR Path="/5B53AFFA/7760FCCC" Ref="TP5"  Part="1"
 AR Path="/5F7B99D0/7760FCCC" Ref="TP27"  Part="1"
-AR Path="/5F7BF5BB/7760FCCC" Ref="TP42"  Part="1"
-F 0 "TP42" H 7508 1868 50  0000 L CNN
+AR Path="/5F7BF5BB/7760FCCC" Ref="TP41"  Part="1"
+F 0 "TP41" H 7508 1868 50  0000 L CNN
 F 1 "REG-I" H 7508 1777 50  0000 L CNN
 F 2 "TestPoint:TestPoint_Pad_1.0x1.0mm" H 7650 1750 50  0001 C CNN
@@
 AR Path="/5B53AFFA/7761CD67" Ref="TP4"  Part="1"
 AR Path="/5F7B99D0/7761CD67" Ref="TP26"  Part="1"
-AR Path="/5F7BF5BB/7761CD67" Ref="TP41"  Part="1"
-F 0 "TP41" H 4858 3674 50  0000 L CNN
+AR Path="/5F7BF5BB/7761CD67" Ref="TP40"  Part="1"
+F 0 "TP40" H 4858 3674 50  0000 L CNN
 F 1 "~REG-O" H 4858 3576 50  0000 L CNN
 F 2 "TestPoint:TestPoint_Pad_1.0x1.0mm" H 5000 3550 50  0001 C CNN
