File: MK1_CPU/8bit-computer/clock.sch (KiCad schematic (older format))
At the start: 24 parts, among them SW1 SW_Push, SW2 SW_NKK_GW12LHP, U3 LM555, U4 74LS04, U5 74LS08, U6 LM555, U7 74LS32, U8 LM555

Commit message: version 2.0
Parts:
- added C4: 0.1µF, Capacitor_THT:C_Disc_D4.3mm_W1.9mm_P5.00mm, symbol Device:C
- added C7: 1µF, Capacitor_THT:CP_Radial_D5.0mm_P2.00mm, symbol Device:CP1
- added D9: GREEN, LED_THT:LED_D3.0mm, symbol Device:LED_ALT
- added R5, R7: 1K, Resistor_THT:R_Axial_DIN0207_L6.3mm_D2.5mm_P7.62mm_Horizontal, symbol Device:R
- added SW1: Multiplier, Button_Switch_THT:SW_DIP_SPSTx03_Slide_9.78x9.8mm_W7.62mm_P2.54mm, symbol Switch:SW_DIP_x03
- added TP1: CLK_IN, TestPoint:TestPoint_Pad_1.0x1.0mm, symbol Connector:TestPoint
- added TP2: CLK, TestPoint:TestPoint_Pad_1.0x1.0mm, symbol Connector:TestPoint
- added TP3: ~CLK, TestPoint:TestPoint_Pad_1.0x1.0mm, symbol Connector:TestPoint
- added unit 3 of U2
- C10: renamed from C8; footprint Capacitor_THT:C_Rect_L7.0mm_W6.0mm_P5.00mm -> Capacitor_THT:C_Disc_D4.3mm_W1.9mm_P5.00mm
- C5: value 0.1µF -> 0.01µF; footprint Capacitor_THT:C_Rect_L7.0mm_W6.0mm_P5.00mm -> Capacitor_THT:C_Disc_D4.3mm_W1.9mm_P5.00mm
- C9: renamed from C7; footprint Capacitor_THT:C_Rect_L7.0mm_W6.0mm_P5.00mm -> Capacitor_THT:C_Disc_D4.3mm_W1.9mm_P5.00mm
- R1: renamed from R17; value 1K -> 220
- R2: renamed from R18; value 1K -> 220
- R4: renamed from R20; value 1M -> 330K
- R9: renamed from R23; value 220 -> 1K
- SW2: renamed from SW1; value SW_Push -> Pulse
- SW3: renamed from SW2; value SW_NKK_GW12LHP -> Manual
- U2: renamed from U7; value 74LS32 -> 74HCT32; footprint Package_DIP:DIP-14_W7.62mm_Socket -> Package_DIP:DIP-14_W7.62mm; symbol 8bit-computer-rescue:74LS32 -> 8bit-computer-rescue:74HCT32
- U3, U6: value LM555 -> NE555; footprint Package_DIP:DIP-8_W7.62mm_Socket -> Package_DIP:DIP-8_W7.62mm
- U4: value 74LS04 -> 74HCT04; footprint Package_DIP:DIP-14_W7.62mm_Socket -> Package_DIP:DIP-14_W7.62mm; symbol 8bit-computer-rescue:74LS04 -> 8bit-computer-rescue:74HCT04
- U5: value 74LS08 -> 74HCT08; footprint Package_DIP:DIP-14_W7.62mm_Socket -> Package_DIP:DIP-14_W7.62mm; symbol 8bit-computer-rescue:74LS08 -> 8bit-computer-rescue:74HCT08
- U7: renamed from U8; value LM555 -> NE555; footprint Package_DIP:DIP-8_W7.62mm_Socket -> Package_DIP:DIP-8_W7.62mm
- renumbered C4 to C6, C6 to C8, D9 to D10, R19 to R3, R21 to R6, R22 to R8
Connections:
- net labels added: CLK_IN
- wire segments 128 -> 157
Other:
- moved on the sheet: C2, C3, D10, R9

Commit message: revision 2.0d
Parts:
- renumbered C9 to C10, C10 to C11, C2 to C3, C3 to C4, C4 to C5, C5 to C6, C6 to C7, C7 to C8, C8 to C9
Connections:
- net CLK: now also U2.11; no longer U2.8
- net CLK_IN: now also U2.13; no longer U2.10
- net at U5.3: now also U2.9; no longer U2.4
- net at U5.6: now also U2.10; no longer U2.5
- net at U5.9: now also U2.8; no longer U2.6
- net at U5.8: now also U2.12; no longer U2.9
Changed lines of the file:
@@
 $EndComp
 $Comp
-L Device:C C2
+L Device:C C3
 U 1 1 5B52B714
 P 900 2800
-F 0 "C2" H 925 2900 50  0000 L CNN
+F 0 "C3" H 925 2900 50  0000 L CNN
 F 1 "0.01µF" H 925 2700 50  0000 L CNN
 F 2 "Capacitor_THT:C_Disc_D4.3mm_W1.9mm_P5.00mm" H 938 2650 50  0001 C CNN
@@
 $EndComp
 $Comp
-L Device:C C6
+L Device:C C7
 U 1 1 5B52B758
 P 4150 2550
-F 0 "C6" H 4175 2650 50  0000 L CNN
+F 0 "C7" H 4175 2650 50  0000 L CNN
 F 1 "0.01µF" H 4175 2450 50  0000 L CNN
 F 2 "Capacitor_THT:C_Disc_D4.3mm_W1.9mm_P5.00mm" H 4188 2400 50  0001 C CNN
@@
 $EndComp
 $Comp
-L Device:C C8
+L Device:C C9
 U 1 1 5B52B78B
 P 7400 2600
-F 0 "C8" H 7425 2700 50  0000 L CNN
+F 0 "C9" H 7425 2700 50  0000 L CNN
 F 1 "0.01µF" H 7425 2500 50  0000 L CNN
 F 2 "Capacitor_THT:C_Disc_D4.3mm_W1.9mm_P5.00mm" H 7438 2450 50  0001 C CNN
@@
 $EndComp
 $Comp
-L Device:CP1 C3
+L Device:CP1 C4
 U 1 1 5B52B85D
 P 1300 2800
-F 0 "C3" H 1325 2900 50  0000 L CNN
+F 0 "C4" H 1325 2900 50  0000 L CNN
 F 1 "1µF" H 1325 2700 50  0000 L CNN
 F 2 "Capacitor_THT:CP_Radial_D5.0mm_P2.00mm" H 1300 2800 50  0001 C CNN
@@
 $Comp
 L 8bit-computer-rescue:74HCT32 U2
-U 2 1 5B52B9E8
+U 3 1 5B52B9E8
 P 5600 4600
 F 0 "U2" H 5600 4650 50  0000 C CNN
@@
 F 2 "Package_DIP:DIP-14_W7.62mm" H 5600 4600 50  0001 C CNN
 F 3 "" H 5600 4600 50  0001 C CNN
-	2    5600 4600
+	3    5600 4600
 	1    0    0    -1
 $EndComp
@@
 ~CLK
 $Comp
-L Device:C C10
+L Device:C C11
 U 1 1 5B52B80F
 P 9900 1600
-F 0 "C10" H 9925 1700 50  0000 L CNN
+F 0 "C11" H 9925 1700 50  0000 L CNN
 F 1 "0.1µF" H 9925 1500 50  0000 L CNN
 F 2 "Capacitor_THT:C_Disc_D4.3mm_W1.9mm_P5.00mm" H 9938 1450 50  0001 C CNN
@@
 	2950 2200 3000 2200
 $Comp
-L Device:C C9
+L Device:C C10
 U 1 1 5B64C674
 P 9600 1600
-F 0 "C9" H 9625 1700 50  0000 L CNN
+F 0 "C10" H 9625 1700 50  0000 L CNN
 F 1 "0.1µF" H 9625 1500 50  0000 L CNN
 F 2 "Capacitor_THT:C_Disc_D4.3mm_W1.9mm_P5.00mm" H 9638 1450 50  0001 C CNN
@@
 	1300 2650 1300 2600
 $Comp
-L Device:C C5
+L Device:C C6
 U 1 1 5E7EE4BF
 P 1800 2800
-F 0 "C5" H 1825 2900 50  0000 L CNN
+F 0 "C6" H 1825 2900 50  0000 L CNN
 F 1 "0.01µF" H 1825 2700 50  0000 L CNN
 F 2 "Capacitor_THT:C_Disc_D4.3mm_W1.9mm_P5.00mm" H 1838 2650 50  0001 C CNN
@@
 	1300 2600 1550 2600
 $Comp
-L Device:C C4
+L Device:C C5
 U 1 1 5E81078A
 P 1550 2800
-F 0 "C4" H 1575 2900 50  0000 L CNN
+F 0 "C5" H 1575 2900 50  0000 L CNN
 F 1 "0.1µF" H 1575 2700 50  0000 L CNN
 F 2 "Capacitor_THT:C_Disc_D4.3mm_W1.9mm_P5.00mm" H 1588 2650 50  0001 C CNN
@@
 	1550 3150 1550 3200
 $Comp
-L Device:CP1 C7
+L Device:CP1 C8
 U 1 1 5E83FD17
 P 5500 2550
-F 0 "C7" H 5525 2650 50  0000 L CNN
+F 0 "C8" H 5525 2650 50  0000 L CNN
 F 1 "1µF" H 5525 2450 50  0000 L CNN
 F 2 "Capacitor_THT:CP_Radial_D5.0mm_P2.00mm" H 5500 2550 50  0001 C CNN
@@
 $Comp
 L 8bit-computer-rescue:74HCT32 U2
-U 3 1 5EB34DA9
+U 4 1 5EB34DA9
 P 8300 4800
 F 0 "U2" H 8300 4850 50  0000 C CNN
@@
 F 2 "Package_DIP:DIP-14_W7.62mm" H 8300 4800 50  0001 C CNN
 F 3 "" H 8300 4800 50  0001 C CNN
-	3    8300 4800
-	1    0    0    -1
-$EndComp
+	4    8300 4800
+	1    0    0    -1
+$EndComp
