File: MK1_CPU/8bit-computer/control.sch (KiCad schematic (older format))
At the start: 73 parts, among them SW6 Reset, U13 74LS00, U4 74LS04, U41 74LS00, U42 74LS161, U43 74LS138, U44 AM29F040, U45 AM29F040, U46 AM29F040, U47 74LS04

Commit message: version 2.0
Parts:
- removed D40, D41, D42, D43: GREEN, LED_THT:LED_D3.0mm, symbol Device:LED_ALT
- removed R56, R57, R58, R59, R60, R61, R62, R63, R64, R65, R66, R67, R68, R69, R70, R71, R72, R73, R74, R75, R76, R77, R78, R79, R80, R81, R82, R83, R84, R85: 220, Resistor_THT:R_Axial_DIN0207_L6.3mm_D2.5mm_P7.62mm_Horizontal, symbol Device:R
- removed U13, U41: 74LS00, Package_DIP:DIP-14_W7.62mm_Socket, symbol 8bit-computer-rescue:74LS00
- removed unit 5 of U4
- removed unit 6 of U4
- removed U43: 74LS138, Package_DIP:DIP-16_W7.62mm_Socket, symbol 8bit-computer-rescue:74LS138
- removed unit 1 of U47
- removed unit 2 of U47
- added D106, D110, D112, D114, D116, D118, D120, D122, D138, D139: BLUE, LED_THT:LED_D3.0mm, symbol Device:LED_ALT
- added D98: YELLOW, LED_THT:LED_D3.0mm, symbol Device:LED_ALT
- added JP1: RST_EN, Jumper:SolderJumper-2_P1.3mm_Open_RoundedPad1.0x1.5mm, symbol Jumper:SolderJumper_2_Open
- added JP2: 6-STAGES, Jumper:SolderJumper-2_P1.3mm_Bridged_RoundedPad1.0x1.5mm, symbol Jumper:SolderJumper_2_Bridged
- added R25: 10K, Resistor_THT:R_Axial_DIN0207_L6.3mm_D2.5mm_P7.62mm_Horizontal, symbol Device:R
- added RN13, RN14, RN15, RN16, RN17, RN18, RN19: 1K, Resistor_THT:R_Array_SIP9, symbol Device:R_Network08
- added TP40: ~CU_EN, TestPoint:TestPoint_Pad_1.0x1.0mm, symbol Connector:TestPoint
- added U23: 74HCT86, Package_DIP:DIP-14_W7.62mm, symbol 8bit-computer-rescue:74HCT86
- added unit 2 of U63
- added unit 3 of U63
- added U74: 74HCT08, Package_DIP:DIP-14_W7.62mm, symbol 8bit-computer-rescue:74HCT08
- added U80: AM29F040, Housings_LCC:PLCC-32_THT-Socket, symbol 8bit-computer-rescue:AM29F040
- added U81: 74HCT138, Package_DIP:DIP-16_W7.62mm, symbol 8bit-computer-rescue:74HCT138
- added U82, U83: 74HCT238, Package_DIP:DIP-16_W7.62mm, symbol 74xx_IEEE:74HC238
- added unit 4 of U84
- C39: renamed from C17; footprint Capacitor_THT:C_Rect_L7.0mm_W6.0mm_P5.00mm -> Capacitor_THT:C_Disc_D4.3mm_W1.9mm_P5.00mm
- C40: renamed from C18; footprint Capacitor_THT:C_Rect_L7.0mm_W6.0mm_P5.00mm -> Capacitor_THT:C_Disc_D4.3mm_W1.9mm_P5.00mm
- D100: renamed from D39; value GREEN -> YELLOW
- D99: renamed from D38; value GREEN -> YELLOW
- R36: renamed from R55; value 1K -> 10K
- U63, U84: renamed from U47; value 74LS04 -> 74HCT04; footprint Package_DIP:DIP-14_W7.62mm_Socket -> Package_DIP:DIP-14_W7.62mm; symbol 8bit-computer-rescue:74LS04 -> 8bit-computer-rescue:74HCT04
- U63: renamed from U4; value 74LS04 -> 74HCT04; footprint Package_DIP:DIP-14_W7.62mm_Socket -> Package_DIP:DIP-14_W7.62mm; symbol 8bit-computer-rescue:74LS04 -> 8bit-computer-rescue:74HCT04
- U75: renamed from U42; value 74LS161 -> 74HCT161; footprint Package_DIP:DIP-16_W7.62mm_Socket -> Package_DIP:DIP-16_W7.62mm; symbol 8bit-computer-rescue:74LS161 -> 8bit-computer-rescue:74HCT161
- renumbered D44 to D105, D45 to D107, D46 to D109, D47 to D111, D48 to D113, D49 to D115, D50 to D117, D51 to D119, D52 to D121, D53 to D123, D54 to D124, D55 to D125, D56 to D126, D57 to D127, D58 to D128, D59 to D129, D60 to D130, D61 to D131, D62 to D132, D63 to D133, D64 to D134, D65 to D135, D66 to D136, D67 to D137, SW6 to SW10, U44 to U77, U45 to U78, U46 to U79
Connections:
- net labels added: CI, CLR_IN, DI, E0, E1, EI, EXT_I, IRQ0, IRQ1, NOT, PE, SD, SUB, U0, U1, ~BO, ~CU_EN, ~DO, ~PI, ~PO, ~SO
- net labels removed: CE, SO, ~J
- wire segments 470 -> 811
- no-connect marks 7 -> 14
Other:
- note added: "AI"
- note added: "AND"
- note added: "AO"
- note added: "BI"
- note added: "BO"
- note added: "CI"
- note added: "CO"
- note added: "DI"
- note added: "DO"
- note added: "E0"
- note added: "E1"
- note added: "EI"
- note added: "EO"
- note added: "HLT"
- note added: "II"
- note added: "IO"
- note added: "MI"
- note added: "NOT"
- note added: "OI"
- note added: "OR"
- note added: "PE"
- note added: "PI"
- note added: "PO"
- note added: "RI"
- note added: "RO"
- note added: "ROT"
- note added: "SD"
- note added: "SHF"
- note added: "SI"
- note added: "SO"
- note added: "SU"
- note added: "SUB"
- note added: "U0"
- note added: "U1"
- moved on the sheet: D100, D105, D107, D109, D111, D113, D115, D117, D119, D121, D123, D124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

Commit message: 2.0b hardware revision
Parts:
- removed JP1: RST_EN, Jumper:SolderJumper-2_P1.3mm_Open_RoundedPad1.0x1.5mm, symbol Jumper:SolderJumper_2_Open
- removed JP2: 6-STAGES, Jumper:SolderJumper-2_P1.3mm_Bridged_RoundedPad1.0x1.5mm, symbol Jumper:SolderJumper_2_Bridged
- removed R25: 10K, Resistor_THT:R_Axial_DIN0207_L6.3mm_D2.5mm_P7.62mm_Horizontal, symbol Device:R
- removed unit 4 of U63
- removed U74: 74HCT08, Package_DIP:DIP-14_W7.62mm, symbol 8bit-computer-rescue:74HCT08
- added C44: 0.01µF, Capacitor_THT:C_Disc_D4.3mm_W1.9mm_P5.00mm, symbol Device:C
Connections:
- net GND: now also C44.2
- net RGT: now also U80.18 (D4); no longer U83.9 (Y6)
- net ~CLR: now also U23.5 (IN2)
- net at U80.13 (D0): now also RN13.9 (R8), U23.4 (IN1), C44.1
Changed lines of the file:
@@
 	4600 4350 4000 4350
 Wire Wire Line
-	3200 3300 3400 3300
-Connection ~ 3400 3300
-Wire Wire Line
-	3200 3500 3500 3500
-Connection ~ 3500 3500
-Wire Wire Line
 	3400 1950 3400 3000
 Wire Wire Line
@@
 Wire Wire Line
 	3600 3950 3600 6500
-Wire Wire Line
-	3400 3300 3400 3750
-Wire Wire Line
-	3500 3500 3500 3850
 Wire Wire Line
 	3300 850  4600 850
@@
 	4500 3050 5600 3050
 Connection ~ 5600 3050
-Text HLabel 10650 6950 2    60   Output ~ 0
+Text HLabel 9950 9750 2    60   Output ~ 0
 RGT
 Text HLabel 10650 2650 2    60   Output ~ 0
@@
 $EndComp
 Wire Wire Line
-	2850 4350 2850 5250
-Wire Wire Line
 	1200 8200 1200 8800
-Wire Wire Line
-	2400 6650 2850 6650
 Connection ~ 2300 7800
 Wire Wire Line
@@
 	1600 7250 1600 7350
 Wire Wire Line
-	950  8450 950  8350
+	950  8450 950  8400
 $Comp
 L power:GND #PWR099
@@
 Wire Wire Line
 	800  4700 800  2850
-Wire Wire Line
-	700  6750 700  5900
 Wire Wire Line
 	5850 6050 5850 8650
@@
 	8500 9650 8500 9150
 Wire Wire Line
-	8600 9750 9200 9750
-Wire Wire Line
 	8700 9850 9200 9850
 Wire Wire Line
@@
 Wire Wire Line
 	10450 9500 10650 9500
-NoConn ~ 9200 9750
 NoConn ~ 9200 9850
 NoConn ~ 9200 9950
@@
 Wire Wire Line
 	1750 1050 2100 1050
-Wire Wire Line
-	900  6050 900  5900
-$Comp
-L Jumper:SolderJumper_2_Open JP1
-U 1 1 76AA61F3
-P 2100 6050
-F 0 "JP1" H 2100 6255 50  0000 C CNN
-F 1 "RST_EN" H 2100 6164 50  0000 C CNN
-F 2 "Jumper:SolderJumper-2_P1.3mm_Open_RoundedPad1.0x1.5mm" H 2100 6050 50  0001 C CNN
-F 3 "~" H 2100 6050 50  0001 C CNN
-	1    2100 6050
-	1    0    0    -1
-$EndComp
-Wire Wire Line
-	2250 6050 5850 6050
-Wire Wire Line
-	900  6050 1950 6050
-$Comp
-L Jumper:SolderJumper_2_Bridged JP2
-U 1 1 771B8E30
-P 2850 5400
-F 0 "JP2" H 2850 5605 50  0000 C CNN
-F 1 "6-STAGES" H 2850 5514 50  0000 C CNN
-F 2 "Jumper:SolderJumper-2_P1.3mm_Bridged_RoundedPad1.0x1.5mm" H 2850 5400 50  0001 C CNN
-F 3 "~" H 2850 5400 50  0001 C CNN
-	1    2850 5400
-	0    -1   -1   0
-$EndComp
-Wire Wire Line
-	2850 6650 2850 6400
 $Comp
 L Connector:TestPoint TP?
@@
 Wire Wire Line
 	8500 600  10200 600
-$Comp
-L Device:R R25
-U 1 1 78B5F375
-P 2650 6400
-F 0 "R25" V 2730 6400 50  0000 C CNN
-F 1 "10K" V 2650 6400 50  0000 C CNN
-F 2 "Resistor_THT:R_Axial_DIN0207_L6.3mm_D2.5mm_P7.62mm_Horizontal" V 2580 6400 50  0001 C CNN
-F 3 "" H 2650 6400 50  0001 C CNN
-	1    2650 6400
-	0    -1   -1   0
-$EndComp
-Wire Wire Line
-	2800 6400 2850 6400
-Connection ~ 2850 6400
-Wire Wire Line
-	2850 6400 2850 5550
-$Comp
-L power:VCC #PWR0123
-U 1 1 78CAE6D6
-P 2450 6300
-F 0 "#PWR0123" H 2450 6150 50  0001 C CNN
-F 1 "VCC" H 2450 6450 50  0000 C CNN
-F 2 "" H 2450 6300 50  0001 C CNN
-F 3 "" H 2450 6300 50  0001 C CNN
-	1    2450 6300
-	1    0    0    -1
-$EndComp
-Wire Wire Line
-	2450 6300 2450 6400
-Wire Wire Line
-	2450 6400 2500 6400
 NoConn ~ 9000 12000
 Wire Wire Line
 	8350 6850 9250 6850
 Wire Wire Line
-	700  6750 1200 6750
-$Comp
-L 8bit-computer-rescue:74HCT08 U74
-U 2 1 60AB6A7F
-P 1800 6750
-F 0 "U74" H 1800 7116 50  0000 C CNN
-F 1 "74HCT08" H 1800 7025 50  0000 C CNN
-F 2 "Package_DIP:DIP-14_W7.62mm" H 1800 6750 50  0001 C CNN
-F 3 "" H 1800 6750 50  0001 C CNN
-	2    1800 6750
-	-1   0    0    -1
-$EndComp
-Wire Wire Line
 	2400 8800 2600 8800
-Connection ~ 2300 7450
-Wire Wire Line
-	2300 7050 2300 7450
-Wire Wire Line
-	2500 6850 2400 6850
-Wire Wire Line
-	2500 7050 2500 6850
-Wire Wire Line
-	2300 7050 2500 7050
-$Comp
-L 8bit-computer-rescue:74HCT08 U74
-U 4 1 5F44AF9F
-P 2600 3400
-F 0 "U74" H 2600 3766 50  0000 C CNN
-F 1 "74HCT08" H 2600 3675 50  0000 C CNN
-F 2 "Package_DIP:DIP-14_W7.62mm" H 2600 3400 50  0001 C CNN
-F 3 "" H 2600 3400 50  0001 C CNN
-	4    2600 3400
-	-1   0    0    -1
-$EndComp
-$Comp
-L 8bit-computer-rescue:74HCT04 U63
-U 4 1 5B624D8F
-P 1600 3850
-F 0 "U63" H 1795 3965 50  0000 C CNN
-F 1 "74HCT04" H 1790 3725 50  0000 C CNN
-F 2 "Package_DIP:DIP-14_W7.62mm" H 1600 3850 50  0001 C CNN
-F 3 "" H 1600 3850 50  0001 C CNN
-	4    1600 3850
-	0    1    1    0
-$EndComp
 Wire Wire Line
 	3300 1850 3300 2950
-Wire Wire Line
-	1600 3400 2000 3400
-Wire Wire Line
-	1600 4350 1600 4300
-Wire Wire Line
-	1600 4350 2850 4350
 $Comp
 L 8bit-computer-rescue:74HCT86 U23
@@
 Connection ~ 3400 3000
 Wire Wire Line
-	3400 3000 3400 3300
-Wire Wire Line
 	1100 1050 1100 3050
 Wire Wire Line
@@
 Connection ~ 3500 3050
 Wire Wire Line
-	3500 3050 3500 3500
-Wire Wire Line
 	9500 11450 9500 13800
 Wire Wire Line
@@
 	3150 13800 9500 13800
 Wire Wire Line
-	900  6050 550  6050
-Wire Wire Line
 	550  6050 550  1550
-Connection ~ 900  6050
 Wire Wire Line
 	550  1550 2100 1550
@@
 Wire Wire Line
 	8950 3750 8950 3850
+$Comp
+L Device:C C44
+U 1 1 5E9FDDA2
+P 650 6350
+F 0 "C44" H 675 6450 50  0000 L CNN
+F 1 "0.01µF" H 675 6250 50  0000 L CNN
+F 2 "Capacitor_THT:C_Disc_D4.3mm_W1.9mm_P5.00mm" H 688 6200 50  0001 C CNN
+F 3 "" H 650 6350 50  0001 C CNN
+	1    650  6350
+	1    0    0    -1
+$EndComp
+Wire Wire Line
+	650  6200 650  6050
+Wire Wire Line
+	650  6500 650  8400
+Wire Wire Line
+	650  8400 950  8400
+Connection ~ 950  8400
+Wire Wire Line
+	950  8400 950  8350
+Wire Wire Line
+	3400 3000 3400 3750
+Wire Wire Line
+	3500 3050 3500 3850
+Wire Wire Line
+	2300 6750 2300 7450
+Connection ~ 2300 7450
+Connection ~ 650  6050
+Wire Wire Line
+	650  6050 550  6050
+Wire Wire Line
+	650  6050 700  6050
+Wire Wire Line
+	900  5900 900  6750
+Wire Wire Line
+	900  6750 2300 6750
+Wire Wire Line
+	700  5900 700  6050
+Connection ~ 700  6050
+Wire Wire Line
+	700  6050 5850 6050
+Wire Wire Line
+	8600 9750 9950 9750
+NoConn ~ 10650 6950
 $EndSCHEMATC

Commit message: revision 2.0d
Parts:
- removed unit 6 of U63
- added R30, R31, R32: 10K, Resistor_THT:R_Axial_DIN0207_L6.3mm_D2.5mm_P7.62mm_Horizontal, symbol Device:R
- renumbered C44 to C39, C39 to C40, C40 to C41, D113 to D100, D114 to D101, D115 to D102, D116 to D103, D117 to D104, D118 to D105, D119 to D106, D120 to D107, D121 to D108, D122 to D109, D123 to D110, D124 to D111, D125 to D112, D126 to D113, D127 to D114, D128 to D115, D129 to D116, D130 to D117, D131 to D118, D132 to D119, D133 to D120, D134 to D121, D135 to D122, D136 to D123, D137 to D124, D138 to D125, D139 to D126, D98 to D90, D99 to D91, D100 to D92, D105 to D93, D106 to D94, D107 to D95, D109 to D96, D110 to D97, D111 to D98, D112 to D99, R36 to R29, TP40 to TP39, U23 to U24, U84 to U60, U63 to U60, U75 to U72, U77 to U73, U78 to U74, U79 to U75, U80 to U76, U81 to U77, U82 to U78, U83 to U79
Connections:
- net GND: now also R30.2, R31.2, R32.2
- net OI: now also R32.1
- net SD: now also R30.1
- net SU: now also R31.1
- net ~PI: now also U60.12; no longer U60.2
- net at D119.2 (A), U78.7 (Y7): now also U60.13; no longer U60.1
- net at U60.9, U75.18 (D4): now also D102.2 (A)
- now unconnected: RN16.5 (R4), U74.13 (D0)
- no-connect marks 14 -> 16
Other:
- note added: "FI"
- note removed: "IO"
