File: MK1_CPU/8bit-computer/inst-register.sch (KiCad schematic (older format))
At the start: 38 parts, among them U55 74LS00, U58 74LS245, U59 74LS273, U60 74LS273, U61 74LS00

Commit message: version 2.0
Parts:
- removed R103, R104, R105, R106, R107, R108, R109, R110, R111, R112, R113, R114, R115, R116, R117, R118: 220, Resistor_THT:R_Axial_DIN0207_L6.3mm_D2.5mm_P7.62mm_Horizontal, symbol Device:R
- removed U55, U61: 74LS00, Package_DIP:DIP-14_W7.62mm_Socket, symbol 8bit-computer-rescue:74LS00
- added C34, C35: *, Capacitor_THT:C_Disc_D4.3mm_W1.9mm_P5.00mm, symbol Device:C
- added RN11: 220, Resistor_THT:R_Array_SIP9, symbol Device:R_Network08
- added RN12: 1K, Resistor_THT:R_Array_SIP9, symbol Device:R_Network08
- added TP28: ~IO, TestPoint:TestPoint_Pad_1.0x1.0mm, symbol Connector:TestPoint
- added TP29: II, TestPoint:TestPoint_Pad_1.0x1.0mm, symbol Connector:TestPoint
- added U58: 74HCT08, Package_DIP:DIP-14_W7.62mm, symbol 8bit-computer-rescue:74HCT08
- added U63: 74HCT04, Package_DIP:DIP-14_W7.62mm, symbol 8bit-computer-rescue:74HCT04
- C36: renamed from C23; footprint Capacitor_THT:C_Rect_L7.0mm_W6.0mm_P5.00mm -> Capacitor_THT:C_Disc_D4.3mm_W1.9mm_P5.00mm
- U60: renamed from U58; value 74LS245 -> 74HCT245; footprint Package_DIP:DIP-20_W7.62mm_Socket -> Package_DIP:DIP-20_W7.62mm; symbol 8bit-computer-rescue:74LS245 -> 8bit-computer-rescue:74HCT245
- U61: renamed from U59; value 74LS273 -> 74HCT273; footprint Package_DIP:DIP-20_W7.62mm_Socket -> Package_DIP:DIP-20_W7.62mm; symbol 8bit-computer-rescue:74LS273 -> 8bit-computer-rescue:74HCT273
- U62: renamed from U60; value 74LS273 -> 74HCT273; footprint Package_DIP:DIP-20_W7.62mm_Socket -> Package_DIP:DIP-20_W7.62mm; symbol 8bit-computer-rescue:74LS273 -> 8bit-computer-rescue:74HCT273
- renumbered D84 to D72, D85 to D73, D86 to D74, D87 to D75, D88 to D76, D89 to D77, D90 to D78, D91 to D79, D92 to D80, D93 to D81, D94 to D82, D95 to D83, D96 to D84, D97 to D85, D98 to D86, D99 to D87
Connections:
- net labels added: ~CLK
- net labels removed: CLK
- wire segments 241 -> 213

Commit message: 2.0b hardware revision
Parts:
- added C47: 0.01, Capacitor_THT:C_Disc_D4.3mm_W1.9mm_P5.00mm, symbol Device:C
Connections:
- net GND: now also C47.2
- net HL: now also C47.1
Changed lines of the file:
@@
 	10000 2600 10150 2600
 Wire Wire Line
-	8600 3050 10000 3050
+	8600 3050 9400 3050
 Wire Wire Line
 	7400 1800 7400 2850
 Wire Wire Line
 	10000 3050 10000 4200
-Connection ~ 10000 3050
-Wire Wire Line
-	10000 3050 10150 3050
 Wire Wire Line
 	7100 2000 7100 4100
@@
 $EndComp
 Wire Wire Line
-	7250 3250 7250 3350
+	7250 3250 7250 3300
 Wire Wire Line
 	7250 2950 7250 2850
@@
 Wire Wire Line
 	1950 3250 1950 4750
+Connection ~ 10000 3050
+Wire Wire Line
+	10000 3050 10150 3050
+$Comp
+L Device:C C47
+U 1 1 5F13FC24
+P 9400 3250
+F 0 "C47" H 9425 3350 50  0000 L CNN
+F 1 "0.01" H 9425 3150 50  0000 L CNN
+F 2 "Capacitor_THT:C_Disc_D4.3mm_W1.9mm_P5.00mm" H 9438 3100 50  0001 C CNN
+F 3 "" H 9400 3250 50  0001 C CNN
+	1    9400 3250
+	1    0    0    -1
+$EndComp
+Wire Wire Line
+	9400 3400 9400 3500
+Wire Wire Line
+	9400 3100 9400 3050
+Connection ~ 9400 3050
+Wire Wire Line
+	9400 3050 10000 3050
+Wire Wire Line
+	7250 3300 9100 3300
+Wire Wire Line
+	9100 3300 9100 3500
+Wire Wire Line
+	9100 3500 9400 3500
+Connection ~ 7250 3300
+Wire Wire Line
+	7250 3300 7250 3350
 $EndSCHEMATC

Commit message: revision 2.0d
Parts:
- removed C34, C35: *, Capacitor_THT:C_Disc_D4.3mm_W1.9mm_P5.00mm, symbol Device:C
- removed C47: 0.01, Capacitor_THT:C_Disc_D4.3mm_W1.9mm_P5.00mm, symbol Device:C
- removed D72, D73, D74, D75, D76, D77, D78, D79: YELLOW, LED_THT:LED_D3.0mm, symbol Device:LED_ALT
- removed RN11: 220, Resistor_THT:R_Array_SIP9, symbol Device:R_Network08
- removed TP28: ~IO, TestPoint:TestPoint_Pad_1.0x1.0mm, symbol Connector:TestPoint
- removed unit 2 of U58
- removed unit 3 of U58
- removed U60: 74HCT245, Package_DIP:DIP-20_W7.62mm, symbol 8bit-computer-rescue:74HCT245
- removed U62: 74HCT273, Package_DIP:DIP-20_W7.62mm, symbol 8bit-computer-rescue:74HCT273
- removed U63: 74HCT04, Package_DIP:DIP-14_W7.62mm, symbol 8bit-computer-rescue:74HCT04
- renumbered D80 to D72, D81 to D73, D82 to D74, D83 to D75, D84 to D76, D85 to D77, D86 to D78, D87 to D79, RN12 to RN11, TP29 to TP28
Connections:
- net II: now also U58.5; no longer U58.13
- net ~CLK: now also U58.4; no longer U58.12
- net at U61.11 (Cp): now also TP28.1, U58.6
Other:
- moved on the sheet: D72, D73, D74, D75, D76, D77, D78, D79, RN11, TP28
