File: MK1_CPU/8bit-computer/mar.sch (KiCad schematic (older format))
At the start: 27 parts, among them SW3 SW_NKK_GW12LHP, SW4 SW_DIP_x08, U26 74LS08, U28 74LS157, U29 74LS157, U30 74LS273

Commit message: version 2.0
Parts:
- removed D33: GREEN, LED_THT:LED_D3.0mm, symbol Device:LED_ALT
- removed R42, R43, R44, R45, R46, R48, R50, R51: 220, Resistor_THT:R_Axial_DIN0207_L6.3mm_D2.5mm_P7.62mm_Horizontal, symbol Device:R
- removed R49: 1K, Resistor_THT:R_Axial_DIN0207_L6.3mm_D2.5mm_P7.62mm_Horizontal, symbol Device:R
- removed SW3: SW_NKK_GW12LHP, Button_Switch_THT:SW_NKK_GW12LJP, symbol 8bit-computer-rescue:SW_NKK_GW12LHP
- removed SW4: SW_DIP_x08, Button_Switch_THT:SW_DIP_SPSTx08_Slide_9.78x22.5mm_W7.62mm_P2.54mm, symbol 8bit-computer-rescue:SW_DIP_x08-8bit-computer-rescue
- added C16: *, Capacitor_THT:C_Disc_D4.3mm_W1.9mm_P5.00mm, symbol Device:C
- added R12: 10K, Resistor_THT:R_Axial_DIN0207_L6.3mm_D2.5mm_P7.62mm_Horizontal, symbol Device:R
- added R14, R15: 1K, Resistor_THT:R_Axial_DIN0207_L6.3mm_D2.5mm_P7.62mm_Horizontal, symbol Device:R
- added RN5: 470, Resistor_THT:R_Array_SIP9, symbol Device:R_Network08
- added SW4: Prog, Button_Switch_THT:SW_DIP_SPSTx01_Slide_9.78x4.72mm_W7.62mm_P2.54mm, symbol Switch:SW_DIP_x01
- added SW5: Address, Button_Switch_THT:SW_DIP_SPSTx10_Slide_9.78x27.58mm_W7.62mm_P2.54mm, symbol Switch:SW_DIP_x10
- added TP15: MI, TestPoint:TestPoint_Pad_1.0x1.0mm, symbol Connector:TestPoint
- added U84: 74HCT04, Package_DIP:DIP-14_W7.62mm, symbol 8bit-computer-rescue:74HCT04
- C17: renamed from C12; footprint Capacitor_THT:C_Rect_L7.0mm_W6.0mm_P5.00mm -> Capacitor_THT:C_Disc_D4.3mm_W1.9mm_P5.00mm
- D29: renamed from D28; value YELLOW -> RED
- D30: renamed from D29; value YELLOW -> RED
- D31: renamed from D30; value YELLOW -> RED
- D32: renamed from D31; value YELLOW -> RED
- D34, D35, D36, D37: value YELLOW -> RED
- R13: renamed from R47; value 1K -> 470
- U29: renamed from U28; footprint Package_DIP:DIP-16_W7.62mm_Socket -> Package_DIP:DIP-16_W7.62mm; symbol 8bit-computer-rescue:74LS157 -> 8bit-computer-rescue:74HCT157
- U30: renamed from U29; footprint Package_DIP:DIP-16_W7.62mm_Socket -> Package_DIP:DIP-16_W7.62mm; symbol 8bit-computer-rescue:74LS157 -> 8bit-computer-rescue:74HCT157
- U31: renamed from U30; value 74LS273 -> 74HCT273; footprint Package_DIP:DIP-20_W7.62mm_Socket -> Package_DIP:DIP-20_W7.62mm; symbol 8bit-computer-rescue:74LS273 -> 8bit-computer-rescue:74HCT273
- U32: renamed from U26; value 74LS08 -> 74HCT08; footprint Package_DIP:DIP-14_W7.62mm_Socket -> Package_DIP:DIP-14_W7.62mm; symbol 8bit-computer-rescue:74LS08 -> 8bit-computer-rescue:74HCT08
- renumbered D32 to D33
Connections:
- net labels added: HL, STK, ~PROG
- net labels removed: PROG
- wire segments 186 -> 197

Commit message: 2.0b hardware revision
Parts:
- removed unit 3 of U84
- added unit 4 of U32
- added unit 3 of U32
- C16: value * -> 0.01
Connections:
- net GND: now also U32.7 (GND), U32.7 (GND)
- net HL: now also U32.8; no longer U84.4
- net STK: now also U32.11
- net VCC: now also R13.2, U32.14 (VCC), U32.14 (VCC); no longer R13.1
- net ~PROG: now also U84.3
- net at D33.2 (A): now also R13.1; no longer R13.2
- net at R14.2, SW5.20: now also U32.9; no longer U84.3
- net at R15.2, SW5.11: now also U32.12
- new net: U32.10, U32.13, U84.4
Other:
- moved on the sheet: D33, R13, R14, SW4, U84B
Changed lines of the file:
@@
 L Device:LED_ALT D33
 U 1 1 5B56564B
-P 2050 4650
-F 0 "D33" H 2050 4750 50  0000 C CNN
-F 1 "RED" H 2050 4550 50  0000 C CNN
-F 2 "LED_THT:LED_D3.0mm" H 2050 4650 50  0001 C CNN
-F 3 "" H 2050 4650 50  0001 C CNN
-	1    2050 4650
-	1    0    0    -1
-$EndComp
-Wire Wire Line
-	1600 4700 1750 4700
-Wire Wire Line
-	1750 4700 1750 4650
-Wire Wire Line
-	1750 4650 1900 4650
+P 2250 4650
+F 0 "D33" H 2250 4750 50  0000 C CNN
+F 1 "RED" H 2250 4550 50  0000 C CNN
+F 2 "LED_THT:LED_D3.0mm" H 2250 4650 50  0001 C CNN
+F 3 "" H 2250 4650 50  0001 C CNN
+	1    2250 4650
+	1    0    0    -1
+$EndComp
+Wire Wire Line
+	1600 4650 1750 4650
+Wire Wire Line
+	1750 4650 2100 4650
 $Comp
 L Device:R R13
 U 1 1 5B565870
-P 2400 4350
-F 0 "R13" V 2480 4350 50  0000 C CNN
-F 1 "470" V 2400 4350 50  0000 C CNN
-F 2 "Resistor_THT:R_Axial_DIN0207_L6.3mm_D2.5mm_P7.62mm_Horizontal" V 2330 4350 50  0001 C CNN
-F 3 "" H 2400 4350 50  0001 C CNN
-	1    2400 4350
-	1    0    0    -1
-$EndComp
-Wire Wire Line
-	2400 4500 2400 4650
+P 2800 4650
+F 0 "R13" V 2880 4650 50  0000 C CNN
+F 1 "470" V 2800 4650 50  0000 C CNN
+F 2 "Resistor_THT:R_Axial_DIN0207_L6.3mm_D2.5mm_P7.62mm_Horizontal" V 2730 4650 50  0001 C CNN
+F 3 "" H 2800 4650 50  0001 C CNN
+	1    2800 4650
+	0    -1   -1   0
+$EndComp
 $Comp
 L power:GND #PWR026
 U 1 1 5B565911
-P 1000 4800
-F 0 "#PWR026" H 1000 4550 50  0001 C CNN
-F 1 "GND" H 1000 4650 50  0000 C CNN
-F 2 "" H 1000 4800 50  0001 C CNN
-F 3 "" H 1000 4800 50  0001 C CNN
-	1    1000 4800
-	1    0    0    -1
-$EndComp
-Wire Wire Line
-	1000 4800 1000 4700
+P 1000 4750
+F 0 "#PWR026" H 1000 4500 50  0001 C CNN
+F 1 "GND" H 1000 4600 50  0000 C CNN
+F 2 "" H 1000 4750 50  0001 C CNN
+F 3 "" H 1000 4750 50  0001 C CNN
+	1    1000 4750
+	1    0    0    -1
+$EndComp
+Wire Wire Line
+	1000 4750 1000 4650
 $Comp
 L power:VCC #PWR028
 U 1 1 5B565949
-P 2550 4000
-F 0 "#PWR028" H 2550 3850 50  0001 C CNN
-F 1 "VCC" H 2550 4150 50  0000 C CNN
-F 2 "" H 2550 4000 50  0001 C CNN
-F 3 "" H 2550 4000 50  0001 C CNN
-	1    2550 4000
-	1    0    0    -1
-$EndComp
-Wire Wire Line
-	2400 4200 2400 4100
-Wire Wire Line
-	2400 4100 2550 4100
-Wire Wire Line
-	2550 4000 2550 4100
-Connection ~ 2550 4100
+P 4200 4550
+F 0 "#PWR028" H 4200 4400 50  0001 C CNN
+F 1 "VCC" H 4200 4700 50  0000 C CNN
+F 2 "" H 4200 4550 50  0001 C CNN
+F 3 "" H 4200 4550 50  0001 C CNN
+	1    4200 4550
+	1    0    0    -1
+$EndComp
+Wire Wire Line
+	4200 4550 4200 4650
 Wire Wire Line
 	3800 3600 3800 4100
@@
 $EndComp
 Wire Wire Line
-	2200 4650 2400 4650
-Wire Wire Line
-	3500 3700 4700 3700
-Wire Wire Line
 	3200 2000 3200 2100
 Connection ~ 4500 2000
@@
 Text HLabel 10150 4450 2    60   Input ~ 0
 ~CLR
-Text HLabel 3800 4750 2    60   Output ~ 0
-~PROG
-Wire Wire Line
-	3500 4750 3800 4750
 $Comp
 L Device:C C17
@@
 	3750 1700 6600 1700
 Wire Wire Line
-	3500 3700 3500 4750
-Wire Wire Line
 	1750 4650 1750 3700
-Wire Wire Line
-	1750 3700 3500 3700
 Connection ~ 1750 4650
-Connection ~ 3500 3700
 Wire Wire Line
 	4300 3900 7050 3900
@@
 Wire Wire Line
 	7650 3600 8000 3600
-Text HLabel 1050 5600 0    60   Output ~ 0
+Text HLabel 1050 6150 0    60   Output ~ 0
 HL
 $Comp
@@
 	5800 5600 5700 5600
 Wire Wire Line
-	3250 5600 3250 6050
-Wire Wire Line
 	5900 6050 5900 5550
-Wire Wire Line
-	3250 6050 4200 6050
 $Comp
 L Device:R R14
 U 1 1 60388B79
-P 4200 5900
-F 0 "R14" V 4280 5900 50  0000 C CNN
-F 1 "1K" V 4200 5900 50  0000 C CNN
-F 2 "Resistor_THT:R_Axial_DIN0207_L6.3mm_D2.5mm_P7.62mm_Horizontal" V 4130 5900 50  0001 C CNN
-F 3 "" H 4200 5900 50  0001 C CNN
-	1    4200 5900
-	1    0    0    -1
-$EndComp
-Text HLabel 2450 5050 0    60   Output ~ 0
+P 4200 5800
+F 0 "R14" V 4280 5800 50  0000 C CNN
+F 1 "1K" V 4200 5800 50  0000 C CNN
+F 2 "Resistor_THT:R_Axial_DIN0207_L6.3mm_D2.5mm_P7.62mm_Horizontal" V 4130 5800 50  0001 C CNN
+F 3 "" H 4200 5800 50  0001 C CNN
+	1    4200 5800
+	1    0    0    -1
+$EndComp
+Text HLabel 1050 5650 0    60   Output ~ 0
 STK
 $Comp
@@
 P 8500 5400
 F 0 "C16" H 8525 5500 50  0000 L CNN
-F 1 "*" H 8525 5300 50  0000 L CNN
+F 1 "0.01" H 8525 5300 50  0000 L CNN
 F 2 "Capacitor_THT:C_Disc_D4.3mm_W1.9mm_P5.00mm" H 8538 5250 50  0001 C CNN
 F 3 "" H 8500 5400 50  0001 C CNN
@@
 L Switch:SW_DIP_x01 SW4
 U 1 1 78059831
-P 1300 4700
-F 0 "SW4" H 1300 4967 50  0000 C CNN
-F 1 "Prog" H 1300 4876 50  0000 C CNN
-F 2 "Button_Switch_THT:SW_DIP_SPSTx01_Slide_9.78x4.72mm_W7.62mm_P2.54mm" H 1300 4700 50  0001 C CNN
-F 3 "~" H 1300 4700 50  0001 C CNN
-	1    1300 4700
+P 1300 4650
+F 0 "SW4" H 1300 4917 50  0000 C CNN
+F 1 "Prog" H 1300 4826 50  0000 C CNN
+F 2 "Button_Switch_THT:SW_DIP_SPSTx01_Slide_9.78x4.72mm_W7.62mm_P2.54mm" H 1300 4650 50  0001 C CNN
+F 3 "~" H 1300 4650 50  0001 C CNN
+	1    1300 4650
 	1    0    0    -1
 $EndComp
@@
 Wire Wire Line
 	5000 4850 5000 4950
-Wire Wire Line
-	3300 4500 3300 4100
-Wire Wire Line
-	2550 4100 3300 4100
 $Comp
 L 8bit-computer-rescue:74HCT04 U84
 U 2 1 5EC4E515
-P 2150 5600
-F 0 "U84" H 2150 5915 50  0000 C CNN
-F 1 "74HCT04" H 2150 5824 50  0000 C CNN
-F 2 "Package_DIP:DIP-14_W7.62mm" H 2150 5600 50  0001 C CNN
-F 3 "" H 2150 5600 50  0001 C CNN
-	2    2150 5600
+P 3400 5750
+F 0 "U84" H 3400 6065 50  0000 C CNN
+F 1 "74HCT04" H 3400 5974 50  0000 C CNN
+F 2 "Package_DIP:DIP-14_W7.62mm" H 3400 5750 50  0001 C CNN
+F 3 "" H 3400 5750 50  0001 C CNN
+	2    3400 5750
 	-1   0    0    -1
 $EndComp
-Wire Wire Line
-	1700 5600 1050 5600
 Connection ~ 4350 5550
 Wire Wire Line
 	4350 5550 5000 5550
-$Comp
-L 8bit-computer-rescue:74HCT04 U84
-U 3 1 5ECE301B
-P 3150 5050
-F 0 "U84" H 3150 5365 50  0000 C CNN
-F 1 "74HCT04" H 3150 5274 50  0000 C CNN
-F 2 "Package_DIP:DIP-14_W7.62mm" H 3150 5050 50  0001 C CNN
-F 3 "" H 3150 5050 50  0001 C CNN
-	3    3150 5050
-	-1   0    0    -1
-$EndComp
-Wire Wire Line
-	2450 5050 2700 5050
-Wire Wire Line
-	3600 5050 3600 5550
-Wire Wire Line
-	3600 5550 4350 5550
 Wire Wire Line
 	4800 3600 4800 4850
@@
 	4350 5450 4350 5550
 Wire Wire Line
-	4350 5150 4350 4500
-Wire Wire Line
-	4350 4500 4200 4500
-Connection ~ 4200 6050
-Wire Wire Line
-	4200 6050 5900 6050
-Wire Wire Line
-	2600 5600 3250 5600
-Wire Wire Line
-	4200 4500 4200 5750
-Connection ~ 4200 4500
-Wire Wire Line
-	4200 4500 3300 4500
+	4350 5150 4350 4650
 Wire Wire Line
 	5000 4850 4800 4850
@@
 Wire Wire Line
 	4800 4850 4800 5600
+$Comp
+L 8bit-computer-rescue:74HCT08 U32
+U 4 1 5EA11381
+P 2200 5650
+F 0 "U32" H 2200 6016 50  0000 C CNN
+F 1 "74HCT08" H 2200 5925 50  0000 C CNN
+F 2 "Package_DIP:DIP-14_W7.62mm" H 2200 5650 50  0001 C CNN
+F 3 "" H 2200 5650 50  0001 C CNN
+	4    2200 5650
+	-1   0    0    -1
+$EndComp
+$Comp
+L 8bit-computer-rescue:74HCT08 U32
+U 3 1 5EA35B55
+P 2200 6150
+F 0 "U32" H 2200 6516 50  0000 C CNN
+F 1 "74HCT08" H 2200 6425 50  0000 C CNN
+F 2 "Package_DIP:DIP-14_W7.62mm" H 2200 6150 50  0001 C CNN
+F 3 "" H 2200 6150 50  0001 C CNN
+	3    2200 6150
+	-1   0    0    -1
+$EndComp
+Wire Wire Line
+	2800 5750 2950 5750
+Wire Wire Line
+	2950 6250 2800 6250
+Text HLabel 1050 5050 0    60   Output ~ 0
+~PROG
+Wire Wire Line
+	1750 4650 1750 4900
+Wire Wire Line
+	2950 5750 2950 6250
+Wire Wire Line
+	4200 5950 4200 6050
+Connection ~ 4200 6050
+Wire Wire Line
+	4200 6050 5900 6050
+Wire Wire Line
+	2400 4650 2650 4650
+Wire Wire Line
+	2950 4650 4200 4650
+Wire Wire Line
+	4200 5650 4200 4650
+Connection ~ 4200 4650
+Wire Wire Line
+	4200 4650 4350 4650
+Wire Wire Line
+	1750 3700 4700 3700
+Wire Wire Line
+	1050 5050 1750 5050
+Wire Wire Line
+	1750 5050 1750 4900
+Connection ~ 1750 4900
+Wire Wire Line
+	2800 5550 4350 5550
+Wire Wire Line
+	2800 6050 4200 6050
+Connection ~ 2950 5750
+Wire Wire Line
+	3900 4900 3900 5750
+Wire Wire Line
+	3900 5750 3850 5750
+Wire Wire Line
+	1750 4900 3900 4900
+Wire Wire Line
+	1050 5650 1600 5650
+Wire Wire Line
+	1050 6150 1600 6150
 $EndSCHEMATC

Commit message: revision 2.0d
Parts:
- renumbered C16 to C17, C17 to C18, U32 to U29, U29 to U30, U30 to U31, U31 to U32, U84 to U4
Connections:
- net CLK: now also U29.9; no longer U29.1
- net GND: now also SW5.20, SW5.9; no longer SW5.1, SW5.12
- net HL: now also U29.6; no longer U29.8
- net MI: now also U29.10; no longer U29.2
- net STK: now also U29.3; no longer U29.11
- net ~PROG: now also U4.9; no longer U4.3
- net at C17.1, TP15.1, U32.11 (Cp): now also U29.8; no longer U29.3
- net at R15.2, SW5.11: now also U29.1; no longer U29.12
- net at U31.2 (I0a): now also SW5.1; no longer SW5.9
- new net: U29.2, U29.5, U4.8
- new net: R14.2, SW5.12, U29.4
Changed lines of the file:
@@
 P 4250 2850
 AR Path="/5B5601B5" Ref="U?"  Part="1"
-AR Path="/5B55F546/5B5601B5" Ref="U29"  Part="1"
-F 0 "U29" H 4300 3000 50  0000 C CNN
+AR Path="/5B55F546/5B5601B5" Ref="U30"  Part="1"
+F 0 "U30" H 4300 3000 50  0000 C CNN
 F 1 "74LS157" H 4300 2700 50  0000 C CNN
 F 2 "Package_DIP:DIP-16_W7.62mm" H 4250 2850 50  0001 C CNN
@@
 	1000 4750 1000 4650
 $Comp
-L power:VCC #PWR028
+L power:VCC #PWR029
 U 1 1 5B565949
 P 4200 4550
-F 0 "#PWR028" H 4200 4400 50  0001 C CNN
+F 0 "#PWR029" H 4200 4400 50  0001 C CNN
 F 1 "VCC" H 4200 4700 50  0000 C CNN
 F 2 "" H 4200 4550 50  0001 C CNN
@@
 	2900 2400 2900 2500
 $Comp
-L power:GND #PWR029
+L power:GND #PWR028
 U 1 1 5B566978
 P 3200 3300
-F 0 "#PWR029" H 3200 3050 50  0001 C CNN
+F 0 "#PWR028" H 3200 3050 50  0001 C CNN
 F 1 "GND" H 3200 3150 50  0000 C CNN
 F 2 "" H 3200 3300 50  0001 C CNN
@@
 ~CLR
 $Comp
-L Device:C C17
+L Device:C C18
 U 1 1 5B635507
 P 10050 6100
-F 0 "C17" H 10075 6200 50  0000 L CNN
+F 0 "C18" H 10075 6200 50  0000 L CNN
 F 1 "0.1µF" H 10075 6000 50  0000 L CNN
 F 2 "Capacitor_THT:C_Disc_D4.3mm_W1.9mm_P5.00mm" H 10088 5950 50  0001 C CNN
@@
 P 6200 2850
 AR Path="/5F36DA86" Ref="U?"  Part="1"
-AR Path="/5B55F546/5F36DA86" Ref="U30"  Part="1"
-F 0 "U30" H 6250 3000 50  0000 C CNN
+AR Path="/5B55F546/5F36DA86" Ref="U31"  Part="1"
+F 0 "U31" H 6250 3000 50  0000 C CNN
 F 1 "74LS157" H 6250 2700 50  0000 C CNN
 F 2 "Package_DIP:DIP-16_W7.62mm" H 6200 2850 50  0001 C CNN
@@
 Wire Wire Line
 	5900 3600 5900 4450
-Wire Wire Line
-	5650 3600 5650 4500
 Text HLabel 9900 3300 2    60   Input ~ 0
 BUS_4
@@
 	5750 3600 5750 4500
 $Comp
-L 8bit-computer-rescue:74HCT273 U31
+L 8bit-computer-rescue:74HCT273 U32
 U 1 1 5E6918D9
 P 8700 3400
-F 0 "U31" H 8700 4125 50  0000 C CNN
+F 0 "U32" H 8700 4125 50  0000 C CNN
 F 1 "74HCT273" H 8700 4034 50  0000 C CNN
 F 2 "Package_DIP:DIP-20_W7.62mm" H 8700 3400 50  0001 C CNN
@@
 $EndComp
 Wire Wire Line
-	5650 4500 5100 4500
-Wire Wire Line
 	5200 4450 5900 4450
 Wire Wire Line
@@
 Wire Wire Line
 	3950 4300 5600 4300
-Wire Wire Line
-	5100 5550 5100 5600
-Connection ~ 5100 5600
-Wire Wire Line
-	5100 5600 4800 5600
 Wire Wire Line
 	5200 5550 5200 5600
 Connection ~ 5200 5600
 Wire Wire Line
-	5200 5600 5100 5600
-Wire Wire Line
 	5300 5550 5300 5600
 Connection ~ 5300 5600
@@
 	5800 5600 5700 5600
 Wire Wire Line
-	5900 6050 5900 5550
+	5100 6050 5100 5550
 $Comp
 L Device:R R14
@@
 	3700 3600 3700 4250
 $Comp
-L Device:C C16
+L Device:C C17
 U 1 1 60550665
 P 8500 5400
-F 0 "C16" H 8525 5500 50  0000 L CNN
+F 0 "C17" H 8525 5500 50  0000 L CNN
 F 1 "0.01" H 8525 5300 50  0000 L CNN
 F 2 "Capacitor_THT:C_Disc_D4.3mm_W1.9mm_P5.00mm" H 8538 5250 50  0001 C CNN
@@
 	5200 4450 5200 4950
 Wire Wire Line
-	5100 4500 5100 4950
-Wire Wire Line
 	9850 4850 10150 4850
 Wire Wire Line
 	9850 4650 10150 4650
 $Comp
-L 8bit-computer-rescue:74HCT08 U32
-U 1 1 5E6D035A
+L 8bit-computer-rescue:74HCT08 U29
+U 3 1 5E6D035A
 P 9250 4750
-F 0 "U32" H 9250 5116 50  0000 C CNN
+F 0 "U29" H 9250 5116 50  0000 C CNN
 F 1 "74HCT08" H 9250 5025 50  0000 C CNN
 F 2 "Package_DIP:DIP-14_W7.62mm" H 9250 4750 50  0001 C CNN
 F 3 "" H 9250 4750 50  0001 C CNN
-	1    9250 4750
+	3    9250 4750
 	-1   0    0    -1
 $EndComp
@@
 $EndComp
 Wire Wire Line
-	5800 5600 6750 5600
-Wire Wire Line
-	5900 4950 5900 4850
-Wire Wire Line
-	5900 4850 5000 4850
-Wire Wire Line
 	5000 4850 5000 4950
 $Comp
-L 8bit-computer-rescue:74HCT04 U84
-U 2 1 5EC4E515
+L 8bit-computer-rescue:74HCT04 U4
+U 4 1 5EC4E515
 P 3400 5750
-F 0 "U84" H 3400 6065 50  0000 C CNN
+F 0 "U4" H 3400 6065 50  0000 C CNN
 F 1 "74HCT04" H 3400 5974 50  0000 C CNN
 F 2 "Package_DIP:DIP-14_W7.62mm" H 3400 5750 50  0001 C CNN
 F 3 "" H 3400 5750 50  0001 C CNN
-	2    3400 5750
+	4    3400 5750
 	-1   0    0    -1
 $EndComp
@@
 Wire Wire Line
 	5000 4850 4800 4850
-Connection ~ 5000 4850
 Connection ~ 4800 4850
 Wire Wire Line
 	4800 4850 4800 5600
 $Comp
-L 8bit-computer-rescue:74HCT08 U32
-U 4 1 5EA11381
+L 8bit-computer-rescue:74HCT08 U29
+U 1 1 5EA11381
 P 2200 5650
-F 0 "U32" H 2200 6016 50  0000 C CNN
+F 0 "U29" H 2200 6016 50  0000 C CNN
 F 1 "74HCT08" H 2200 5925 50  0000 C CNN
 F 2 "Package_DIP:DIP-14_W7.62mm" H 2200 5650 50  0001 C CNN
 F 3 "" H 2200 5650 50  0001 C CNN
-	4    2200 5650
+	1    2200 5650
 	-1   0    0    -1
 $EndComp
 $Comp
-L 8bit-computer-rescue:74HCT08 U32
-U 3 1 5EA35B55
+L 8bit-computer-rescue:74HCT08 U29
+U 2 1 5EA35B55
 P 2200 6150
-F 0 "U32" H 2200 6516 50  0000 C CNN
+F 0 "U29" H 2200 6516 50  0000 C CNN
 F 1 "74HCT08" H 2200 6425 50  0000 C CNN
 F 2 "Package_DIP:DIP-14_W7.62mm" H 2200 6150 50  0001 C CNN
 F 3 "" H 2200 6150 50  0001 C CNN
-	3    2200 6150
+	2    2200 6150
 	-1   0    0    -1
 $EndComp
@@
 Connection ~ 4200 6050
 Wire Wire Line
-	4200 6050 5900 6050
+	4200 6050 5100 6050
 Wire Wire Line
 	2400 4650 2650 4650
@@
 Wire Wire Line
 	1050 6150 1600 6150
+Wire Wire Line
+	4800 5600 5200 5600
+Wire Wire Line
+	5800 5600 5900 5600
+Wire Wire Line
+	5650 4900 5900 4900
+Wire Wire Line
+	5900 4900 5900 4950
+Wire Wire Line
+	5650 3600 5650 4900
+Wire Wire Line
+	5100 4950 5100 4850
+Wire Wire Line
+	5100 4850 5000 4850
+Connection ~ 5000 4850
+Wire Wire Line
+	5900 5550 5900 5600
+Connection ~ 5900 5600
+Wire Wire Line
+	5900 5600 6750 5600
 $EndSCHEMATC
