File: MK1_CPU/8bit-computer/output.sch (KiCad schematic (older format))
At the start: 18 parts, among them SW5 SW_NKK_GW12LHP, U2 74LS73, U31 LM555, U32 74LS08, U33 74LS273, U35 28C64, U36 7SEGMENT_CC, U37 74LS139, U38 7SEGMENT_CC, U39 7SEGMENT_CC, U40 7SEGMENT_CC

Commit message: version 2.0
Parts:
- removed R52: 10k, Resistor_THT:R_Axial_DIN0207_L6.3mm_D2.5mm_P7.62mm_Horizontal, symbol Device:R
- removed SW5: SW_NKK_GW12LHP, Button_Switch_THT:SW_NKK_GW12LJP, symbol 8bit-computer-rescue:SW_NKK_GW12LHP
- added C20: *, Capacitor_THT:C_Disc_D4.3mm_W1.9mm_P5.00mm, symbol Device:C
- added R18, R19, R20: 10K, Resistor_THT:R_Axial_DIN0207_L6.3mm_D2.5mm_P7.62mm_Horizontal, symbol Device:R
- added SW6: Mode, Button_Switch_THT:SW_DIP_SPSTx03_Slide_9.78x9.8mm_W7.62mm_P2.54mm, symbol Switch:SW_DIP_x03
- added TP16: OI, TestPoint:TestPoint_Pad_1.0x1.0mm, symbol Connector:TestPoint
- C21: renamed from C15; footprint Capacitor_THT:C_Rect_L7.0mm_W6.0mm_P5.00mm -> Capacitor_THT:C_Disc_D4.3mm_W1.9mm_P5.00mm
- C22: renamed from C16; footprint Capacitor_THT:C_Rect_L7.0mm_W6.0mm_P5.00mm -> Capacitor_THT:C_Disc_D4.3mm_W1.9mm_P5.00mm
- U32: value 74LS08 -> 74HCT08; footprint Package_DIP:DIP-14_W7.62mm_Socket -> Package_DIP:DIP-14_W7.62mm; symbol 8bit-computer-rescue:74LS08 -> 8bit-computer-rescue:74HCT08
- U33: renamed from U31; value LM555 -> NE555; footprint Package_DIP:DIP-8_W7.62mm_Socket -> Package_DIP:DIP-8_W7.62mm
- U34: renamed from U33; value 74LS273 -> 74HCT273; footprint Package_DIP:DIP-20_W7.62mm_Socket -> Package_DIP:DIP-20_W7.62mm; symbol 8bit-computer-rescue:74LS273 -> 8bit-computer-rescue:74HCT273
- U35: renamed from U2; value 74LS73 -> 74HCT107; footprint Package_DIP:DIP-14_W7.62mm_Socket -> Package_DIP:DIP-14_W7.62mm; symbol 74xx:74LS73 -> 74xx:74LS107
- U38: renamed from U37; value 74LS139 -> 74HCT139; footprint Package_DIP:DIP-16_W7.62mm_Socket -> Package_DIP:DIP-16_W7.62mm; symbol 8bit-computer-rescue:74LS139 -> 8bit-computer-rescue:74HCT139
- renumbered C13 to C18, C14 to C19, R53 to R16, R54 to R17, U35 to U36, U36 to U37, U38 to U39, U39 to U40, U40 to U41
Connections:
- wire segments 213 -> 227

Commit message: revision 2.0d
Parts:
- renumbered C18 to C19, C19 to C20, C20 to C21, C21 to C22, C22 to C23, U32 to U29
Connections:
- net CLK: now also U29.13; no longer U29.5
- net OI: now also U29.12; no longer U29.4
- net at C21.1, TP16.1, U34.11 (Cp): now also U29.11; no longer U29.6
Changed lines of the file:
@@
 $EndComp
 $Comp
-L Device:C C19
+L Device:C C20
 U 1 1 5B57E38D
 P 900 2800
-F 0 "C19" H 925 2900 50  0000 L CNN
+F 0 "C20" H 925 2900 50  0000 L CNN
 F 1 "0.01µF" H 925 2700 50  0000 L CNN
 F 2 "Capacitor_THT:C_Disc_D4.3mm_W1.9mm_P5.00mm" H 938 2650 50  0001 C CNN
@@
 $EndComp
 $Comp
-L Device:C C18
+L Device:C C19
 U 1 1 5B57E3C8
 P 600 2800
-F 0 "C18" H 625 2900 50  0000 L CNN
+F 0 "C19" H 625 2900 50  0000 L CNN
 F 1 "0.01µF" H 625 2700 50  0000 L CNN
 F 2 "Capacitor_THT:C_Disc_D4.3mm_W1.9mm_P5.00mm" H 638 2650 50  0001 C CNN
@@
 $EndComp
 $Comp
-L 8bit-computer-rescue:74HCT08 U32
-U 2 1 5B57E43D
+L 8bit-computer-rescue:74HCT08 U29
+U 4 1 5B57E43D
 P 1700 4900
-F 0 "U32" H 1700 4950 50  0000 C CNN
+F 0 "U29" H 1700 4950 50  0000 C CNN
 F 1 "74HCT08" H 1700 4850 50  0000 C CNN
 F 2 "Package_DIP:DIP-14_W7.62mm" H 1700 4900 50  0001 C CNN
 F 3 "" H 1700 4900 50  0001 C CNN
-	2    1700 4900
+	4    1700 4900
 	1    0    0    -1
 $EndComp
@@
 Connection ~ 4750 5450
 $Comp
-L Device:C C21
+L Device:C C22
 U 1 1 5B635F85
 P 7000 5350
-F 0 "C21" H 7025 5450 50  0000 L CNN
+F 0 "C22" H 7025 5450 50  0000 L CNN
 F 1 "0.1µF" H 7025 5250 50  0000 L CNN
 F 2 "Capacitor_THT:C_Disc_D4.3mm_W1.9mm_P5.00mm" H 7038 5200 50  0001 C CNN
@@
 $EndComp
 $Comp
-L Device:C C22
+L Device:C C23
 U 1 1 5B64F6D6
 P 7300 5350
-F 0 "C22" H 7325 5450 50  0000 L CNN
+F 0 "C23" H 7325 5450 50  0000 L CNN
 F 1 "0.1µF" H 7325 5250 50  0000 L CNN
 F 2 "Capacitor_THT:C_Disc_D4.3mm_W1.9mm_P5.00mm" H 7338 5200 50  0001 C CNN
@@
 $EndComp
 $Comp
-L Device:C C20
+L Device:C C21
 U 1 1 5E900E70
 P 2750 5200
-F 0 "C20" H 2775 5300 50  0000 L CNN
+F 0 "C21" H 2775 5300 50  0000 L CNN
 F 1 "*" H 2775 5100 50  0000 L CNN
 F 2 "Capacitor_THT:C_Disc_D4.3mm_W1.9mm_P5.00mm" H 2788 5050 50  0001 C CNN
