File: MK1_CPU/8bit-computer/program-counter.sch (KiCad schematic (older format))
At the start: 20 parts, among them U48 74LS245, U49 74LS161, U50 74LS161

Commit message: version 2.0
Parts:
- removed R86, R87, R88, R89, R90, R91, R92, R93: 220, Resistor_THT:R_Axial_DIN0207_L6.3mm_D2.5mm_P7.62mm_Horizontal, symbol Device:R
- added C23: *, Capacitor_THT:C_Disc_D4.3mm_W1.9mm_P5.00mm, symbol Device:C
- added RN6: 220, Resistor_THT:R_Array_SIP9, symbol Device:R_Network08
- added TP17: ~PO, TestPoint:TestPoint_Pad_1.0x1.0mm, symbol Connector:TestPoint
- added TP18: PE, TestPoint:TestPoint_Pad_1.0x1.0mm, symbol Connector:TestPoint
- added TP19: ~PI, TestPoint:TestPoint_Pad_1.0x1.0mm, symbol Connector:TestPoint
- C24: renamed from C19; footprint Capacitor_THT:C_Rect_L7.0mm_W6.0mm_P5.00mm -> Capacitor_THT:C_Disc_D4.3mm_W1.9mm_P5.00mm
- D38: renamed from D68; value GREEN -> YELLOW
- D39: renamed from D69; value GREEN -> YELLOW
- D40: renamed from D70; value GREEN -> YELLOW
- D41: renamed from D71; value GREEN -> YELLOW
- D42: renamed from D72; value GREEN -> YELLOW
- D43: renamed from D73; value GREEN -> YELLOW
- D44: renamed from D74; value GREEN -> YELLOW
- D45: renamed from D75; value GREEN -> YELLOW
- U42: renamed from U48; value 74LS245 -> 74HCT245; footprint Package_DIP:DIP-20_W7.62mm_Socket -> Package_DIP:DIP-20_W7.62mm; symbol 8bit-computer-rescue:74LS245 -> 8bit-computer-rescue:74HCT245
- U43: renamed from U49; value 74LS161 -> 74HCT161; footprint Package_DIP:DIP-16_W7.62mm_Socket -> Package_DIP:DIP-16_W7.62mm; symbol 8bit-computer-rescue:74LS161 -> 8bit-computer-rescue:74HCT161
- U44: renamed from U50; value 74LS161 -> 74HCT161; footprint Package_DIP:DIP-16_W7.62mm_Socket -> Package_DIP:DIP-16_W7.62mm; symbol 8bit-computer-rescue:74LS161 -> 8bit-computer-rescue:74HCT161
Connections:
- net labels added: PE, ~PI, ~PO
- net labels removed: CE, ~CO, ~J
- wire segments 142 -> 150

Commit message: revision 2.0d
Parts:
- C24: renamed from C23; value * -> 0.01µf
- renumbered C24 to C25
Changed lines of the file:
@@
 ~PO
 $Comp
-L Device:C C24
+L Device:C C25
 U 1 1 5B635AE5
 P 8200 2850
-F 0 "C24" H 8225 2950 50  0000 L CNN
+F 0 "C25" H 8225 2950 50  0000 L CNN
 F 1 "0.1µF" H 8225 2750 50  0000 L CNN
 F 2 "Capacitor_THT:C_Disc_D4.3mm_W1.9mm_P5.00mm" H 8238 2700 50  0001 C CNN
@@
 $EndComp
 $Comp
-L Device:C C23
+L Device:C C24
 U 1 1 6181F7E7
 P 7150 4400
-F 0 "C23" H 7175 4500 50  0000 L CNN
-F 1 "*" H 7175 4300 50  0000 L CNN
+F 0 "C24" H 7175 4500 50  0000 L CNN
+F 1 "0.01µf" H 7175 4300 50  0000 L CNN
 F 2 "Capacitor_THT:C_Disc_D4.3mm_W1.9mm_P5.00mm" H 7188 4250 50  0001 C CNN
 F 3 "" H 7150 4400 50  0001 C CNN
