File: MK1_CPU/8bit-computer/ram.sch (KiCad schematic (older format))
At the start: 30 parts, among them SW7 SW_Push, SW8 SW_DIP_x08, U41 74LS00, U51 74LS157, U52 CY62256, U53 74LS245, U54 74LS245, U55 74LS00, U56 74LS157, U57 74LS157

Commit message: version 2.0
Parts:
- removed C20: 0.01µF, Capacitor_THT:C_Disc_D4.3mm_W1.9mm_P5.00mm, symbol Device:C
- removed R100, R101, R94, R95, R96, R97, R98, R99: 220, Resistor_THT:R_Axial_DIN0207_L6.3mm_D2.5mm_P7.62mm_Horizontal, symbol Device:R
- removed R102: 1K, Resistor_THT:R_Axial_DIN0207_L6.3mm_D2.5mm_P7.62mm_Horizontal, symbol Device:R
- removed U55: 74LS00, Package_DIP:DIP-14_W7.62mm_Socket, symbol 8bit-computer-rescue:74LS00
- added C25: *, Capacitor_THT:C_Disc_D4.3mm_W1.9mm_P5.00mm, symbol Device:C
- added D48, D55: YELLOW, LED_THT:LED_D3.0mm, symbol Device:LED_ALT
- added R21, R22: 10K, Resistor_THT:R_Axial_DIN0207_L6.3mm_D2.5mm_P7.62mm_Horizontal, symbol Device:R
- added R23, R24: 220, Resistor_THT:R_Axial_DIN0207_L6.3mm_D2.5mm_P7.62mm_Horizontal, symbol Device:R
- added RN7: 1K, Resistor_THT:R_Array_SIP9, symbol Device:R_Network08
- added SW8: Show, Button_Switch_THT:SW_PUSH_6mm_H5mm, symbol 8bit-computer-rescue:SW_Push-8bit-computer-rescue
- added TP20: ~RO, TestPoint:TestPoint_Pad_1.0x1.0mm, symbol Connector:TestPoint
- added TP21: RI, TestPoint:TestPoint_Pad_1.0x1.0mm, symbol Connector:TestPoint
- added U4: 74HCT04, Package_DIP:DIP-14_W7.62mm, symbol 8bit-computer-rescue:74HCT04
- added unit 3 of U46
- added unit 2 of U46
- added unit 4 of U46
- C26: renamed from C21; footprint Capacitor_THT:C_Rect_L7.0mm_W6.0mm_P5.00mm -> Capacitor_THT:C_Disc_D4.3mm_W1.9mm_P5.00mm
- C27: renamed from C22; footprint Capacitor_THT:C_Rect_L7.0mm_W6.0mm_P5.00mm -> Capacitor_THT:C_Disc_D4.3mm_W1.9mm_P5.00mm
- D46: renamed from D76; value RED -> GREEN
- D47: renamed from D77; value RED -> GREEN
- D49: renamed from D78; value RED -> GREEN
- D50: renamed from D79; value RED -> GREEN
- D51: renamed from D80; value RED -> GREEN
- D52: renamed from D81; value RED -> GREEN
- D53: renamed from D82; value RED -> GREEN
- D54: renamed from D83; value RED -> GREEN
- SW7: value SW_Push -> Write
- SW9: renamed from SW8; value SW_DIP_x08 -> Data
- U45: renamed from U51; value 74LS157 -> 74HCT157; footprint Package_DIP:DIP-16_W7.62mm_Socket -> Package_DIP:DIP-16_W7.62mm; symbol 8bit-computer-rescue:74LS157 -> 8bit-computer-rescue:74HCT157
- U46: renamed from U41; value 74LS00 -> 74HCT00; footprint Package_DIP:DIP-14_W7.62mm_Socket -> Package_DIP:DIP-14_W7.62mm; symbol 8bit-computer-rescue:74LS00 -> 8bit-computer-rescue:74HCT00
- U48: renamed from U53; value 74LS245 -> 74HCT245; footprint Package_DIP:DIP-20_W7.62mm_Socket -> Package_DIP:DIP-20_W7.62mm; symbol 8bit-computer-rescue:74LS245 -> 8bit-computer-rescue:74HCT245
- U49: renamed from U54; value 74LS245 -> 74HCT245; footprint Package_DIP:DIP-20_W7.62mm_Socket -> Package_DIP:DIP-20_W7.62mm; symbol 8bit-computer-rescue:74LS245 -> 8bit-computer-rescue:74HCT245
- U50: renamed from U56; footprint Package_DIP:DIP-16_W7.62mm_Socket -> Package_DIP:DIP-16_W7.62mm; symbol 8bit-computer-rescue:74LS157 -> 8bit-computer-rescue:74HCT157
- U51: renamed from U57; footprint Package_DIP:DIP-16_W7.62mm_Socket -> Package_DIP:DIP-16_W7.62mm; symbol 8bit-computer-rescue:74LS157 -> 8bit-computer-rescue:74HCT157
- renumbered U52 to U47
Connections:
- net labels added: ~PROG
- net labels removed: PROG
- wire segments 296 -> 309

Commit message: 2.0b hardware revision
Parts:
- added C45: 0.01uf, Capacitor_THT:C_Disc_D4.3mm_W1.9mm_P5.00mm, symbol Device:C
Connections:
- net GND: now also C45.2
- net STK: now also C45.1
Changed lines of the file:
@@
 	2400 700  2400 550
 Wire Wire Line
-	2400 550  3850 550
+	2400 550  2850 550
 Connection ~ 3850 550
 Connection ~ 5500 1450
-Wire Wire Line
-	5500 1450 8900 1450
 Wire Wire Line
 	4700 5500 4700 6600
@@
 Wire Wire Line
 	4650 4900 4750 4900
+$Comp
+L Device:C C?
+U 1 1 5EFCB8CD
+P 2850 850
+AR Path="/5B55F546/5EFCB8CD" Ref="C?"  Part="1"
+AR Path="/5B551E96/5EFCB8CD" Ref="C45"  Part="1"
+F 0 "C45" H 2875 950 50  0000 L CNN
+F 1 "0.01uf" H 2875 750 50  0000 L CNN
+F 2 "Capacitor_THT:C_Disc_D4.3mm_W1.9mm_P5.00mm" H 2888 700 50  0001 C CNN
+F 3 "" H 2850 850 50  0001 C CNN
+	1    2850 850
+	1    0    0    -1
+$EndComp
+Wire Wire Line
+	2850 700  2850 550
+Connection ~ 2850 550
+Wire Wire Line
+	2850 550  3850 550
+Wire Wire Line
+	2850 1000 2850 1400
+Wire Wire Line
+	2850 1400 2400 1400
+Connection ~ 2400 1400
+Wire Wire Line
+	5500 1450 8900 1450
 $EndSCHEMATC

Commit message: revision 2.0d
Parts:
- added C44: 0.01µf, Capacitor_THT:C_Disc_D4.3mm_W1.9mm_P5.00mm, symbol Device:C
- C27: renamed from C45; value 0.01uf -> 0.01µf
- renumbered C25 to C26, C26 to C28, C27 to C29
Connections:
- net A0: now also U47.21 (A0); no longer U47.23 (A1)
- net A1: now also U47.23 (A1); no longer U47.24 (A2)
- net A2: now also U47.24 (A2); no longer U47.25 (A3)
- net A3: now also U47.25 (A3); no longer U47.26 (A4)
- net A4: now also U47.26 (A4); no longer U47.1 (A5)
- net A5: now also U47.1 (A5); no longer U47.2 (A6)
- net A6: now also U47.2 (A6); no longer U47.3 (A7)
- net A7: now also U47.3 (A7); no longer U47.4 (A8)
- net GND: now also C44.2
- net HL: now also U47.4 (A8), C44.1; no longer U47.21 (A0)
- net ~PROG: now also U4.11; no longer U4.9
- net at U46.11, U47.22 (~OE~): now also U4.13; no longer U4.11
- net at TP21.1, U48.19 (CE): now also U4.12; no longer U4.10
- net at U46.10: now also U4.10; no longer U4.8
Changed lines of the file:
@@
 Connection ~ 8300 5500
 $Comp
-L Device:C C27
+L Device:C C29
 U 1 1 5B634C8D
 P 10200 1250
-F 0 "C27" H 10225 1350 50  0000 L CNN
+F 0 "C29" H 10225 1350 50  0000 L CNN
 F 1 "0.1µF" H 10225 1150 50  0000 L CNN
 F 2 "Capacitor_THT:C_Disc_D4.3mm_W1.9mm_P5.00mm" H 10238 1100 50  0001 C CNN
@@
 $EndComp
 $Comp
-L Device:C C26
+L Device:C C28
 U 1 1 5B64E398
 P 9900 1250
-F 0 "C26" H 9925 1350 50  0000 L CNN
+F 0 "C28" H 9925 1350 50  0000 L CNN
 F 1 "0.1µF" H 9925 1150 50  0000 L CNN
 F 2 "Capacitor_THT:C_Disc_D4.3mm_W1.9mm_P5.00mm" H 9938 1100 50  0001 C CNN
@@
 A7
 Wire Wire Line
-	4650 650  8900 650
-Wire Wire Line
-	4550 750  8900 750
-Wire Wire Line
-	4450 850  8900 850
-Wire Wire Line
-	4350 950  8900 950
-Wire Wire Line
-	8900 1050 4250 1050
-Wire Wire Line
-	8900 1150 4150 1150
-Wire Wire Line
-	8900 1250 4050 1250
-Wire Wire Line
-	8900 1350 3950 1350
-Wire Wire Line
-	3950 1350 3950 1450
+	8900 1050 4350 1050
+Wire Wire Line
+	8900 1150 4250 1150
+Wire Wire Line
+	8900 1250 4150 1250
+Wire Wire Line
+	8900 1350 4050 1350
+Wire Wire Line
+	4050 1350 4050 1450
 Text HLabel 8900 1450 2    60   Input ~ 0
 HL
@@
 L power:GND #PWR054
 U 1 1 5B55504F
-P 2550 2150
-F 0 "#PWR054" H 2550 1900 50  0001 C CNN
-F 1 "GND" H 2550 2000 50  0000 C CNN
-F 2 "" H 2550 2150 50  0001 C CNN
-F 3 "" H 2550 2150 50  0001 C CNN
-	1    2550 2150
-	1    0    0    -1
-$EndComp
-Wire Wire Line
-	4750 1450 5500 1450
+P 2850 1600
+F 0 "#PWR054" H 2850 1350 50  0001 C CNN
+F 1 "GND" H 2850 1450 50  0000 C CNN
+F 2 "" H 2850 1600 50  0001 C CNN
+F 3 "" H 2850 1600 50  0001 C CNN
+	1    2850 1600
+	1    0    0    -1
+$EndComp
 $Comp
 L 8bit-computer-rescue:74HCT157 U?
@@
 	3250 2750 3250 2450
 Wire Wire Line
-	2550 2000 2750 2000
-Wire Wire Line
-	2550 2000 2550 2150
-Wire Wire Line
-	2750 2550 3350 2550
-Connection ~ 2750 2000
-Wire Wire Line
-	2750 2000 2750 2550
-Wire Wire Line
-	2750 1450 2750 2000
+	2850 1450 2850 1600
 Text HLabel 4600 5500 0    60   Input ~ 0
 RI
@@
 Wire Wire Line
 	2400 1000 2400 1100
-$Comp
-L power:GND #PWR053
-U 1 1 5EADA2E6
-P 2400 1400
-F 0 "#PWR053" H 2400 1150 50  0001 C CNN
-F 1 "GND" H 2400 1250 50  0000 C CNN
-F 2 "" H 2400 1400 50  0001 C CNN
-F 3 "" H 2400 1400 50  0001 C CNN
-	1    2400 1400
-	1    0    0    -1
-$EndComp
 Wire Wire Line
 	2400 700  2400 550
@@
 	2400 550  2850 550
 Connection ~ 3850 550
-Connection ~ 5500 1450
 Wire Wire Line
 	4700 5500 4700 6600
@@
 Connection ~ 3650 1450
 Wire Wire Line
-	4050 1250 4050 1450
-Wire Wire Line
-	4350 950  4350 1450
-Wire Wire Line
-	4450 850  4450 1450
-Wire Wire Line
-	4550 750  4550 1450
-Wire Wire Line
-	4650 650  4650 1450
-Wire Wire Line
-	4150 1150 4150 1450
+	4150 1250 4150 1450
+Wire Wire Line
+	4450 950  4450 1450
+Wire Wire Line
+	4550 850  4550 1450
+Wire Wire Line
+	4650 750  4650 1450
+Wire Wire Line
+	4750 650  4750 1450
+Wire Wire Line
+	4250 1150 4250 1450
 Connection ~ 4750 2450
 Wire Wire Line
-	2750 1450 3350 1450
-Wire Wire Line
 	3350 1450 3450 1450
-Connection ~ 3350 1450
-Wire Wire Line
-	4250 1050 4250 1450
+Wire Wire Line
+	4350 1050 4350 1450
 $Comp
 L 8bit-computer-rescue:CY62256 U47
@@
 $Comp
 L 8bit-computer-rescue:74HCT04 U4
-U 5 1 606744A7
+U 6 1 606744A7
 P 5750 5600
 F 0 "U4" V 5796 5422 50  0000 R CNN
@@
 F 2 "Package_DIP:DIP-14_W7.62mm" H 5750 5600 50  0001 C CNN
 F 3 "" H 5750 5600 50  0001 C CNN
-	5    5750 5600
+	6    5750 5600
 	0    -1   -1   0
 $EndComp
@@
 $Comp
 L 8bit-computer-rescue:74HCT04 U4
-U 4 1 60405EA8
+U 5 1 60405EA8
 P 2950 7800
 F 0 "U4" H 2950 8115 50  0000 C CNN
@@
 F 2 "Package_DIP:DIP-14_W7.62mm" H 2950 7800 50  0001 C CNN
 F 3 "" H 2950 7800 50  0001 C CNN
-	4    2950 7800
+	5    2950 7800
 	1    0    0    -1
 $EndComp
@@
 P 2000 6950
 AR Path="/5B55F546/61951656" Ref="C?"  Part="1"
-AR Path="/5B551E96/61951656" Ref="C25"  Part="1"
-F 0 "C25" H 2025 7050 50  0000 L CNN
+AR Path="/5B551E96/61951656" Ref="C26"  Part="1"
+F 0 "C26" H 2025 7050 50  0000 L CNN
 F 1 "*" H 2025 6850 50  0000 L CNN
 F 2 "Capacitor_THT:C_Disc_D4.3mm_W1.9mm_P5.00mm" H 2038 6800 50  0001 C CNN
@@
 P 2850 850
 AR Path="/5B55F546/5EFCB8CD" Ref="C?"  Part="1"
-AR Path="/5B551E96/5EFCB8CD" Ref="C45"  Part="1"
-F 0 "C45" H 2875 950 50  0000 L CNN
-F 1 "0.01uf" H 2875 750 50  0000 L CNN
+AR Path="/5B551E96/5EFCB8CD" Ref="C27"  Part="1"
+F 0 "C27" H 2875 950 50  0000 L CNN
+F 1 "0.01µf" H 2875 750 50  0000 L CNN
 F 2 "Capacitor_THT:C_Disc_D4.3mm_W1.9mm_P5.00mm" H 2888 700 50  0001 C CNN
 F 3 "" H 2850 850 50  0001 C CNN
@@
 	2850 550  3850 550
 Wire Wire Line
-	2850 1000 2850 1400
-Wire Wire Line
-	2850 1400 2400 1400
-Connection ~ 2400 1400
-Wire Wire Line
-	5500 1450 8900 1450
+	5500 1450 5850 1450
+$Comp
+L Device:C C?
+U 1 1 5FC6F279
+P 5850 1600
+AR Path="/5B55F546/5FC6F279" Ref="C?"  Part="1"
+AR Path="/5B551E96/5FC6F279" Ref="C44"  Part="1"
+F 0 "C44" H 5875 1700 50  0000 L CNN
+F 1 "0.01µf" H 5875 1500 50  0000 L CNN
+F 2 "Capacitor_THT:C_Disc_D4.3mm_W1.9mm_P5.00mm" H 5888 1450 50  0001 C CNN
+F 3 "" H 5850 1600 50  0001 C CNN
+	1    5850 1600
+	1    0    0    -1
+$EndComp
+Connection ~ 5850 1450
+Wire Wire Line
+	5850 1450 8900 1450
+Wire Wire Line
+	5850 2200 5500 2200
+Wire Wire Line
+	5850 1750 5850 2200
+Connection ~ 5500 2200
+Wire Wire Line
+	4450 950  8900 950
+Wire Wire Line
+	4550 850  8900 850
+Wire Wire Line
+	4650 750  8900 750
+Wire Wire Line
+	4750 650  8900 650
+Wire Wire Line
+	5500 1450 5500 1400
+Wire Wire Line
+	5500 1400 3950 1400
+Wire Wire Line
+	3950 1400 3950 1450
+Connection ~ 5500 1450
+Wire Wire Line
+	3350 1450 2850 1450
+Wire Wire Line
+	2850 1000 2850 1450
+Connection ~ 3350 1450
+Wire Wire Line
+	2400 1400 2400 1450
+Wire Wire Line
+	2400 2550 3350 2550
+Wire Wire Line
+	2850 1450 2400 1450
+Connection ~ 2850 1450
+Connection ~ 2400 1450
+Wire Wire Line
+	2400 1450 2400 2550
 $EndSCHEMATC
