File: MK1_CPU/8bit-computer/stack-register.sch (KiCad schematic (older format))
At the start: 24 parts, among them U47 74LS04, U68 74LS245, U69 74LS04, U70 74LS273, U71 74LS04, U72 74LS04, U73 74LS08

Commit message: version 2.0
Parts:
- removed R127, R128, R129, R130, R131, R132, R133, R134: 220, Resistor_THT:R_Axial_DIN0207_L6.3mm_D2.5mm_P7.62mm_Horizontal, symbol Device:R
- removed U47, U69, U71, U72: 74LS04, Package_DIP:DIP-14_W7.62mm_Socket, symbol 8bit-computer-rescue:74LS04
- removed U70: 74LS273, Package_DIP:DIP-20_W7.62mm_Socket, symbol 8bit-computer-rescue:74LS273
- removed U73: 74LS08, Package_DIP:DIP-14_W7.62mm_Socket, symbol 8bit-computer-rescue:74LS08
- added C29, C30, C31: *, Capacitor_THT:C_Disc_D4.3mm_W1.9mm_P5.00mm, symbol Device:C
- added RN8: 220, Resistor_THT:R_Array_SIP9, symbol Device:R_Network08
- added TP22: ~SO, TestPoint:TestPoint_Pad_1.0x1.0mm, symbol Connector:TestPoint
- added TP23: SU, TestPoint:TestPoint_Pad_1.0x1.0mm, symbol Connector:TestPoint
- added TP24: SD, TestPoint:TestPoint_Pad_1.0x1.0mm, symbol Connector:TestPoint
- added TP25: SI, TestPoint:TestPoint_Pad_1.0x1.0mm, symbol Connector:TestPoint
- added U32: 74HCT08, Package_DIP:DIP-14_W7.62mm, symbol 8bit-computer-rescue:74HCT08
- added U53, U54: 74HCT193, Package_DIP:DIP-16_W7.62mm, symbol 74xx_IEEE:74LS193
- added U55: 74HCT00, Package_DIP:DIP-14_W7.62mm, symbol 8bit-computer-rescue:74HCT00
- C28: renamed from C25; footprint Capacitor_THT:C_Rect_L7.0mm_W6.0mm_P5.00mm -> Capacitor_THT:C_Disc_D4.3mm_W1.9mm_P5.00mm
- D56: renamed from D108; value RED -> YELLOW
- D57: renamed from D109; value RED -> YELLOW
- D58: renamed from D110; value RED -> YELLOW
- D59: renamed from D111; value RED -> YELLOW
- D60: renamed from D112; value RED -> YELLOW
- D61: renamed from D113; value RED -> YELLOW
- D62: renamed from D114; value RED -> YELLOW
- D63: renamed from D115; value RED -> YELLOW
- U52: renamed from U68; value 74LS245 -> 74HCT245; footprint Package_DIP:DIP-20_W7.62mm_Socket -> Package_DIP:DIP-20_W7.62mm; symbol 8bit-computer-rescue:74LS245 -> 8bit-computer-rescue:74HCT245
Connections:
- net labels added: CLR, SD, SU, ~SO
- net labels removed: SO, ~CLR
- wire segments 193 -> 172
- no-connect marks 0 -> 2

Commit message: 2.0b hardware revision
Parts:
- U55: renamed from U32; value 74HCT08 -> 74HCT00; symbol 8bit-computer-rescue:74HCT08 -> 8bit-computer-rescue:74HCT00
Connections:
- net CLK: now also U55.10, U55.5; no longer U55.10, U55.13
- net SD: now also U55.9; no longer U55.12
- net SU: now also U55.4; no longer U55.9
- net at C29.1, TP24.1, U54.4 (DOWN): now also U55.8; no longer U55.11
- net at C31.1, TP23.1, U54.5 (UP): now also U55.6; no longer U55.8
Other:
- moved on the sheet: C31, TP23
Changed lines of the file:
@@
 SD
 $Comp
-L 8bit-computer-rescue:74HCT08 U32
-U 4 1 61E1C799
+L 8bit-computer-rescue:74HCT00 U55
+U 3 1 61E1C799
 P 9900 1950
-F 0 "U32" H 9900 2316 50  0000 C CNN
-F 1 "74HCT08" H 9900 2225 50  0000 C CNN
+F 0 "U55" H 9900 2316 50  0000 C CNN
+F 1 "74HCT00" H 9900 2225 50  0000 C CNN
 F 2 "Package_DIP:DIP-14_W7.62mm" H 9900 1950 50  0001 C CNN
 F 3 "" H 9900 1950 50  0001 C CNN
-	4    9900 1950
+	3    9900 1950
 	-1   0    0    -1
 $EndComp
@@
 SU
 $Comp
-L 8bit-computer-rescue:74HCT08 U32
-U 3 1 61E20239
+L 8bit-computer-rescue:74HCT00 U55
+U 2 1 61E20239
 P 9900 1250
-F 0 "U32" H 9900 1616 50  0000 C CNN
-F 1 "74HCT08" H 9900 1525 50  0000 C CNN
+F 0 "U55" H 9900 1616 50  0000 C CNN
+F 1 "74HCT00" H 9900 1525 50  0000 C CNN
 F 2 "Package_DIP:DIP-14_W7.62mm" H 9900 1250 50  0001 C CNN
 F 3 "" H 9900 1250 50  0001 C CNN
-	3    9900 1250
+	2    9900 1250
 	-1   0    0    -1
 $EndComp
@@
 	7550 1950 7550 3100
 Wire Wire Line
-	9300 1250 8900 1250
-Wire Wire Line
 	7650 1250 7650 3100
 Wire Wire Line
@@
 	10750 2050 10750 2950
 Wire Wire Line
-	8900 1650 8900 1750
+	7900 1650 7900 1750
 $Comp
 L Device:C C?
 U 1 1 61E3D8BB
-P 8900 1500
+P 7900 1500
 AR Path="/5B55F546/61E3D8BB" Ref="C?"  Part="1"
 AR Path="/6432FCD8/61E3D8BB" Ref="C31"  Part="1"
-F 0 "C31" H 8925 1600 50  0000 L CNN
-F 1 "*" H 8925 1400 50  0000 L CNN
-F 2 "Capacitor_THT:C_Disc_D4.3mm_W1.9mm_P5.00mm" H 8938 1350 50  0001 C CNN
-F 3 "" H 8900 1500 50  0001 C CNN
-	1    8900 1500
-	1    0    0    -1
-$EndComp
-Wire Wire Line
-	8900 1350 8900 1250
+F 0 "C31" H 7925 1600 50  0000 L CNN
+F 1 "*" H 7925 1400 50  0000 L CNN
+F 2 "Capacitor_THT:C_Disc_D4.3mm_W1.9mm_P5.00mm" H 7938 1350 50  0001 C CNN
+F 3 "" H 7900 1500 50  0001 C CNN
+	1    7900 1500
+	1    0    0    -1
+$EndComp
+Wire Wire Line
+	7900 1350 7900 1250
 $Comp
 L power:GND #PWR?
 U 1 1 61E3D8B3
-P 8900 1750
+P 7900 1750
 AR Path="/5B53AFFA/61E3D8B3" Ref="#PWR?"  Part="1"
 AR Path="/6432FCD8/61E3D8B3" Ref="#PWR070"  Part="1"
-F 0 "#PWR070" H 8900 1500 50  0001 C CNN
-F 1 "GND" H 8900 1600 50  0000 C CNN
-F 2 "" H 8900 1750 50  0001 C CNN
-F 3 "" H 8900 1750 50  0001 C CNN
-	1    8900 1750
-	1    0    0    -1
-$EndComp
-Connection ~ 8900 1250
-Wire Wire Line
-	8900 1250 8250 1250
+F 0 "#PWR070" H 7900 1500 50  0001 C CNN
+F 1 "GND" H 7900 1600 50  0000 C CNN
+F 2 "" H 7900 1750 50  0001 C CNN
+F 3 "" H 7900 1750 50  0001 C CNN
+	1    7900 1750
+	1    0    0    -1
+$EndComp
 $Comp
 L power:GND #PWR?
@@
 L Connector:TestPoint TP?
 U 1 1 777183BC
-P 8250 1200
+P 7900 1200
 AR Path="/5B533ECB/777183BC" Ref="TP?"  Part="1"
 AR Path="/6432FCD8/777183BC" Ref="TP23"  Part="1"
-F 0 "TP23" H 8308 1318 50  0000 L CNN
-F 1 "SU" H 8308 1227 50  0000 L CNN
-F 2 "TestPoint:TestPoint_Pad_1.0x1.0mm" H 8450 1200 50  0001 C CNN
-F 3 "~" H 8450 1200 50  0001 C CNN
-	1    8250 1200
-	1    0    0    -1
-$EndComp
-Wire Wire Line
-	8250 1200 8250 1250
-Connection ~ 8250 1250
-Wire Wire Line
-	8250 1250 7650 1250
+F 0 "TP23" H 7958 1318 50  0000 L CNN
+F 1 "SU" H 7958 1227 50  0000 L CNN
+F 2 "TestPoint:TestPoint_Pad_1.0x1.0mm" H 8100 1200 50  0001 C CNN
+F 3 "~" H 8100 1200 50  0001 C CNN
+	1    7900 1200
+	1    0    0    -1
+$EndComp
+Wire Wire Line
+	7900 1200 7900 1250
 NoConn ~ 6000 4200
 NoConn ~ 6100 4200
@@
 Wire Wire Line
 	6100 2900 6700 2900
+Connection ~ 7900 1250
+Wire Wire Line
+	7900 1250 7650 1250
+Wire Wire Line
+	7900 1250 9300 1250
 $EndSCHEMATC

Commit message: revision 2.0d
Parts:
- renumbered C28 to C30, C29 to C31, C31 to C32, C30 to C33
Connections:
- net CLK: now also U55.10, U55.2, U55.5; no longer U55.10, U55.2, U55.5
- net SD: now also U55.4; no longer U55.9
- net SI: now also U55.9; no longer U55.1
- net SU: now also U55.1; no longer U55.4
- net at C33.1, TP25.1, U53.11 (~LOAD)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: now also U55.8; no longer U55.3
- net at C31.1, TP24.1, U54.4 (DOWN): now also U55.6; no longer U55.8
- net at C32.1, TP23.1, U54.5 (UP): now also U55.3; no longer U55.6
Changed lines of the file:
@@
 P 1800 3450
 AR Path="/5B53AFFA/643B20EF" Ref="C?"  Part="1"
-AR Path="/6432FCD8/643B20EF" Ref="C28"  Part="1"
-F 0 "C28" H 1825 3550 50  0000 L CNN
+AR Path="/6432FCD8/643B20EF" Ref="C30"  Part="1"
+F 0 "C30" H 1825 3550 50  0000 L CNN
 F 1 "0.1µF" H 1825 3350 50  0000 L CNN
 F 2 "Capacitor_THT:C_Disc_D4.3mm_W1.9mm_P5.00mm" H 1838 3300 50  0001 C CNN
@@
 P 8850 3350
 AR Path="/5B53AFFA/6171D2B2" Ref="#PWR?"  Part="1"
-AR Path="/6432FCD8/6171D2B2" Ref="#PWR069"  Part="1"
-F 0 "#PWR069" H 8850 3100 50  0001 C CNN
+AR Path="/6432FCD8/6171D2B2" Ref="#PWR070"  Part="1"
+F 0 "#PWR070" H 8850 3100 50  0001 C CNN
 F 1 "GND" H 8850 3200 50  0000 C CNN
 F 2 "" H 8850 3350 50  0001 C CNN
@@
 P 8850 3100
 AR Path="/5B55F546/6196F0C9" Ref="C?"  Part="1"
-AR Path="/6432FCD8/6196F0C9" Ref="C30"  Part="1"
-F 0 "C30" H 8875 3200 50  0000 L CNN
+AR Path="/6432FCD8/6196F0C9" Ref="C33"  Part="1"
+F 0 "C33" H 8875 3200 50  0000 L CNN
 F 1 "*" H 8875 3000 50  0000 L CNN
 F 2 "Capacitor_THT:C_Disc_D4.3mm_W1.9mm_P5.00mm" H 8888 2950 50  0001 C CNN
@@
 $Comp
 L 8bit-computer-rescue:74HCT00 U55
-U 3 1 61E1C799
+U 2 1 61E1C799
 P 9900 1950
 F 0 "U55" H 9900 2316 50  0000 C CNN
@@
 F 2 "Package_DIP:DIP-14_W7.62mm" H 9900 1950 50  0001 C CNN
 F 3 "" H 9900 1950 50  0001 C CNN
-	3    9900 1950
+	2    9900 1950
 	-1   0    0    -1
 $EndComp
@@
 $Comp
 L 8bit-computer-rescue:74HCT00 U55
-U 2 1 61E20239
+U 1 1 61E20239
 P 9900 1250
 F 0 "U55" H 9900 1616 50  0000 C CNN
@@
 F 2 "Package_DIP:DIP-14_W7.62mm" H 9900 1250 50  0001 C CNN
 F 3 "" H 9900 1250 50  0001 C CNN
-	2    9900 1250
+	1    9900 1250
 	-1   0    0    -1
 $EndComp
@@
 $Comp
 L 8bit-computer-rescue:74HCT00 U55
-U 1 1 61E25797
+U 3 1 61E25797
 P 9900 2850
 F 0 "U55" H 9900 3256 50  0000 C CNN
@@
 F 2 "Package_DIP:DIP-14_W7.62mm" H 9900 2850 50  0001 C CNN
 F 3 "" H 9900 2850 50  0001 C CNN
-	1    9900 2850
+	3    9900 2850
 	-1   0    0    -1
 $EndComp
@@
 P 7900 1500
 AR Path="/5B55F546/61E3D8BB" Ref="C?"  Part="1"
-AR Path="/6432FCD8/61E3D8BB" Ref="C31"  Part="1"
-F 0 "C31" H 7925 1600 50  0000 L CNN
+AR Path="/6432FCD8/61E3D8BB" Ref="C32"  Part="1"
+F 0 "C32" H 7925 1600 50  0000 L CNN
 F 1 "*" H 7925 1400 50  0000 L CNN
 F 2 "Capacitor_THT:C_Disc_D4.3mm_W1.9mm_P5.00mm" H 7938 1350 50  0001 C CNN
@@
 P 7900 1750
 AR Path="/5B53AFFA/61E3D8B3" Ref="#PWR?"  Part="1"
-AR Path="/6432FCD8/61E3D8B3" Ref="#PWR070"  Part="1"
-F 0 "#PWR070" H 7900 1500 50  0001 C CNN
+AR Path="/6432FCD8/61E3D8B3" Ref="#PWR069"  Part="1"
+F 0 "#PWR069" H 7900 1500 50  0001 C CNN
 F 1 "GND" H 7900 1600 50  0000 C CNN
 F 2 "" H 7900 1750 50  0001 C CNN
@@
 P 6000 2250
 AR Path="/5B55F546/61E4E10B" Ref="C?"  Part="1"
-AR Path="/6432FCD8/61E4E10B" Ref="C29"  Part="1"
-F 0 "C29" H 6025 2350 50  0000 L CNN
+AR Path="/6432FCD8/61E4E10B" Ref="C31"  Part="1"
+F 0 "C31" H 6025 2350 50  0000 L CNN
 F 1 "*" H 6025 2150 50  0000 L CNN
 F 2 "Capacitor_THT:C_Disc_D4.3mm_W1.9mm_P5.00mm" H 6038 2100 50  0001 C CNN
