File: MK1_CPU/8bit-computer/ext_interface.sch (KiCad schematic (older format))
At the start: 17 parts, among them J3 EXT-Bus, J4 EXT-Signal, J5 EXT-Power, U64 74HCT08, U71 74HCT02, U72 74HCT245, U73 74HCT107, U74 74HCT08

Commit message: 2.0b hardware revision
Parts:
- added R26, R27: 1K, symbol Device:R
Connections:
- net GND: now also R26.2, R27.2
- net at J4.1 (Pin_1), U73.1 (J): now also R26.1
- net at J4.2 (Pin_2), U73.8 (J): now also R27.1
Changed lines of the file:
@@
 	6250 4500 6500 4500
 Wire Wire Line
-	5500 5100 5500 7000
-Wire Wire Line
-	5400 4500 5400 7000
+	5500 5100 5500 6350
+Wire Wire Line
+	5400 4500 5400 6250
 Wire Wire Line
 	5450 5000 5150 5000
@@
 	0    -1   1    0
 $EndComp
+Connection ~ 5400 6250
+Wire Wire Line
+	5400 6250 5400 7000
+Connection ~ 5500 6350
+Wire Wire Line
+	5500 6350 5500 7000
+$Comp
+L Device:R R27
+U 1 1 5EC16046
+P 4800 6650
+F 0 "R27" H 4870 6696 50  0000 L CNN
+F 1 "1K" H 4870 6605 50  0000 L CNN
+F 2 "" V 4730 6650 50  0001 C CNN
+F 3 "~" H 4800 6650 50  0001 C CNN
+	1    4800 6650
+	1    0    0    -1
+$EndComp
+$Comp
+L Device:R R26
+U 1 1 5EC16961
+P 4550 6650
+F 0 "R26" H 4620 6696 50  0000 L CNN
+F 1 "1K" H 4620 6605 50  0000 L CNN
+F 2 "" V 4480 6650 50  0001 C CNN
+F 3 "~" H 4550 6650 50  0001 C CNN
+	1    4550 6650
+	1    0    0    -1
+$EndComp
+Wire Wire Line
+	4800 6350 4800 6500
+Wire Wire Line
+	4800 6350 5500 6350
+Wire Wire Line
+	4550 6250 4550 6500
+Wire Wire Line
+	4550 6250 5400 6250
+Wire Wire Line
+	4550 6800 4550 6900
+Wire Wire Line
+	4550 6900 4650 6900
+Wire Wire Line
+	4800 6900 4800 6800
+$Comp
+L power:GND #PWR096
+U 1 1 5EC29412
+P 4650 7000
+F 0 "#PWR096" H 4650 6750 50  0001 C CNN
+F 1 "GND" H 4655 6827 50  0000 C CNN
+F 2 "" H 4650 7000 50  0001 C CNN
+F 3 "" H 4650 7000 50  0001 C CNN
+	1    4650 7000
+	1    0    0    -1
+$EndComp
+Wire Wire Line
+	4650 7000 4650 6900
+Connection ~ 4650 6900
+Wire Wire Line
+	4650 6900 4800 6900
 $EndSCHEMATC

Commit message: revision 2.0d
Parts:
- removed J4: EXT-Signal, Connector_PinHeader_2.54mm:PinHeader_1x08_P2.54mm_Vertical, symbol Connector_Generic:Conn_01x08
- removed J5: EXT-Power, Connector_PinHeader_2.54mm:PinHeader_1x02_P2.54mm_Vertical, symbol Connector_Generic:Conn_01x02
- J4: renamed from J3; value EXT-Bus -> EXT-CONN; footprint Connector_PinHeader_2.54mm:PinHeader_1x08_P2.54mm_Vertical -> Connector_PinHeader_2.54mm:PinHeader_2x09_P2.54mm_Vertical; symbol Connector_Generic:Conn_01x08 -> Connector_Generic:Conn_02x09_Odd_Even
- R27: renamed from R26; footprint (none) -> Resistor_THT:R_Axial_DIN0207_L6.3mm_D2.5mm_P7.62mm_Horizontal
- R28: renamed from R27; footprint (none) -> Resistor_THT:R_Axial_DIN0207_L6.3mm_D2.5mm_P7.62mm_Horizontal
- renumbered D96 to D88, D97 to D89, R33 to R25, R34 to R26, TP35 to TP34, TP36 to TP35, TP37 to TP36, TP38 to TP37, TP39 to TP38, U74 to U64, U71 to U69, U72 to U70, U73 to U71
Connections:
- net CLK: now also J4.15 (Pin_15)
- net CLR: now also J4.13 (Pin_13)
- net E0: now also J4.5 (Pin_5), U64.10; no longer U64.2
- net E1: now also J4.7 (Pin_7), U64.5; no longer U64.13
- net EXT_IN: now also U64.4, U64.9; no longer U64.1, U64.12
- net GND: now also J4.17 (Pin_17)
- net U0: now also J4.9 (Pin_9)
- net U1: now also J4.11 (Pin_11)
- net VCC: now also J4.18 (Pin_18)
- net at U70.2 (A0): now also J4.2 (Pin_2); no longer J4.1 (Pin_1)
- net at U70.3 (A1): now also J4.4 (Pin_4); no longer J4.2 (Pin_2)
- net at U70.4 (A2): now also J4.6 (Pin_6); no longer J4.3 (Pin_3)
- net at U70.5 (A3): now also J4.8 (Pin_8); no longer J4.4 (Pin_4)
- net at U70.6 (A4): now also J4.10 (Pin_10); no longer J4.5 (Pin_5)
- net at U70.7 (A5): now also J4.12 (Pin_12); no longer J4.6 (Pin_6)
- net at U70.8 (A6): now also J4.14 (Pin_14); no longer J4.7 (Pin_7)
- net at U70.9 (A7): now also J4.16 (Pin_16); no longer J4.8 (Pin_8)
- net at R27.1, U71.1 (J): now also J4.1 (Pin_1)
- net at R28.1, U71.8 (J): now also J4.3 (Pin_3)
- net at U69.5: now also U64.6; no longer U64.11
- net at U69.9: now also U64.8; no longer U64.3
Other:
- moved on the sheet: R27, R28, U71C

Commit message: PCB tracks revision
Parts:
- added C45: 0.01µF, Capacitor_THT:C_Disc_D4.3mm_W1.9mm_P5.00mm, symbol Device:C
Connections:
- net EXT_IN: now also C45.1
- net GND: now also C45.2
Changed lines of the file:
@@
 $EndComp
 Wire Wire Line
-	5000 4550 5000 4750
+	5000 4550 5000 4700
 Connection ~ 3600 3750
 Connection ~ 3500 3650
@@
 Connection ~ 2700 3450
 Wire Wire Line
-	2700 3450 5000 3450
+	2700 3450 3150 3450
 $Comp
 L Connector:TestPoint TP?
@@
 Wire Wire Line
 	6050 1800 6050 2600
+$Comp
+L Device:C C?
+U 1 1 5EA144EC
+P 3150 4050
+AR Path="/5B57D8E5/5EA144EC" Ref="C?"  Part="1"
+AR Path="/6017B840/5EA144EC" Ref="C45"  Part="1"
+F 0 "C45" H 3175 4150 50  0000 L CNN
+F 1 "0.01µF" H 3175 3950 50  0000 L CNN
+F 2 "Capacitor_THT:C_Disc_D4.3mm_W1.9mm_P5.00mm" H 3188 3900 50  0001 C CNN
+F 3 "" H 3150 4050 50  0001 C CNN
+	1    3150 4050
+	1    0    0    -1
+$EndComp
+Wire Wire Line
+	3150 3900 3150 3450
+Connection ~ 3150 3450
+Wire Wire Line
+	3150 3450 5000 3450
+Wire Wire Line
+	3150 4200 3150 4700
+Wire Wire Line
+	3150 4700 5000 4700
+Connection ~ 5000 4700
+Wire Wire Line
+	5000 4700 5000 4750
 $EndSCHEMATC
